File: focus_coil/focus_coil_drive.brd (EAGLE design)
At the start: 203.2 x 101.6 mm, 8 parts, among them J1 JST-VH-2, P1 44PINEDGE, P2 5K, Q1 MJ15016G

Commit message: more work
Parts:
- removed Q1: MJ15016G, keiths:TO3
- J1: value JST-VH-2 -> JST-VH-3; device keiths:VHR-2N -> keiths:VHR-3N
- moved J1 52.1 mm to (12.7, -57.1)
Connections:
- removed net FOCUS_COIL_1: Q1.C, Q1.C/
- net +50V: now also J1.P$1
- net BASE: now also J1.P$2; no longer J1.P$1, Q1.B
- net GND: now also J1.P$3; no longer J1.P$2
Changed lines of the file:
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@@
 </autorouter>
 <elements>
-<element name="Q1" library="keiths" package="TO3" value="MJ15016G" x="162.56" y="46.99" smashed="yes" rot="R180">
-<attribute name="NAME" x="185.42" y="40.64" size="1.9304" layer="25" font="vector" ratio="10" rot="R180"/>
-<attribute name="VALUE" x="156.21" y="62.23" size="1.9304" layer="27" font="vector" ratio="10" rot="R180" display="off"/>
-</element>
 <element name="D16" library="keiths" package="DO35-7" value="1N4148" x="88.9" y="62.23"/>
 <element name="D1" library="keiths" package="DO35-7" value="1N4148" x="74.93" y="62.23"/>
@@
 </element>
 <element name="R3" library="keiths" package="0207/10" value="8.2K" x="38.1" y="62.23" rot="R180"/>
-<element name="J1" library="keiths" package="VHR-2N" value="JST-VH-2" x="12.7" y="-5.08"/>
 <element name="P1" library="keiths" package="44PINEDGE" value="44PINEDGE" x="46.99" y="-24.13"/>
+<element name="J1" library="keiths" package="VHR-3N" value="JST-VH-3" x="12.7" y="-57.15"/>
 </elements>
 <signals>
-<signal name="FOCUS_COIL_1">
-<contactref element="Q1" pad="C/"/>
-<contactref element="Q1" pad="C"/>
-<wire x1="177.673" y1="46.99" x2="147.447" y2="46.99" width="0" layer="19" extent="1-1"/>
-</signal>
 <signal name="BASE">
-<contactref element="Q1" pad="B"/>
 <contactref element="P2" pad="2"/>
-<contactref element="J1" pad="P$1"/>
-<wire x1="64.643" y1="40.64" x2="164.338" y2="41.529" width="0" layer="19" extent="1-1"/>
-<wire x1="3.7" y1="-3.1" x2="64.643" y2="40.64" width="0" layer="19" extent="1-1"/>
+<contactref element="J1" pad="P$2"/>
+<wire x1="3.7" y1="-57.15" x2="64.643" y2="40.64" width="0" layer="19" extent="1-1"/>
 </signal>
 <signal name="+50V">
 <contactref element="D16" pad="A"/>
 <contactref element="P1" pad="E"/>
+<contactref element="J1" pad="P$1"/>
 <wire x1="21.2344" y1="-19.304" x2="92.71" y2="62.23" width="0" layer="19" extent="16-16"/>
+<wire x1="3.7" y1="-61.11875" x2="21.2344" y2="-19.304" width="0" layer="19" extent="16-16"/>
 </signal>
 <signal name="N$1">
@@
 <signal name="GND">
 <contactref element="R3" pad="2"/>
-<contactref element="J1" pad="P$2"/>
 <contactref element="P1" pad="D"/>
-<wire x1="3.7" y1="-7.06" x2="33.02" y2="62.23" width="0" layer="19" extent="1-1"/>
-<wire x1="17.272" y1="-19.304" x2="3.7" y2="-7.06" width="0" layer="19" extent="16-16"/>
+<contactref element="J1" pad="P$3"/>
+<wire x1="17.272" y1="-19.304" x2="33.02" y2="62.23" width="0" layer="19" extent="16-16"/>
+<wire x1="3.7" y1="-53.18125" x2="17.272" y2="-19.304" width="0" layer="19" extent="16-16"/>
 </signal>
 </signals>
