File: focus_coil/focus_coil_drive.sch (EAGLE design)
At the start: 8 parts, among them J1 JST-VH-2, P1 44PINEDGE, P2 5K, Q1 MJ15016G

Commit message: more work
Parts:
- removed Q1: MJ15016G, keiths:MJ15016G
- J1: value JST-VH-2 -> JST-VH-3; device keiths:JST-VH-2 -> keiths:JST-VH-3
Connections:
- removed net FOCUS_COIL_1: Q1.C
- net +50V: now also J1.1
- net BASE: now also J1.2; no longer J1.1, Q1.B
- net GND: now also J1.3; no longer J1.2
Other:
- note added: "to focus transistor"
- note removed: "To external focus transistor."
- moved on the sheet: D1, D16, P1, P2, R3, ZD1
