File: yoke/mimic1567heatSink.brd (EAGLE design)
At the start: 762 x 762 mm, 72 parts, among them J1 COIL 1, J10 8 PIN JONES, J11 GND, J12 JST-VH-2, J13 OUT_2, J14 RESISTOR_2, J15 265 V, J16 GND, J17 265 V, J18 GND, J19 GND, J2 OUT_1, J20 GND, J21 GND, J22 2 Pin Jones, J23 JST-VH-2, J24 JST-VH-2, J25 JST-VH-2, J26 JST-VH-2, J27 JST-VH-2, J28 JST-VH-5, J29 JST-VH-2, J3 RESISTOR_1, J30 JST-VH-2, J31 JST-VH-2, J32 JST-VH-2, J33 JST-VH-5, J34 JST-VH-2, J35 JST-VH-2, J36 JST-VH-2, J4 COIL 2, J5 COIL 1, J6 OUT_1, J7 OUT_2, J8 RESISTOR_2, J9 RESISTOR_1, P1 1 K, P2 1 K, P3 1 K, P4 1 K, Q1 MJ10007, Q2 MJ10007, Q3 MJ10007, Q4 MJ10007, Q5 MJ15016G

Commit message: more work
Parts:
- removed J13, J7: OUT_2, keiths:AWG18
- removed J21: GND, keiths:AWG18
- removed J23, J24, J25, J26, J27, J29, J32, J34, J35, J36: JST-VH-2, keiths:VHR-2N
- removed J4: COIL 2, keiths:AWG18
- removed J8: RESISTOR_2, keiths:AWG18
- added J37: +265 V, keiths:AWG18
- J1: value COIL 1 -> JST-VH-5; device keiths:AWG18 -> keiths:VHR-5N
- J11: value GND -> +50V
- J12: value JST-VH-2 -> JST-VH-3; device keiths:VHR-2N -> keiths:VHR-3N
- J14: value RESISTOR_2 -> JST-VH-2; device keiths:AWG18 -> keiths:VHR-2N
- J15, J17: value 265 V -> JST-VH-3; device keiths:AWG18 -> keiths:VHR-3N
- J18: value GND -> JST-VH-2; device keiths:AWG18 -> keiths:VHR-2N
- J19, J20: value GND -> JST-VH-3; device keiths:AWG18 -> keiths:VHR-3N
- J2: value OUT_1 -> JST-VH-3; device keiths:AWG18 -> keiths:VHR-3N
- J3, J9: value RESISTOR_1 -> JST-VH-3; device keiths:AWG18 -> keiths:VHR-3N
- J5: value COIL 1 -> JST-VH-3; device keiths:AWG18 -> keiths:VHR-3N
- J6: value OUT_1 -> JST-VH-5; device keiths:AWG18 -> keiths:VHR-5N
- moved J20 1411.1 mm to (-33.0, -614.7)
- moved J14 1388.6 mm to (-33.0, -582.9)
- moved J18 1334.0 mm to (-33.0, -591.8)
- moved J3 1319.4 mm to (-33.0, -627.4)
- moved J19 1282.2 mm to (-33.0, -602.0)
- moved J2 1186.3 mm to (-33.0, -519.4)
- moved Q1 1179.0 mm to (-24.1, -500.4), turned to 0 degrees
- moved J1 1133.2 mm to (48.3, -497.8)
- moved J9 1132.1 mm to (-33.0, -359.4)
- moved R1 1124.2 mm to (14.0, -415.3)
- moved J5 1119.6 mm to (-33.0, -372.1)
- moved R2 1104.6 mm to (14.0, -463.6)
- moved Q2 1098.3 mm to (16.5, -500.4), turned to 0 degrees
- moved J6 1092.9 mm to (-33.0, -342.9)
- moved J15 706.1 mm to (-33.0, -326.4)
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Connections:
- removed net N$34: J17.P$1, R8.1
- removed net N$35: J13.P$1, Q4.B
- removed net N$37: J20.P$1, R9.P$2
- removed net N$38: J21.P$1, R10.P$2
- removed net N$39: J27.P$1, J33.P$1
- removed net N$40: J26.P$1, J33.P$2
- removed net N$41: J25.P$1, J33.P$3
- removed net N$42: J12.P$1, J33.P$4
- new net +265V: J17.P$1, R5.1, R8.1
- new net N$13: J15.P$1, J37.P$1
- new net N$17: J15.P$3, J16.P$1
- new net N$25: J19.P$1, J3.P$1
- net +50V: now also J17.P$2, J20.P$1
- net FOCUS_COIL: now also J18.P$1; no longer J24.P$1
- net GND: now also C1.P$2, C2.P$2, D12.A, D5.A, J1.P$5, J12.P$3, J17.P$3, J18.P$2, J2.P$3, J20.P$3, J28.P$5, J5.P$3, J6.P$5, J9.P$3, P1.E, P2.E, P3.E, P4.E, R1.P$2, R10.P$2, R2.P$2, R3.2, R4.2, R6.2, R7.2, R9.P$2; no longer J24.P$2, J29.P$2
- net N$1: now also J20.P$2; no longer J29.P$1
- net N$16: now also J15.P$2; no longer C1.P$2, C2.P$2, D12.A, D5.A, J16.P$1, J28.P$5, P1.E, P2.E, P3.E, P4.E, R3.2, R4.2, R6.2, R7.2
- net N$2: now also J1.P$1; no longer J2.P$1
- net N$20: now also J6.P$3, Q4.B; no longer J15.P$1, R5.1
- net N$24: now also J14.P$2; no longer J32.P$2
- net N$28: now also J6.P$2; no longer J9.P$1
- net N$3: now also J1.P$2; no longer J3.P$1
- net N$32: now also J14.P$1; no longer J32.P$1
- net N$36: now also J6.P$4; no longer J14.P$1
- net N$5: now also J1.P$4, Q2.E, R2.P$1; no longer J7.P$1, Q2.B
- net N$6: now also J1.P$3, Q2.B; no longer J8.P$1, Q2.E, R2.P$1
- net N$7: now also J19.P$3, J3.P$3; no longer J18.P$1, R1.P$2
- net N$8: now also J19.P$2, J3.P$2; no longer J19.P$1, R2.P$2
- net X_A: now also J12.P$1, J2.P$1, J33.P$1; no longer J1.P$1
- net X_B: now also J12.P$2, J2.P$2, J33.P$2; no longer J4.P$1
- net Y_A: now also J33.P$3, J9.P$1
- net Y_B: now also J33.P$4, J5.P$2, J9.P$2; no longer J23.P$1
