File: yoke/mimic1567heatSink.sch (EAGLE design)
At the start: 72 parts, among them J1 COIL 1, J10 8 PIN JONES, J11 GND, J12 JST-VH-2, J13 OUT_2, J14 RESISTOR_2, J15 265 V, J16 GND, J17 265 V, J18 GND, J19 GND, J2 OUT_1, J20 GND, J21 GND, J22 2 Pin Jones, J23 JST-VH-2, J24 JST-VH-2, J25 JST-VH-2, J26 JST-VH-2, J27 JST-VH-2, J28 JST-VH-5, J29 JST-VH-2, J3 RESISTOR_1, J30 JST-VH-2, J31 JST-VH-2, J32 JST-VH-2, J33 JST-VH-5, J34 JST-VH-2, J35 JST-VH-2, J36 JST-VH-2, J4 COIL 2, J5 COIL 1, J6 OUT_1, J7 OUT_2, J8 RESISTOR_2, J9 RESISTOR_1, P1 1 K, P2 1 K, P3 1 K, P4 1 K, Q1 MJ10007, Q2 MJ10007, Q3 MJ10007, Q4 MJ10007, Q5 MJ15016G

Commit message: more work
Parts:
- removed J13, J7: OUT_2, keiths:AWG18
- removed J21: GND, keiths:AWG18
- removed J23, J24, J25, J26, J27, J29, J32, J34, J35, J36: JST-VH-2, keiths:JST-VH-2
- removed J4: COIL 2, keiths:AWG18
- removed J8: RESISTOR_2, keiths:AWG18
- added J37: +265 V, keiths:AWG18
- J1: value COIL 1 -> JST-VH-5; device keiths:AWG18 -> keiths:JST-VH-5
- J11: value GND -> +50V
- J12: value JST-VH-2 -> JST-VH-3; device keiths:JST-VH-2 -> keiths:JST-VH-3
- J14: value RESISTOR_2 -> JST-VH-2; device keiths:AWG18 -> keiths:JST-VH-2
- J15, J17: value 265 V -> JST-VH-3; device keiths:AWG18 -> keiths:JST-VH-3
- J18: value GND -> JST-VH-2; device keiths:AWG18 -> keiths:JST-VH-2
- J19, J20: value GND -> JST-VH-3; device keiths:AWG18 -> keiths:JST-VH-3
- J2: value OUT_1 -> JST-VH-3; device keiths:AWG18 -> keiths:JST-VH-3
- J3, J9: value RESISTOR_1 -> JST-VH-3; device keiths:AWG18 -> keiths:JST-VH-3
- J5: value COIL 1 -> JST-VH-3; device keiths:AWG18 -> keiths:JST-VH-3
- J6: value OUT_1 -> JST-VH-5; device keiths:AWG18 -> keiths:JST-VH-5
Connections:
- removed net N$34: J17.P$1, R8.P$1
- removed net N$35: J13.P$1, Q4.B
- removed net N$37: J20.P$1, R9.P$2
- removed net N$38: J21.P$1, R10.P$2
- removed net N$39: J27.1, J33.1
- removed net N$40: J26.1, J33.2
- removed net N$41: J25.1, J33.3
- removed net N$42: J12.1, J33.4
- new net +265V: J17.1, R5.P$1, R8.P$1
- new net N$13: J15.1, J37.P$1
- new net N$17: J15.3, J16.P$1
- new net N$25: J19.1, J3.1
- net +50V: now also J17.2, J20.1
- net FOCUS_COIL: now also J18.1; no longer J24.1
- net GND: now also C1.2, C2.2, D12.A, D5.A, J1.5, J12.3, J17.3, J18.2, J2.3, J20.3, J28.5, J5.3, J6.5, J9.3, P1.3, P2.3, P3.3, P4.3, R1.P$2, R10.P$2, R2.P$2, R3.P$2, R4.P$2, R6.P$2, R7.P$2, R9.P$2; no longer J24.2, J29.2
- net N$1: now also J20.2; no longer J29.1
- net N$16: now also J15.2; no longer C1.2, C2.2, D12.A, D5.A, J16.P$1, J28.5, P1.3, P2.3, P3.3, P4.3, R3.P$2, R4.P$2, R6.P$2, R7.P$2
- net N$2: now also J1.1; no longer J2.P$1
- net N$20: now also J6.3, Q4.B; no longer J15.P$1, R5.P$1
- net N$24: now also J14.2; no longer J32.2
- net N$26: now also J6.1; no longer J6.P$1
- net N$28: now also J6.2; no longer J9.P$1
- net N$3: now also J1.2; no longer J3.P$1
- net N$32: now also J14.1; no longer J32.1
- net N$36: now also J6.4; no longer J14.P$1
- net N$5: now also J1.4, Q2.E, R2.P$1; no longer J7.P$1, Q2.B
- net N$6: now also J1.3, Q2.B; no longer J8.P$1, Q2.E, R2.P$1
- net N$7: now also J19.3, J3.3; no longer J18.P$1, R1.P$2
- net N$8: now also J19.2, J3.2; no longer J19.P$1, R2.P$2
- net X_A: now also J12.1, J2.1, J33.1; no longer J1.P$1
- net X_B: now also J12.2, J2.2, J33.2; no longer J4.P$1
- net Y_A: now also J33.3, J5.1, J9.1; no longer J5.P$1
- net Y_B: now also J33.4, J5.2, J9.2; no longer J23.1
Other:
- note added: "Damping plate assembly."
- note added: "Focus coil cable one from card cage to focus coil drive transistor."
- note added: "Focus coil cable two from Drive Transistor to damping plate."
- note added: "Focus coil drive transistor."
- note added: "X Yoke Current"
- note added: "Y Yoke Current."
- note added: "Yoke Current Cable."
- moved on the sheet: C1, C2, D1, D10, D11, D12, D13, D14, D2, D3, D4, D5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

Commit message: EOD backup
Other:
- note added: "5 x 20 Volts Zeners"
Changed lines of the file:
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@@
 <text x="76.2" y="281.94" size="5.08" layer="91" font="vector" ratio="10">X Yoke Current</text>
 <text x="76.2" y="129.54" size="5.08" layer="91" font="vector" ratio="10">Y Yoke Current.</text>
+<text x="477.52" y="200.66" size="3.81" layer="91" font="vector" ratio="10">5 x 20 Volts
+Zeners</text>
 </plain>
 <instances>
