File: yoke/mimic1575.sch (EAGLE design)
At the start: 69 parts, among them P1 20, P6 44PINEDGE, Q1 2N3904, Q10 2N3906, Q11 2N3904, Q12 2N3904, Q13 2N3904, Q14 2N3906, Q15 2N3904, Q16 2N2222A, Q19 2N2907, Q2 2N3904, Q20 2N3904, Q21 2N3906, Q22 2N3906, Q3 2N3904, Q4 2N3904, Q5 2N2222A, Q6 2N3904, Q7 2N3906, Q8 2N3904, Q9 2N3906

Commit message: update netlist
Parts:
- Q1, Q12: value 2N3904 -> KSP05TA; device keiths:2N3904 -> keiths:KSP05TA; PN 2N3904 -> (none)
Changed lines of the file:
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@@
 <part name="R12" library="keiths" deviceset="AXIALRESISTOR" device="QUARTER_WATT" value="470"/>
 <part name="R14" library="keiths" deviceset="AXIALRESISTOR" device="QUARTER_WATT" value="27"/>
-<part name="Q1" library="keiths" deviceset="2N3904" device="">
-<attribute name="PN" value="2N3904"/>
-</part>
 <part name="C1" library="keiths" deviceset="CAP0.1UF100V" device="" value="0.001uF">
 <attribute name="MPN" value="1000 pf"/>
@@
 <part name="SUPPLY3" library="supply2" deviceset="GND" device=""/>
 <part name="D2" library="keiths" deviceset="1N4148" device="" value="1N4148"/>
-<part name="Q12" library="keiths" deviceset="2N3904" device="">
-<attribute name="PN" value="2N3904"/>
-</part>
 <part name="R3" library="keiths" deviceset="AXIALRESISTOR" device="QUARTER_WATT" value="680"/>
 <part name="R24" library="keiths" deviceset="AXIALRESISTOR" device="QUARTER_WATT" value="680"/>
@@
 </part>
 <part name="Q16" library="keiths" deviceset="2N2222" device="" technology="A"/>
+<part name="Q1" library="keiths" deviceset="KSP05TA" device=""/>
+<part name="Q12" library="keiths" deviceset="KSP05TA" device=""/>
 </parts>
 <sheets>
@@
 <attribute name="VALUE" x="254.508" y="215.392" size="1.9304" layer="96" font="vector" ratio="10"/>
 </instance>
-<instance part="Q1" gate="G1" x="236.22" y="162.56" smashed="yes" rot="MR0">
-<attribute name="NAME" x="238.76" y="166.37" size="1.9304" layer="95" font="vector" ratio="10"/>
-<attribute name="VALUE" x="238.76" y="157.48" size="1.9304" layer="96" font="vector" ratio="10"/>
-<attribute name="PN" x="236.22" y="162.56" size="1.778" layer="96" rot="MR0" display="off"/>
-</instance>
 <instance part="C1" gate="G$1" x="289.56" y="243.84" smashed="yes" rot="R90">
 <attribute name="NAME" x="284.48" y="245.491" size="1.9304" layer="95" font="vector" ratio="10"/>
@@
 <attribute name="NAME" x="207.01" y="195.58" size="1.9304" layer="95" font="vector" ratio="10"/>
 <attribute name="VALUE" x="213.36" y="195.58" size="1.9304" layer="96" font="vector" ratio="10"/>
-</instance>
-<instance part="Q12" gate="G1" x="210.82" y="162.56" smashed="yes" rot="MR180">
-<attribute name="NAME" x="215.9" y="166.37" size="1.9304" layer="95" font="vector" ratio="10"/>
-<attribute name="VALUE" x="215.9" y="160.02" size="1.9304" layer="96" font="vector" ratio="10"/>
-<attribute name="PN" x="210.82" y="162.56" size="1.778" layer="96" rot="MR180" display="off"/>
 </instance>
 <instance part="R3" gate="G$1" x="200.66" y="162.56" smashed="yes" rot="R270">
@@
 </instance>
 <instance part="Q16" gate="G$1" x="330.2" y="142.24"/>
+<instance part="Q1" gate="G$1" x="236.22" y="162.56" smashed="yes" rot="MR0">
+<attribute name="NAME" x="237.49" y="166.7256" size="1.9304" layer="95" font="vector" ratio="10"/>
+<attribute name="VALUE" x="237.49" y="159.1056" size="1.9304" layer="96" font="vector" ratio="10"/>
+</instance>
+<instance part="Q12" gate="G$1" x="210.82" y="162.56" smashed="yes" rot="MR180">
+<attribute name="NAME" x="214.63" y="164.1856" size="1.9304" layer="95" font="vector" ratio="10"/>
+<attribute name="VALUE" x="214.63" y="159.1056" size="1.9304" layer="96" font="vector" ratio="10"/>
+</instance>
 </instances>
 <busses>
@@
 <net name="N$15" class="0">
 <segment>
-<pinref part="Q12" gate="G1" pin="E"/>
 <wire x1="213.36" y1="167.64" x2="213.36" y2="172.72" width="0.1524" layer="91"/>
 <wire x1="213.36" y1="172.72" x2="233.68" y2="172.72" width="0.1524" layer="91"/>
-<pinref part="Q1" gate="G1" pin="C"/>
 <wire x1="233.68" y1="172.72" x2="233.68" y2="167.64" width="0.1524" layer="91"/>
 <pinref part="Q19" gate="G$1" pin="E"/>
@@
 <junction x="213.36" y="172.72"/>
 <pinref part="Q10" gate="G$1" pin="C"/>
+<pinref part="Q1" gate="G$1" pin="C"/>
+<pinref part="Q12" gate="G$1" pin="E"/>
 </segment>
 </net>
 <net name="N$17" class="0">
 <segment>
-<pinref part="Q12" gate="G1" pin="B"/>
 <pinref part="R3" gate="G$1" pin="P$1"/>
-<wire x1="205.74" y1="162.56" x2="208.28" y2="162.56" width="0.1524" layer="91"/>
+<pinref part="Q12" gate="G$1" pin="B"/>
+<wire x1="208.28" y1="162.56" x2="205.74" y2="162.56" width="0.1524" layer="91"/>
 </segment>
 </net>
 <net name="N$19" class="0">
 <segment>
-<pinref part="Q1" gate="G1" pin="B"/>
 <wire x1="238.76" y1="162.56" x2="254" y2="162.56" width="0.1524" layer="91"/>
 <wire x1="254" y1="162.56" x2="254" y2="139.7" width="0.1524" layer="91"/>
 <pinref part="R24" gate="G$1" pin="P$1"/>
 <wire x1="254" y1="139.7" x2="208.28" y2="139.7" width="0.1524" layer="91"/>
+<pinref part="Q1" gate="G$1" pin="B"/>
 </segment>
 </net>
 <net name="N$20" class="0">
 <segment>
-<pinref part="Q12" gate="G1" pin="C"/>
-<pinref part="Q1" gate="G1" pin="E"/>
 <wire x1="233.68" y1="157.48" x2="233.68" y2="152.4" width="0.1524" layer="91"/>
 <wire x1="233.68" y1="152.4" x2="213.36" y2="152.4" width="0.1524" layer="91"/>
@@
 <wire x1="289.56" y1="152.4" x2="271.78" y2="152.4" width="0.1524" layer="91"/>
 <junction x="271.78" y="152.4"/>
-</segment>
-</net>
+<pinref part="Q1" gate="G$1" pin="E"/>
+<pinref part="Q12" gate="G$1" pin="C"/>
+</segment>
+</net>

Commit message: backup
Parts:
- removed P6: 44PINEDGE, keiths:44PINEDGE
- removed Q21, Q22: 2N3906, keiths:2N3906
- added P2: 20, keiths:POT-3006P
- added Q17, Q18: 2N3904, keiths:2N3904
- C1: value 0.001uF -> 0.022 uF; device keiths:CAP0.1UF100V -> keiths:ECQ-E2223JF; MPN 1000 pf -> (none); PN (none) -> ECQ-E2223JFB
- C10: value 0.1uF -> 3.3 UF; device keiths:CAP0.1UF100V -> keiths:ECW-FD2W335K
- C11: value 3.3 UF -> 56 pF; device keiths:ECW-FD2W335K -> keiths:CAP0.1UF100V; MPN (none) -> 68 pF
- C3: value 56 pF -> 120pF; MPN 68 pF -> 1000 pf
- C4: value 0.022 uF -> 0.001uF; device keiths:ECQ-E2223JF -> keiths:CAP0.1UF100V; MPN (none) -> 1000 pf; PN ECQ-E2223JFB -> (none)
- C5: value 680pF -> 0.022 uF; device keiths:CAP0.1UF100V -> keiths:ECQ-E2223JF; MPN 1000 pf -> (none); PN (none) -> ECQ-E2223JFB
- C6: value 330pF -> 0.022uF; device keiths:CAP0.1UF100V -> keiths:ECQ-E2223JF; MPN 1000 pf -> (none); PN (none) -> ECQ-E2223JFB
- C7: value 120pF -> 680pF
- C8: value 0.022 uF -> 330pF; device keiths:ECQ-E2223JF -> keiths:CAP0.1UF100V; MPN (none) -> 1000 pf; PN ECQ-E2223JFB -> (none)
- C9: value 0.022 uF -> 0.1uF; device keiths:ECQ-E2223JF -> keiths:CAP0.1UF100V; PN ECQ-E2223JFB -> (none)
- P1: value 20 -> 44PINEDGE; device keiths:POT-3006P -> keiths:44PINEDGE
- Q1: value KSP05TA -> 2N3906; device keiths:KSP05TA -> keiths:2N3906
- Q10, Q7: value 2N3906 -> KSP05TA; device keiths:2N3906 -> keiths:KSP05TA
- Q12: value KSP05TA -> 2N3904; device keiths:KSP05TA -> keiths:2N3904; PN (none) -> 2N3904
- Q14: value 2N3906 -> 2N3904; device keiths:2N3906 -> keiths:2N3904; PN (none) -> 2N3904
- Q19: value 2N2907 -> 2N3904; device keiths:2N2907 -> keiths:2N3904; PN 2N2907A -> 2N3904
- Q2, Q3, Q6: value 2N3904 -> 2N3906; device keiths:2N3904 -> keiths:2N3906; PN 2N3904 -> (none)
- Q20: value 2N3904 -> 2N2222A; device keiths:2N3904 -> keiths:2N2222A; PN 2N3904 -> (none)
- Q4: value 2N3904 -> 2N2907; device keiths:2N3904 -> keiths:2N2907; PN 2N3904 -> 2N2907A
- Q5: value 2N2222A -> 2N3906; device keiths:2N2222A -> keiths:2N3906
- R1: value 220 -> 120
- R10: value 1 K -> 1K
- R11: value 1500 -> 27
- R12: value 470 -> 27
- R13: value 560 -> 470
- R14: value 27 -> 1.5K
- R15, R21, R4: value 120 -> 27
- R16: value 560 -> 220
- R17: value 560 -> 1.5K
- R18, R5: value 27 -> 120
- R19, R25: value 27 -> 560
- R2: value 560 -> 120
- R20: value 27 -> 330
- R22: value 1.5 K -> 1K
- R23: value 10 K -> 120
- R24, R3: value 680 -> 560
- R26: value 120 -> 1K
- R27: value 1 K -> 120
- R28: value 27 -> 1K
- R29: value 330 -> 560
- R30: value 1 K -> 10K
- R31: value 120 -> 560
- R6: value 1 K -> 27
- R7: value 560 -> 27
- R8: value 120 -> 680
- R9: value 560 -> 680
- ZD3: value (none) -> BAT43
Connections:
- removed net +10V1: Q5.C, R10.P$2, R12.P$2, R16.P$2, R19.P$2, R2.P$2, R20.P$2, R25.P$2, R5.P$2, R8.P$2, R9.P$2
- net +10V: now also P1.A, Q20.C, R12.P$2, R13.P$2, R17.P$2, R19.P$2, R2.P$2, R20.P$2, R24.P$2, R28.P$2, R4.P$2, R6.P$2, R7.P$2; no longer P6.A, R22.P$2
- net -15V: now also P1.C, Q15.E, Q18.E, Q19.E, R11.P$1, R15.P$1, R25.P$1, R3.P$1, R30.P$1, R31.P$1, R5.P$1; no longer P6.C, Q2.E, Q3.E, Q4.E, R13.P$1, R14.P$1, R17.P$1, R23.P$1, R26.P$1, R28.P$1, R7.P$1
- net E_IN: now also P1.E, R1.P$2; no longer P6.E, R31.P$2
- net GND: now also C1.1, C3.2, C5.1, C6.1, P1.D, R10.P$1; no longer C4.1, C7.2, C8.1, C9.1, P6.D, R27.P$1
- net H_IN: now also C9.1, P1.H, P2.1, R22.P$1; no longer C11.1, P1.1, P6.H, R30.P$1
- net K_IN: now also P1.K, Q11.B; no longer P6.K, Q20.B
- net N$1: now also C4.1, R16.P$1; no longer C1.1, R1.P$1
- net N$10: now also Q5.E, R6.P$1; no longer Q9.E, R20.P$1
- net N$11: now also Q19.C, Q20.B, R29.P$1, R30.P$2; no longer Q4.C, Q5.B, R16.P$1, R23.P$2
- net N$12: now also Q19.B, R27.P$2; no longer Q4.B, R15.P$2
- net N$13: now also C2.2, Q4.C, R5.P$2; no longer C4.2, Q19.C, R21.P$2
- net N$14: now also Q12.B, Q14.B, Q17.B, Q9.C; no longer Q11.B, Q15.B, Q21.C, Q6.B
- net N$15: now also Q3.C, Q4.E, Q7.E; no longer Q1.C, Q12.E, Q19.E
- net N$16: now also Q6.E, R7.P$1; no longer Q22.E, R25.P$1
- net N$17: now also Q7.B, R8.P$1; no longer Q12.B, R3.P$1
- net N$18: now also Q14.E, R18.P$2; no longer Q11.E, R26.P$2
- net N$19: now also Q10.B, R9.P$1; no longer Q1.B, R24.P$1
- net N$2: now also C7.1, C8.1, Q15.C, R19.P$1; no longer C5.1, C6.1, Q2.C, R2.P$1
- net N$20: now also C3.1, Q10.E, Q7.C; no longer C7.1, Q1.E, Q12.C
- net N$21: now also Q1.B, Q3.B, Q5.B, Q5.C, Q6.B, R10.P$2; no longer Q10.B, Q14.B, Q21.B, Q22.B, Q9.C, R27.P$2
- net N$22: now also Q14.C; no longer Q11.C
- net N$23: now also D1.A, Q6.C, R8.P$2, R9.P$2; no longer D2.A, Q22.C, R24.P$2, R3.P$2
- net N$24: now also Q9.E, R12.P$1; no longer Q21.E, R5.P$1
- net N$25: now also Q2.B, R1.P$1; no longer Q7.B, R31.P$1
- net N$26: now also Q1.E, R2.P$1; no longer Q14.E, R8.P$1
- net N$27: now also C5.2, R17.P$1; no longer C8.2, R22.P$1
- net N$28: now also Q12.E, R15.P$2; no longer Q6.E, R14.P$2
- net N$3: now also C4.2, Q15.B, R23.P$1; no longer C1.2, Q2.B, R4.P$1
- net N$30: now also Q1.C, Q2.E, Q4.B; no longer Q14.C, Q19.B, Q7.E
- net N$31: now also C1.2, Q2.C, R3.P$2; no longer C2.2, Q7.C, R13.P$2
- net N$33: now also Q3.E, R4.P$1; no longer Q10.E, R19.P$1
- net N$34: now also Q12.C, R14.P$1, R16.P$2; no longer Q6.C, R1.P$2, R11.P$1
- net N$36: now also Q17.E, R21.P$2; no longer Q15.E, R28.P$2
- net N$37: now also Q11.E, R14.P$2; no longer Q20.E, R11.P$2
- net N$38: now also Q11.C, R13.P$1; no longer Q20.C, R12.P$1
- net N$39: now also Q17.C, R22.P$2; no longer Q15.C, R30.P$2
- net N$4: now also C11.1, R23.P$2, R26.P$2, R27.P$1; no longer C3.1, R15.P$1, R4.P$2, R6.P$2
- net N$40: now also C6.2, R20.P$1; no longer C9.2, R29.P$1
- net N$5: now also C11.2, Q18.C, R26.P$1, R28.P$1; no longer C3.2, Q3.C, R10.P$1, R6.P$1
- net N$6: now also D1.C, Q20.E, R31.P$2; no longer D2.C, Q5.E, R17.P$2
- net N$7: now also R11.P$2; no longer R18.P$2
- net N$8: now also D2.C, Q18.B; no longer D1.C, Q3.B
- net N$9: now also C7.2, C8.2, D2.A, R24.P$1, R25.P$2; no longer C5.2, C6.2, D1.A, R7.P$2, R9.P$1
- net Z_OUT: now also C9.2, P1.Z, P2.2, P2.3; no longer C11.2, P1.2, P1.3, P6.Z
Other:
- moved on the sheet: C1, C10, C11, C2, C3, C4, C5, C6, C7, C8, C9, D1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

Commit message: new .brd files
Parts:
- added U$1, U$2: FIDUCIAL, adafruit:FIDUCIAL
- C1: value 0.022 uF -> 0.022uF
- C11: value 56 pF -> 56pF
Changed lines of the file:
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@@
 <part name="R2" library="keiths" deviceset="AXIALRESISTOR" device="QUARTER_WATT" value="120"/>
 <part name="R3" library="keiths" deviceset="AXIALRESISTOR" device="QUARTER_WATT" value="560"/>
-<part name="C1" library="keiths" deviceset="ECQ-E2223JF" device="" value="0.022 uF">
+<part name="C1" library="keiths" deviceset="ECQ-E2223JF" device="" value="0.022uF">
 <attribute name="PN" value="ECQ-E2223JFB"/>
 </part>
@@
 <part name="R23" library="keiths" deviceset="AXIALRESISTOR" device="QUARTER_WATT" value="120"/>
 <part name="R26" library="keiths" deviceset="AXIALRESISTOR" device="QUARTER_WATT" value="1K"/>
-<part name="C11" library="keiths" deviceset="CAP0.1UF100V" device="" value="56 pF">
+<part name="C11" library="keiths" deviceset="CAP0.1UF100V" device="" value="56pF">
 <attribute name="MPN" value="68 pF"/>
 </part>
@@
 <part name="Q10" library="keiths" deviceset="KSP05TA" device=""/>
 <part name="Q7" library="keiths" deviceset="KSP05TA" device=""/>
+<part name="U$1" library="adafruit" deviceset="FIDUCIAL" device=""/>
+<part name="U$2" library="adafruit" deviceset="FIDUCIAL" device=""/>
 </parts>
 <sheets>
@@
 <attribute name="VALUE" x="214.63" y="159.1056" size="1.9304" layer="96" font="vector" ratio="10"/>
 </instance>
+<instance part="U$1" gate="G$1" x="25.4" y="411.48"/>
+<instance part="U$2" gate="G$1" x="40.64" y="411.48"/>
 </instances>
 <busses>

Commit message: preamplifier card being routed
Parts:
- removed C11: 56pF, keiths:CAP0.1UF100V
- removed Q19: 2N3904, keiths:2N3904
- removed Q20: 2N2222A, keiths:2N2222A
- removed R30: 10K, keiths:AXIALRESISTORQUARTER_WATT
- removed R31: 560, keiths:AXIALRESISTORQUARTER_WATT
- added C100: 120pF, keiths:CAP0.1UF100V
- added Q100, Q101: KSP05TA, keiths:KSP05TA
- added R100, R101: 680, keiths:AXIALRESISTORQUARTER_WATT
- C1: value 0.022uF -> 0.1uF; device keiths:ECQ-E2223JF -> keiths:CAP0.1UF100V; PN ECQ-E2223JFB -> (none)
- C10: value 3.3 UF -> 56pF; device keiths:ECW-FD2W335K -> keiths:CAP0.1UF100V; MPN (none) -> 68 pF
- C2: value 0.022 uF -> 3.3 UF; device keiths:ECQ-E2223JF -> keiths:ECW-FD2W335K; PN ECQ-E2223JFB -> (none)
- C3: value 120pF -> 680pF
- C4: value 0.001uF -> 330pF
- C5: value 0.022 uF -> 0.022uF
- C6: value 0.022uF -> 0.022 uF
- C7: value 680pF -> 0.022 uF; device keiths:CAP0.1UF100V -> keiths:ECQ-E2223JF; MPN 1000 pf -> (none); PN (none) -> ECQ-E2223JFB
- C8: value 330pF -> 0.022uF; device keiths:CAP0.1UF100V -> keiths:ECQ-E2223JF; MPN 1000 pf -> (none); PN (none) -> ECQ-E2223JFB
- C9: value 0.1uF -> 0.001uF; MPN (none) -> 1000 pf
- P1: value 44PINEDGE -> 20; device keiths:44PINEDGE -> keiths:POT-3006P
- P2: value 20 -> 44PINEDGE; device keiths:POT-3006P -> keiths:44PINEDGE
- Q10: value KSP05TA -> 2N3904; device keiths:KSP05TA -> keiths:2N3904; PN (none) -> 2N3904
- Q15: value 2N3904 -> 2N2222A; device keiths:2N3904 -> keiths:2N2222A; PN 2N3904 -> (none)
- Q16: value 2N2222A -> 2N3904; device keiths:2N2222A -> keiths:2N3904; PN (none) -> 2N3904
- Q4: value 2N2907 -> 2N3906; device keiths:2N2907 -> keiths:2N3906; PN 2N2907A -> (none)
- Q5: value 2N3906 -> 2N3904; device keiths:2N3906 -> keiths:2N3904; PN (none) -> 2N3904
- Q7: value KSP05TA -> 2N2907; device keiths:KSP05TA -> keiths:2N2907; PN (none) -> 2N2907A
- Q8: value 2N3904 -> 2N3906; device keiths:2N3904 -> keiths:2N3906; PN 2N3904 -> (none)
- Q9: value 2N3906 -> 2N2222A; device keiths:2N3906 -> keiths:2N2222A
- R10, R22: value 1K -> 120
- R11, R7: value 27 -> 560
- R12: value 27 -> 1.5K
- R13: value 470 -> 560
- R14: value 1.5K -> 120
- R15: value 27 -> 220
- R16: value 220 -> 1K
- R17: value 1.5K -> 27
- R18: value 120 -> 1.5K
- R19: value 560 -> 330
- R2, R5: value 120 -> 27
- R20: value 330 -> 27
- R21: value 27 -> 10K
- R23: value 120 -> 1K
- R24: value 560 -> 120
- R25: value 560 -> 1K
- R26: value 1K -> 27
- R28: value 1K -> 560
- R3: value 560 -> 27
- R6: value 27 -> 470
- R8: value 680 -> 560
- R9: value 680 -> 1K
- ZD2: PN BAT43 -> (none)
- ZD3: PN (none) -> BAT43
Connections:
- removed net N$16 (its old number): Q6.E, R7.P$1
- new net N$26: Q6.E, R1.P$1
- net +10V: now also P2.A, Q9.C, R1.P$2, R11.P$2, R18.P$2, R23.P$2, R3.P$2, R5.P$2, R8.P$2; no longer P1.A, Q20.C, R12.P$2, R13.P$2, R17.P$2, R20.P$2, R24.P$2, R28.P$2, R29.P$2
- net -15V: now also P2.C, Q12.E, Q14.E, R13.P$1, R14.P$1, R17.P$1, R20.P$1, R26.P$1, R27.P$1, R28.P$1, R29.P$1; no longer P1.C, Q15.E, Q19.E, R11.P$1, R15.P$1, R18.P$1, R25.P$1, R3.P$1, R30.P$1, R31.P$1, R5.P$1
- net E_IN: now also P2.E, R10.P$2; no longer P1.E, R1.P$2
- net GND: now also C100.2, C7.1, C8.1, P2.D, R9.P$1; no longer C1.1, C2.1, C3.2, P1.D, R10.P$1
- net H_IN: now also C1.1, C2.1, P1.1, P2.H, R16.P$1; no longer C10.1, C9.1, P1.H, P2.1, R22.P$1
- net K_IN: now also P2.K, Q5.B; no longer P1.K, Q11.B
- net N$1: now also C9.1, R15.P$1; no longer C4.1, R16.P$1
- net N$10: now also Q4.E, R5.P$1; no longer Q5.E, R6.P$1
- net N$11: now also Q14.C, Q9.B, R11.P$1, R21.P$2, ZD2.C; no longer Q19.C, Q20.B, R29.P$1, R30.P$2, ZD3.C
- net N$12: now also Q14.B, R24.P$2, ZD2.A; no longer Q19.B, R27.P$2, ZD3.A
- net N$13: now also C6.2, Q7.C, R14.P$2; no longer C2.2, Q4.C, R5.P$2
- net N$14: now also Q10.B, Q10.C, Q11.B, Q16.B, Q2.C; no longer Q12.B, Q14.B, Q8.B, Q8.C, Q9.C
- net N$15: now also Q1.C, Q100.E, Q101.C; no longer Q10.C, Q3.C, Q4.E
- net N$17: now also Q100.B, R100.P$1; no longer Q7.B, R8.P$1
- net N$18: now also Q17.E, R27.P$2; no longer Q14.E, R18.P$2
- net N$19: now also Q101.B, R101.P$1; no longer Q10.B, R9.P$1
- net N$2: now also C3.1, C4.1, Q12.C, R7.P$1; no longer C7.1, C8.1, Q15.C, R19.P$1
- net N$20: now also C100.1, Q100.C, Q101.E; no longer C3.1, Q10.E, Q7.C
- net N$21: now also Q2.B, Q4.B, Q4.C, R9.P$2; no longer Q5.B, Q5.C, Q9.B, R10.P$2
- net N$22: now also Q15.B, Q17.C; no longer Q14.C, Q16.B
- net N$23: now also Q3.C, R100.P$2, R101.P$2; no longer Q6.C, R8.P$2, R9.P$2
- net N$24: now also Q2.E, R3.P$1; no longer Q9.E, R12.P$1
- net N$25: now also Q8.B, R10.P$1; no longer Q2.B, R1.P$1
- net N$27: now also C7.2, R18.P$1; no longer C5.2, R17.P$1
- net N$28: now also Q11.E, R17.P$2; no longer Q12.E, R15.P$2
- net N$3: now also C9.2, Q12.B, R22.P$1; no longer C4.2, Q15.B, R23.P$1
- net N$30: now also Q6.C, Q7.B, Q8.E; no longer Q1.C, Q2.E, Q4.B
- net N$31: now also C5.2, Q8.C, R13.P$2; no longer C1.2, Q2.C, R3.P$2
- net N$34: now also Q11.C, R12.P$1, R15.P$2; no longer Q12.C, R14.P$1, R16.P$2
- net N$36: now also Q16.E, R26.P$2; no longer Q17.E, R21.P$2
- net N$37: now also Q5.E, R12.P$2; no longer Q11.E, R14.P$2
- net N$38: now also Q5.C, R6.P$1; no longer Q11.C, R13.P$1
- net N$39: now also Q15.E, Q16.C, R16.P$2; no longer Q16.E, Q17.C, R22.P$2
- net N$4: now also C10.1, R22.P$2, R24.P$1, R25.P$2; no longer C11.1, R23.P$2, R26.P$2, R27.P$1
- net N$40: now also C8.2, Q15.C, R19.P$1; no longer C6.2, Q16.C, R20.P$1
- net N$5: now also C10.2, R23.P$1, R25.P$1, ZD3.C; no longer C11.2, R26.P$1, R28.P$1, ZD2.C
- net N$6: now also Q9.E, R29.P$2; no longer Q20.E, R31.P$2
- net N$7: now also Q10.E, R20.P$2; no longer Q8.E, R11.P$2
- net N$8: now also ZD3.A; no longer ZD2.A
- net N$9: now also C3.2, C4.2, R28.P$2, R8.P$1; no longer C7.2, C8.2, R24.P$1, R25.P$2
- net Z_OUT: now also C1.2, C2.2, P1.2, P1.3, P2.Z; no longer C10.2, C9.2, P1.Z, P2.2, P2.3
Other:
- moved on the sheet: C1, C10, C2, C3, C4, C5, C6, C7, C8, C9, Q1, Q11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
