File: yoke/mimic1575.sch (EAGLE design)
At the start: 71 parts, among them P1 20, P2 44PINEDGE, Q1 2N3906, Q10 2N3904, Q100 KSP05TA, Q101 KSP05TA, Q11 2N3904, Q12 2N3904, Q13 2N3904, Q14 2N3904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

Commit message: revised artwork
Parts:
- removed ZD1: BAT43, keiths:1N754A
- added D4: 1N4148, keiths:1N4148
- D1: value 1N4148 -> BAT43; device keiths:1N4148 -> keiths:1N754A; PN (none) -> BAT43
- P2: value 44PINEDGE -> 44PINEDGE-M; device keiths:44PINEDGE -> keiths:44PINEDGE-M
- R24: value 120 -> 1K
- R25: value 1K -> 120
- renumbered ZD2 to D3, ZD3 to D5
Connections:
- net -15V: now also P2.3
- net GND: now also P2.4
- net N$12: now also R25.P$2; no longer R24.P$2
- net N$2: now also D1.C; no longer ZD1.C
- net N$23: now also D2.A; no longer D1.A
- net N$3: now also D1.A; no longer ZD1.A
- net N$4: now also R24.P$2, R25.P$1; no longer R24.P$1, R25.P$2
- net N$5: now also R24.P$1; no longer R25.P$1
- net N$6: now also D2.C; no longer D1.C
- net N$8: now also D4.C; no longer D2.C
- net N$9: now also D4.A; no longer D2.A
Other:
- note added: "X_Y Follow Hold"
- moved on the sheet: D2, P2, R24, R25
