File: yoke/mimic1579.sch (EAGLE design)
At the start: 75 parts, among them P1 44PINEDGE, P2 2K, P3 2K, Q1 2N3904, Q13 2N3904, Q14 2N3904, Q15 2N3906, Q16 2N3904, Q2 2N3906, Q3 2N3906, Q4 2N3906, Q5 2N3904, Q6 2N3904, Q7 2N3906, Q8 2N3904, Q9 2N3904

Commit message: update netlist
Connections:
- new net +10V: P1.A
- new net +5V: P1.B
- net -10V: now also P1.E
- net -15V: now also P1.C
- net F_IN: now also P1.F
- net GND: now also P1.D
- net H_OUT: now also P1.H
- net J_IN: now also P1.J
- net K_IN: now also P1.K
- net L_IN: now also P1.L
- net P_OUT: now also P1.P
- net U_IN: now also P1.U
Other:
- moved on the sheet: P1
Changed lines of the file:
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@@
 </classes>
 <parts>
-<part name="P1" library="keiths" deviceset="44PINEDGE" device=""/>
 <part name="Q5" library="keiths" deviceset="2N3904" device=""/>
 <part name="R2" library="keiths" deviceset="R-1/4WATT" device="" value="4.7K"/>
@@
 <part name="SUPPLY19" library="keiths" deviceset="+5V" device=""/>
 <part name="FRAME1" library="frames" deviceset="FRAME_C_L" device=""/>
+<part name="P1" library="keiths" deviceset="44PINEDGE" device=""/>
 </parts>
 <sheets>
@@
 </plain>
 <instances>
-<instance part="P1" gate="G$1" x="134.62" y="220.98"/>
 <instance part="Q5" gate="G1" x="330.2" y="332.74"/>
 <instance part="R2" gate="&gt;NAME" x="322.58" y="342.9" smashed="yes" rot="MR90">
@@
 <instance part="FRAME1" gate="G$1" x="0" y="0"/>
 <instance part="FRAME1" gate="G$2" x="452.12" y="0"/>
+<instance part="P1" gate="G$1" x="93.98" y="187.96"/>
 </instances>
 <busses>
@@
 </segment>
 <segment>
-<label x="78.74" y="233.68" size="1.9304" layer="95" rot="R180" xref="yes"/>
-<wire x1="83.82" y1="233.68" x2="78.74" y2="233.68" width="0.1524" layer="91"/>
+<label x="111.76" y="200.66" size="1.9304" layer="95" font="vector" ratio="10" xref="yes"/>
+<pinref part="P1" gate="G$1" pin="F"/>
+<wire x1="104.14" y1="200.66" x2="111.76" y2="200.66" width="0.1524" layer="91"/>
 </segment>
 </net>
@@
 </segment>
 <segment>
-<wire x1="106.68" y1="210.82" x2="101.6" y2="210.82" width="0.1524" layer="91"/>
-<label x="101.6" y="210.82" size="1.9304" layer="95" font="vector" ratio="10" rot="MR0" xref="yes"/>
+<pinref part="P1" gate="G$1" pin="D"/>
+<wire x1="104.14" y1="205.74" x2="111.76" y2="205.74" width="0.1524" layer="91"/>
+<label x="111.76" y="205.74" size="1.9304" layer="95" font="vector" ratio="10" xref="yes"/>
 </segment>
 </net>
@@
 </segment>
 <segment>
-<wire x1="83.82" y1="251.46" x2="91.44" y2="251.46" width="0.1524" layer="91"/>
-<label x="91.44" y="251.46" size="1.9304" layer="95" font="vector" ratio="10" xref="yes"/>
+<wire x1="104.14" y1="182.88" x2="132.08" y2="182.88" width="0.1524" layer="91"/>
+<label x="132.08" y="182.88" size="1.9304" layer="95" font="vector" ratio="10" xref="yes"/>
+<pinref part="P1" gate="G$1" pin="P"/>
 </segment>
 </net>
@@
 </segment>
 <segment>
-<wire x1="91.44" y1="261.62" x2="86.36" y2="261.62" width="0.1524" layer="91"/>
-<label x="91.44" y="261.62" size="1.9304" layer="95" font="vector" ratio="10" xref="yes"/>
+<label x="132.08" y="198.12" size="1.9304" layer="95" font="vector" ratio="10" xref="yes"/>
+<pinref part="P1" gate="G$1" pin="H"/>
+<wire x1="104.14" y1="198.12" x2="132.08" y2="198.12" width="0.1524" layer="91"/>
 </segment>
 </net>
@@
 </segment>
 <segment>
-<label x="101.6" y="231.14" size="1.9304" layer="95" font="vector" ratio="10" rot="MR0" xref="yes"/>
-<wire x1="106.68" y1="231.14" x2="101.6" y2="231.14" width="0.1524" layer="91"/>
+<label x="132.08" y="203.2" size="1.9304" layer="95" font="vector" ratio="10" rot="MR180" xref="yes"/>
+<pinref part="P1" gate="G$1" pin="E"/>
+<wire x1="104.14" y1="203.2" x2="132.08" y2="203.2" width="0.1524" layer="91"/>
 </segment>
 </net>
@@
 </segment>
 <segment>
-<label x="101.6" y="193.04" size="1.9304" layer="95" font="vector" ratio="10" rot="MR0" xref="yes"/>
-<wire x1="101.6" y1="193.04" x2="106.68" y2="193.04" width="0.1524" layer="91"/>
+<label x="111.76" y="195.58" size="1.9304" layer="95" font="vector" ratio="10" rot="MR180" xref="yes"/>
+<wire x1="111.76" y1="195.58" x2="104.14" y2="195.58" width="0.1524" layer="91"/>
+<pinref part="P1" gate="G$1" pin="J"/>
 </segment>
 </net>
@@
 </segment>
 <segment>
-<label x="101.6" y="175.26" size="1.9304" layer="95" font="vector" ratio="10" rot="MR0" xref="yes"/>
-<wire x1="101.6" y1="175.26" x2="106.68" y2="175.26" width="0.1524" layer="91"/>
+<label x="111.76" y="190.5" size="1.9304" layer="95" font="vector" ratio="10" rot="MR180" xref="yes"/>
+<wire x1="111.76" y1="190.5" x2="104.14" y2="190.5" width="0.1524" layer="91"/>
+<pinref part="P1" gate="G$1" pin="L"/>
 </segment>
 </net>
@@
 </segment>
 <segment>
-<label x="78.74" y="241.3" size="1.9304" layer="95" rot="MR0" xref="yes"/>
-<wire x1="83.82" y1="241.3" x2="78.74" y2="241.3" width="0.1524" layer="91"/>
+<label x="132.08" y="172.72" size="1.9304" layer="95" font="vector" ratio="10" rot="MR180" xref="yes"/>
+<wire x1="104.14" y1="172.72" x2="132.08" y2="172.72" width="0.1524" layer="91"/>
+<pinref part="P1" gate="G$1" pin="U"/>
 </segment>
 </net>
@@
 </segment>
 <segment>
-<label x="101.6" y="200.66" size="1.9304" layer="95" font="vector" ratio="10" rot="MR0" xref="yes"/>
-<wire x1="106.68" y1="200.66" x2="101.6" y2="200.66" width="0.1524" layer="91"/>
+<pinref part="P1" gate="G$1" pin="C"/>
+<wire x1="104.14" y1="208.28" x2="132.08" y2="208.28" width="0.1524" layer="91"/>
+<label x="132.08" y="208.28" size="1.9304" layer="95" font="vector" ratio="10" xref="yes"/>
 </segment>
 </net>
@@
 </segment>
 <segment>
-<wire x1="101.6" y1="185.42" x2="106.68" y2="185.42" width="0.1524" layer="91"/>
-<label x="101.6" y="185.42" size="1.9304" layer="95" font="vector" ratio="10" rot="MR0" xref="yes"/>
+<wire x1="132.08" y1="193.04" x2="104.14" y2="193.04" width="0.1524" layer="91"/>
+<label x="132.08" y="193.04" size="1.9304" layer="95" font="vector" ratio="10" rot="MR180" xref="yes"/>
+<pinref part="P1" gate="G$1" pin="K"/>
 </segment>
 </net>
@@
 </segment>
 <segment>
-<wire x1="106.68" y1="220.98" x2="101.6" y2="220.98" width="0.1524" layer="91"/>
-<label x="101.6" y="220.98" size="1.9304" layer="95" rot="R180" xref="yes"/>
-</segment>
-</net>
+<label x="111.76" y="210.82" size="1.9304" layer="95" font="vector" ratio="10" xref="yes"/>
+<pinref part="P1" gate="G$1" pin="B"/>
+<wire x1="104.14" y1="210.82" x2="111.76" y2="210.82" width="0.1524" layer="91"/>
+</segment>
+</net>
+<net name="+10V" class="0">
+<segment>
+<pinref part="P1" gate="G$1" pin="A"/>
+<wire x1="104.14" y1="213.36" x2="132.08" y2="213.36" width="0.1524" layer="91"/>
+<label x="132.08" y="213.36" size="1.9304" layer="95" font="vector" ratio="10" xref="yes"/>
+</segment>
+</net>

Commit message: update netlist
Other:
- moved on the sheet: P1
Changed lines of the file:
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@@
 <instance part="FRAME1" gate="G$1" x="0" y="0"/>
 <instance part="FRAME1" gate="G$2" x="452.12" y="0"/>
-<instance part="P1" gate="G$1" x="93.98" y="187.96"/>
+<instance part="P1" gate="G$1" x="96.52" y="215.9"/>
 </instances>
 <busses>
@@
 </segment>
 <segment>
-<label x="111.76" y="200.66" size="1.9304" layer="95" font="vector" ratio="10" xref="yes"/>
+<label x="114.3" y="228.6" size="1.9304" layer="95" font="vector" ratio="10" xref="yes"/>
 <pinref part="P1" gate="G$1" pin="F"/>
-<wire x1="104.14" y1="200.66" x2="111.76" y2="200.66" width="0.1524" layer="91"/>
+<wire x1="106.68" y1="228.6" x2="114.3" y2="228.6" width="0.1524" layer="91"/>
 </segment>
 </net>
@@
 <segment>
 <pinref part="P1" gate="G$1" pin="D"/>
-<wire x1="104.14" y1="205.74" x2="111.76" y2="205.74" width="0.1524" layer="91"/>
-<label x="111.76" y="205.74" size="1.9304" layer="95" font="vector" ratio="10" xref="yes"/>
+<wire x1="106.68" y1="233.68" x2="114.3" y2="233.68" width="0.1524" layer="91"/>
+<label x="114.3" y="233.68" size="1.9304" layer="95" font="vector" ratio="10" xref="yes"/>
 </segment>
 </net>
@@
 </segment>
 <segment>
-<wire x1="104.14" y1="182.88" x2="132.08" y2="182.88" width="0.1524" layer="91"/>
-<label x="132.08" y="182.88" size="1.9304" layer="95" font="vector" ratio="10" xref="yes"/>
+<wire x1="106.68" y1="210.82" x2="134.62" y2="210.82" width="0.1524" layer="91"/>
+<label x="134.62" y="210.82" size="1.9304" layer="95" font="vector" ratio="10" xref="yes"/>
 <pinref part="P1" gate="G$1" pin="P"/>
 </segment>
@@
 </segment>
 <segment>
-<label x="132.08" y="198.12" size="1.9304" layer="95" font="vector" ratio="10" xref="yes"/>
+<label x="134.62" y="226.06" size="1.9304" layer="95" font="vector" ratio="10" xref="yes"/>
 <pinref part="P1" gate="G$1" pin="H"/>
-<wire x1="104.14" y1="198.12" x2="132.08" y2="198.12" width="0.1524" layer="91"/>
+<wire x1="106.68" y1="226.06" x2="134.62" y2="226.06" width="0.1524" layer="91"/>
 </segment>
 </net>
@@
 </segment>
 <segment>
-<label x="132.08" y="203.2" size="1.9304" layer="95" font="vector" ratio="10" rot="MR180" xref="yes"/>
+<label x="134.62" y="231.14" size="1.9304" layer="95" font="vector" ratio="10" rot="MR180" xref="yes"/>
 <pinref part="P1" gate="G$1" pin="E"/>
-<wire x1="104.14" y1="203.2" x2="132.08" y2="203.2" width="0.1524" layer="91"/>
+<wire x1="106.68" y1="231.14" x2="134.62" y2="231.14" width="0.1524" layer="91"/>
 </segment>
 </net>
@@
 </segment>
 <segment>
-<label x="111.76" y="195.58" size="1.9304" layer="95" font="vector" ratio="10" rot="MR180" xref="yes"/>
-<wire x1="111.76" y1="195.58" x2="104.14" y2="195.58" width="0.1524" layer="91"/>
+<label x="114.3" y="223.52" size="1.9304" layer="95" font="vector" ratio="10" rot="MR180" xref="yes"/>
+<wire x1="114.3" y1="223.52" x2="106.68" y2="223.52" width="0.1524" layer="91"/>
 <pinref part="P1" gate="G$1" pin="J"/>
 </segment>
@@
 </segment>
 <segment>
-<label x="111.76" y="190.5" size="1.9304" layer="95" font="vector" ratio="10" rot="MR180" xref="yes"/>
-<wire x1="111.76" y1="190.5" x2="104.14" y2="190.5" width="0.1524" layer="91"/>
+<label x="114.3" y="218.44" size="1.9304" layer="95" font="vector" ratio="10" rot="MR180" xref="yes"/>
+<wire x1="114.3" y1="218.44" x2="106.68" y2="218.44" width="0.1524" layer="91"/>
 <pinref part="P1" gate="G$1" pin="L"/>
 </segment>
@@
 </segment>
 <segment>
-<label x="132.08" y="172.72" size="1.9304" layer="95" font="vector" ratio="10" rot="MR180" xref="yes"/>
-<wire x1="104.14" y1="172.72" x2="132.08" y2="172.72" width="0.1524" layer="91"/>
+<label x="134.62" y="200.66" size="1.9304" layer="95" font="vector" ratio="10" rot="MR180" xref="yes"/>
+<wire x1="106.68" y1="200.66" x2="134.62" y2="200.66" width="0.1524" layer="91"/>
 <pinref part="P1" gate="G$1" pin="U"/>
 </segment>
@@
 <segment>
 <pinref part="P1" gate="G$1" pin="C"/>
-<wire x1="104.14" y1="208.28" x2="132.08" y2="208.28" width="0.1524" layer="91"/>
-<label x="132.08" y="208.28" size="1.9304" layer="95" font="vector" ratio="10" xref="yes"/>
+<wire x1="106.68" y1="236.22" x2="134.62" y2="236.22" width="0.1524" layer="91"/>
+<label x="134.62" y="236.22" size="1.9304" layer="95" font="vector" ratio="10" xref="yes"/>
 </segment>
 </net>
@@
 </segment>
 <segment>
-<wire x1="132.08" y1="193.04" x2="104.14" y2="193.04" width="0.1524" layer="91"/>
-<label x="132.08" y="193.04" size="1.9304" layer="95" font="vector" ratio="10" rot="MR180" xref="yes"/>
+<wire x1="134.62" y1="220.98" x2="106.68" y2="220.98" width="0.1524" layer="91"/>
+<label x="134.62" y="220.98" size="1.9304" layer="95" font="vector" ratio="10" rot="MR180" xref="yes"/>
 <pinref part="P1" gate="G$1" pin="K"/>
 </segment>
@@
 </segment>
 <segment>
-<label x="111.76" y="210.82" size="1.9304" layer="95" font="vector" ratio="10" xref="yes"/>
+<label x="114.3" y="238.76" size="1.9304" layer="95" font="vector" ratio="10" xref="yes"/>
 <pinref part="P1" gate="G$1" pin="B"/>
-<wire x1="104.14" y1="210.82" x2="111.76" y2="210.82" width="0.1524" layer="91"/>
+<wire x1="106.68" y1="238.76" x2="114.3" y2="238.76" width="0.1524" layer="91"/>
 </segment>
 </net>
@@
 <segment>
 <pinref part="P1" gate="G$1" pin="A"/>
-<wire x1="104.14" y1="213.36" x2="132.08" y2="213.36" width="0.1524" layer="91"/>
-<label x="132.08" y="213.36" size="1.9304" layer="95" font="vector" ratio="10" xref="yes"/>
-</segment>
-</net>
+<wire x1="106.68" y1="241.3" x2="134.62" y2="241.3" width="0.1524" layer="91"/>
+<label x="134.62" y="241.3" size="1.9304" layer="95" font="vector" ratio="10" xref="yes"/>
+</segment>
+</net>

Commit message: new .brd files
Parts:
- removed C6: 80pF, keiths:CAP1000PF
- removed P1: 44PINEDGE, keiths:44PINEDGE
- added C5: 80pF, keiths:CAP80PF
- added J1: 44PINEDGE, keiths:44PINEDGE
- added U$1, U$2: FIDUCIAL, adafruit:FIDUCIAL
- C1, C2, C3, C4: device keiths:CAP1000PF -> keiths:CAP80PF; PN FA28X7R2A102KNU06 -> (none)
Connections:
- removed net +10V: P1.A
- removed net +5V: P1.B
- net -10V: now also J1.E; no longer P1.E
- net -15V: now also J1.C, P2.1, P2.2, P3.1, P3.2; no longer P1.C, P2.A, P2.S, P3.A, P3.S
- net F_IN: now also C5.1, J1.F; no longer C1.1, P1.F
- net GND: now also J1.D; no longer P1.D
- net H_OUT: now also J1.H; no longer P1.H
- net J_IN: now also C2.1, J1.J; no longer C6.1, P1.J
- net K_IN: now also J1.K; no longer P1.K
- net L_IN: now also J1.L; no longer P1.L
- net N$1: now also C5.2; no longer C1.2
- net N$14: now also C1.2; no longer C2.2
- net N$16: now also P3.3; no longer P3.E
- net N$30: now also C2.2; no longer C6.2
- net N$4: now also P2.3; no longer P2.E
- net P_OUT: now also J1.P; no longer P1.P
- net U_IN: now also C1.1, J1.U; no longer C2.1, P1.U
Other:
- moved on the sheet: C1, C2

Commit message: preamplifier card being routed
Parts:
- removed D25: 1N4148, keiths:1N4148
- removed P3: 2K, keiths:POT-3006P
- removed Q14, Q16: 2N3904, keiths:2N3904
- removed Q15: 2N3906, keiths:2N3906
- added D19: 1N4148, keiths:1N4148
- added P1: 2K, keiths:POT-3006P
- added Q10, Q12: 2N3906, keiths:2N3906
- added Q11: 2N3904, keiths:2N3904
- D11, D3: value BAT48 -> 1N4148; PN BAT48RL -> (none)
- D17, D2: value 1N4148 -> BAT48; PN (none) -> BAT48RL
- Q2, Q3, Q7: value 2N3906 -> 2N3904; device keiths:2N3906 -> keiths:2N3904
- Q6, Q8: value 2N3904 -> 2N3906; device keiths:2N3904 -> keiths:2N3906
- R1: value 4.75K -> 4.7K
- R10: value 1.5K -> 10K
- R11: value 4.75K -> 10K
- R12: value 4.7K -> 475
- R13, R26: value 475 -> 4.75K
- R14: value 18K -> 475
- R16, R20, R9: value 1.5K -> 475
- R19: value 1.5K -> 4.75K
- R21, R28: value 475 -> 10K
- R22: value 475 -> 1K
- R23: value 10K -> 1K
- R24, R32: value 4.75K -> 475
- R25, R5: value 10K -> 1.5K
- R3: value 4.75K -> 1.5K
- R30, R33: value 475 -> 1.5K
- R31: value 10K -> 4.75K
- R35: value 18K -> 1.5K
- R6: value 1.5K -> 18K
- R7: value 1K -> 18K
- R8: value 1K -> 4.75K
Connections:
- net -10V: now also D17.A, D2.A; no longer D11.A, D3.A
- net -15V: now also P1.1, P1.2, Q11.E, Q3.E, Q5.E, Q7.E, R11.P$2, R15.P$1, R21.P$1, R23.P$2, R25.P$2, R28.P$1, R3.P$2, R30.P$2, R33.P$2, R35.P$2; no longer P3.1, P3.2, Q14.E, Q16.E, Q6.E, Q8.E, R14.P$2, R15.P$2, R16.P$2, R19.P$2, R20.P$2, R23.P$1, R25.P$1, R31.P$1, R8.P$2, R9.P$2
- net F_IN: now also C1.1, R8.P$1; no longer C5.1, R3.P$1
- net GND: now also Q10.E, Q12.E, Q6.E, Q8.E, R7.P$2; no longer Q15.E, Q2.E, Q3.E, Q7.E, R35.P$2
- net H_OUT: now also Q1.C; no longer Q5.C
- net J_IN: now also R13.P$1; no longer R32.P$1
- net K_IN: now also R19.P$1; no longer R1.P$1
- net L_IN: now also R26.P$1; no longer R24.P$1
- net N$1: now also C1.2, Q4.B, R12.P$1; no longer C5.2, Q2.B, R21.P$1
- net N$10: now also D11.C, D12.C, R22.P$1; no longer D6.C, D9.C, R7.P$1
- net N$11: now also D18.C, D19.C, R33.P$1, R35.P$1; no longer D15.C, D8.C, R10.P$1, R9.P$1
- net N$12: now also D10.C, R20.P$1, R24.P$2; no longer D2.C, R13.P$2, R22.P$1
- net N$13: now also Q10.B, R29.P$1; no longer Q7.B, R28.P$1
- net N$14: now also C5.2, Q12.B, R34.P$1; no longer C1.2, Q3.B, R27.P$1
- net N$15: now also R31.P$2, R32.P$2; no longer R11.P$2, R29.P$2
- net N$16: now also P2.3, Q2.B, R2.P$2; no longer P3.3, Q1.B, R12.P$2
- net N$17: now also D15.A, D4.A, D9.A, Q2.E, R6.P$1; no longer D12.A, D14.A, D16.A, Q1.E, R14.P$1
- net N$18: now also D4.C, D6.C, R11.P$1; no longer D12.C, D7.C, R15.P$1
- net N$19: now also D8.C, D9.C; no longer D14.C, D17.C
- net N$2: now also Q5.C, R8.P$2, R9.P$2; no longer Q14.C, R26.P$2, R3.P$2
- net N$21: now also D14.C, D15.C, R25.P$1, R30.P$1; no longer D16.C, D18.C, R19.P$1, R20.P$1
- net N$22: now also Q11.C, R26.P$2, R27.P$2; no longer Q9.C, R24.P$2, R30.P$2
- net N$23: now also R27.P$1, R29.P$2; no longer R28.P$2, R30.P$1
- net N$25: now also D16.C, R32.P$1, R34.P$2; no longer D1.C, R27.P$2, R29.P$1
- net N$3: now also Q8.B, R24.P$1; no longer Q4.B, R13.P$1
- net N$30: now also Q6.B, R16.P$1; no longer Q15.B, R33.P$1
- net N$31: now also Q7.C, R13.P$2, R14.P$2; no longer Q8.C, R32.P$2, R34.P$2
- net N$32: now also D7.C, R14.P$1, R16.P$2; no longer D10.C, R33.P$2, R34.P$1
- net N$33: now also Q11.B, Q3.B, Q3.C, Q5.B, Q7.B, R7.P$1; no longer Q14.B, Q16.B, Q16.C, Q6.B, Q8.B, R35.P$1
- net N$4: now also P1.3, Q1.B, R1.P$2; no longer P2.3, Q5.B, R2.P$2
- net N$5: now also D12.A, D19.A, D3.A, Q1.E; no longer D4.A, D6.A, D8.A, Q5.E
- net N$6: now also D3.C, R10.P$1; no longer D4.C, R5.P$1
- net N$7: now also R22.P$2, R23.P$1; no longer R7.P$2, R8.P$1
- net N$8: now also Q9.C, R19.P$2, R20.P$2; no longer Q6.C, R1.P$2, R22.P$2
- net N$9: now also D1.C, R12.P$2, R9.P$1; no longer D25.C, R21.P$2, R26.P$1
- net P_OUT: now also Q2.C; no longer Q1.C
- net U_IN: now also C5.1, R31.P$1; no longer C1.1, R11.P$1
- net VREF: now also D1.A, D2.C, Q4.C, R1.P$1, R3.P$1; no longer D25.A, D3.C, Q2.C, R2.P$1, R6.P$1
- net VREF1: now also D10.A, D11.A, D8.A, Q8.C, R21.P$2; no longer D17.A, D2.A, D9.A, Q4.C, R23.P$2
- net VREF2: now also D14.A, Q10.C, R28.P$2; no longer D15.A, Q7.C, R31.P$2
- net VREF3: now also D6.A, Q6.C, R15.P$2; no longer D10.A, Q15.C, R25.P$2
- net VREF5: now also D16.A, D17.C, Q12.C, R2.P$1, R5.P$1; no longer D1.A, D11.C, Q3.C, R12.P$1, R16.P$1
Other:
- moved on the sheet: C1, C5, D1, D10, D11, D12, D14, D15, D16, D17, D18, D2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
