File: yoke/mimic1579.sch (EAGLE design)
At the start: 77 parts, among them J1 44PINEDGE, P1 2K, P2 2K, Q1 2N3904, Q10 2N3906, Q11 2N3904, Q12 2N3906, Q13 2N3904, Q2 2N3904, Q3 2N3904, Q4 2N3906, Q5 2N3904, Q6 2N3906, Q7 2N3904, Q8 2N3906, Q9 2N3904

Commit message: revised artwork
Parts:
- removed J1: 44PINEDGE, keiths:44PINEDGE
- added P3: 44PINEDGE-M, keiths:44PINEDGE-M
- R29, R34: value 475 -> 1.5K
- R30, R33, R35: value 1.5K -> 475
- R31: value 4.75K -> 1.5K
- R32: value 475 -> 4.75K
Connections:
- net -10V: now also P3.E; no longer J1.E
- net -15V: now also P3.C, R29.P$2, R31.P$2, R34.P$2; no longer J1.C, R30.P$2, R33.P$2, R35.P$2
- net F_IN: now also P3.F; no longer J1.F
- net GND: now also P3.4, P3.D; no longer J1.D
- net H_OUT: now also P3.H; no longer J1.H
- net J_IN: now also P3.J; no longer J1.J
- net K_IN: now also P3.K; no longer J1.K
- net L_IN: now also P3.L; no longer J1.L
- net N$11: now also R31.P$1, R34.P$1; no longer R33.P$1, R35.P$1
- net N$13: now also R30.P$1; no longer R29.P$1
- net N$14: now also R35.P$1; no longer R34.P$1
- net N$15: now also R33.P$2; no longer R31.P$2
- net N$18: now also D5.C; no longer D6.C
- net N$21: now also R29.P$1; no longer R30.P$1
- net N$23: now also R30.P$2; no longer R29.P$2
- net N$25: now also R33.P$1, R35.P$2; no longer R32.P$1, R34.P$2
- net N$5: now also D11.A; no longer D12.A
- net N$6: now also D6.C; no longer D5.C
- net P_OUT: now also P3.P; no longer J1.P
- net U_IN: now also P3.U, R32.P$1; no longer J1.U, R31.P$1
- net VREF1: now also D12.A; no longer D11.A
Other:
- note added: "X Feed Forward"
- moved on the sheet: C1, C2, C3, C4, C5, D1, D10, D11, D12, D13, D14, D15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

Commit message: added missing connector on bckplane
Parts:
- D1, D10, D11, D12, D13, D14, D15, D16, D17, D18, D19, D2, D3, D4, D5, D6, D7, D8, D9: device keiths:1N4148 -> replacements:1N4148
- R1, R10, R11, R12, R13, R14, R15, R16, R17, R18, R19, R2, R20, R21, R22, R23, R24, R25, R26, R27, R28, R29, R3, R30, R31, R32, R33, R34, R35, R4, R5, R6, R7, R8, R9: device keiths:R-1/4WATT -> replacements:R-1/4WATT
Connections:
- new net N$24: Q3.B, Q3.C, R7.P$1
- net -15V: now also P3.3
- net N$33: no longer Q3.B, Q3.C, R7.P$1
Other:
- moved on the sheet: C5, D12, D14, D15, D16, D18, D19, D4, D5, D6, D8, D9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
