File: yoke/mimic1568_DtoA.sch (EAGLE design)
At the start: 17 parts, among them P1 1K, P2 44PINEDGE, P3 1K, U1 CD74HCT75, U11 OPA2340N, U2 CD74HC573E, U3 CD74HC573E, U5 AD7533, U6 AD7533

Commit message: Friday backup
Parts:
- removed R10: 332, keiths:R-1/4WATT
- removed U11: OPA2340N, keiths:OPA2340N
- added C2, C3, C4, C7, C8: 0.1uF, keiths:CAP0.1UF100V
- added C6: 10pF, keiths:CAP0.1UF100V
- added R4: 332, keiths:R-1/4WATT
- added U4: OPA2340N, keiths:OPA2340N
- C1: value 10pF -> 0.1uF; device keiths:C-0.1 -> keiths:CAP0.1UF100V
- C5: device keiths:C-0.1 -> keiths:CAP0.1UF100V
- P1: PN 3006W-1-102LF -> (none)
- P2: value 44PINEDGE -> 1K; device keiths:44PINEDGE -> keiths:POT-3006P
- P3: value 1K -> 44PINEDGE; device keiths:POT-3006P -> keiths:44PINEDGE; PN 3006W-1-102LF -> (none)
- U1: value CD74HCT75 -> AD7533; device keiths:CD74HCT75 -> keiths:AD7533
- U3: value CD74HC573E -> CD74HCT75; device keiths:CD74HC573E -> keiths:CD74HCT75
- U6: value AD7533 -> CD74HC573E; device keiths:AD7533 -> keiths:CD74HC573E
Connections:
- removed net N$47: R10.P$2, U6.RFB
- new net N$2: R4.P$2, U5.RFB
- net +10V: now also C2.1, P1.2, P1.3, P2.2, P2.3, P3.A; no longer P1.E, P1.S, P3.E, P3.S
- net +15V: now also C4.1, P3.E, U1.VDD, U4P.V+; no longer P2.E, U11P.V+, U6.VDD
- net +5V: now also C1.1, C3.1, C8.1, P3.B, U6.+5V; no longer P2.B, U1.+5V
- net -15V: now also C7.1, P3.C, U4P.V-; no longer P2.C, U11P.V-
- net D0: now also P3.7, U3.1D0, U3.2D0, U6.D0; no longer P2.7, U1.1D0, U1.2D0, U3.D0
- net D1: now also P3.8, U3.1D1, U3.2D1, U6.D1; no longer P2.8, U1.1D1, U1.2D1, U3.D1
- net D2: now also P3.9, U6.D2; no longer P2.9, U3.D2
- net D3: now also P3.10, U6.D3; no longer P2.10, U3.D3
- net D4: now also P3.11, U6.D4; no longer P2.11, U3.D4
- net D5: now also P3.12, U6.D5; no longer P2.12, U3.D5
- net D6: now also P3.13, U6.D6; no longer P2.13, U3.D6
- net D7: now also P3.14, U6.D7; no longer P2.14, U3.D7
- net GND: now also C1.2, C2.2, C3.2, C4.2, C7.2, C8.2, P3.D, U6.!OE; no longer P2.D, U3.!OE
- net N$1: now also U3.2Q1, U5.D0; no longer U1.2Q1, U6.D0
- net N$10: now also U5.D6, U6.Q3; no longer U2.Q3, U6.D6
- net N$11: now also U5.D5, U6.Q4; no longer U2.Q4, U6.D5
- net N$12: now also U5.D4, U6.Q5; no longer U2.Q5, U6.D4
- net N$13: now also U5.D3, U6.Q6; no longer U2.Q6, U6.D3
- net N$14: now also U5.D2, U6.Q7; no longer U2.Q7, U6.D2
- net N$23: now also C5.2, R2.P$2, U4A.OUT; no longer C1.2, R3.P$2, U11A.OUT
- net N$24: now also P1.1, U1.VREF; no longer P1.A, U5.VREF
- net N$25: now also U1.D9, U2.Q0; no longer U3.Q0, U5.D9
- net N$26: now also U1.D8, U2.Q1; no longer U3.Q1, U5.D8
- net N$27: now also U1.D7, U2.Q2; no longer U3.Q2, U5.D7
- net N$28: now also U1.D6, U2.Q3; no longer U3.Q3, U5.D6
- net N$29: now also U1.D5, U2.Q4; no longer U3.Q4, U5.D5
- net N$3: now also U1.D1, U3.1Q0; no longer U1.1Q0, U5.D1
- net N$30: now also U1.D4, U2.Q5; no longer U3.Q5, U5.D4
- net N$31: now also U1.D3, U2.Q6; no longer U3.Q6, U5.D3
- net N$32: now also U1.D2, U2.Q7; no longer U3.Q7, U5.D2
- net N$35: now also U3.2Q0, U5.D1; no longer U1.2Q0, U6.D1
- net N$38: now also U1.RFB; no longer U5.RFB
- net N$4: now also U1.D0, U3.1Q1; no longer U1.1Q1, U5.D0
- net N$44: now also C6.2, R3.P$2, R4.P$1, U4B.OUT; no longer C5.2, R10.P$1, R2.P$2, U11B.OUT
- net N$45: now also C6.1, U4B.-IN, U5.IO1; no longer C5.1, U11B.-IN, U6.IO1
- net N$46: now also U4B.+IN, U5.IO2; no longer U11B.+IN, U6.IO2
- net N$5: now also C5.1, U1.IO1, U4A.-IN; no longer C1.1, U11A.-IN, U5.IO1
- net N$53: now also P2.1, U5.VREF; no longer P3.A, U6.VREF
- net N$6: now also U1.IO2, U4A.+IN; no longer U11A.+IN, U5.IO2
- net N$7: now also U5.D9, U6.Q0; no longer U2.Q0, U6.D9
- net N$8: now also U5.D8, U6.Q1; no longer U2.Q1, U6.D8
- net N$9: now also U5.D7, U6.Q2; no longer U2.Q2, U6.D7
- net XPOS: now also P3.J, R2.P$1; no longer P2.J, R3.P$1
- net X_LSB: now also P3.17, U3.!1LE; no longer P2.17, U1.!1LE
- net X_MSB: now also P3.16, U2.LE; no longer P2.16, U3.LE
- net YPOS: now also P3.K, R3.P$1; no longer P2.K, R2.P$1
- net Y_LSB: now also P3.19, U3.!2LE; no longer P2.19, U1.!2LE
- net Y_MSB: now also P3.18, U6.LE; no longer P2.18, U2.LE
Other:
- moved on the sheet: R1, R2, R3, U1, U2, U5
