File: yoke/mimic1567.brd (EAGLE design)
At the start: 160 x 100 mm, 74 parts, among them J10 OUT_2, J12 COIL 2, J13 OUT_2, J14 RESISTOR_2, J2 RESISTOR_2, J3 GND, J4 GND, J5 OUT_1, J6 COIL 1, J7 RESISTOR_1, J8 OUT_1, J9 RESISTOR_1, P1 25 K, P2 10 K, P3 200, P5 20 K, P6 44PINEDGE, P7 20, Q1 2N3904, Q10 2N2907, Q11 MJ10007, Q12 2N3906, Q14 MJ10007, Q2 2N3904, Q3 2N3904, Q4 2N3904, Q5 2N3904, Q6 2N3904, Q7 2N3904, Q8 2N2907, Q9 2N3906

Commit message: working on wire harness
Parts:
- moved Q11 288.8 mm to (-170.2, -141.0)
- moved J6 199.6 mm to (-163.8, -101.6)
- moved J8 144.5 mm to (-61.0, -3.81)
- moved R2 139.8 mm to (-91.4, -36.8)
- moved J10 137.4 mm to (-8.89, -91.4)
Changed lines of the file:
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@@
 <element name="J3" library="keiths" package="AWG18" value="GND" x="-120.65" y="91.44"/>
 <element name="J4" library="keiths" package="AWG18" value="GND" x="-128.27" y="91.44"/>
-<element name="J6" library="keiths" package="AWG18" value="COIL 1" x="-113.03" y="91.44"/>
+<element name="J6" library="keiths" package="AWG18" value="COIL 1" x="-163.83" y="-101.6"/>
 <element name="J7" library="keiths" package="AWG18" value="RESISTOR_1" x="-90.17" y="91.44"/>
 <element name="P1" library="keiths" package="3006P" value="25 K" x="-82.55" y="78.74">
@@
 <attribute name="PN" value="2N2907A" x="-104.14" y="140.97" size="1.778" layer="27" display="off"/>
 </element>
-<element name="Q11" library="keiths" package="TO3" value="MJ10007" x="105.41" y="-54.61" rot="R90">
-<attribute name="PN" value="MJ10007" x="105.41" y="-54.61" size="1.778" layer="27" rot="R90" display="off"/>
+<element name="Q11" library="keiths" package="TO3" value="MJ10007" x="-170.18" y="-140.97" rot="R90">
+<attribute name="PN" value="MJ10007" x="-170.18" y="-140.97" size="1.778" layer="27" rot="R90" display="off"/>
 </element>
 <element name="Q12" library="keiths" package="TO92" value="2N3906" x="-71.12" y="123.19">
@@
 <attribute name="PN" value="MFR-25FRF52-1K" x="-72.39" y="113.03" size="1.778" layer="27" display="off"/>
 </element>
-<element name="R2" library="keiths" package="R_TWOWATT" value="3.3K 5%" x="31.75" y="-102.87">
-<attribute name="PN" value="RR02J3K3TB" x="31.75" y="-102.87" size="1.778" layer="27" display="off"/>
+<element name="R2" library="keiths" package="R_TWOWATT" value="3.3K 5%" x="-91.44" y="-36.83">
+<attribute name="PN" value="RR02J3K3TB" x="-91.44" y="-36.83" size="1.778" layer="27" display="off"/>
 </element>
 <element name="R20" library="keiths" package="R_QUARTERWATT" value="137 1%" x="-85.09" y="113.03">
@@
 </element>
 <element name="J5" library="keiths" package="AWG18" value="OUT_1" x="-132.08" y="-118.11"/>
-<element name="J8" library="keiths" package="AWG18" value="OUT_1" x="-132.08" y="-129.54"/>
+<element name="J8" library="keiths" package="AWG18" value="OUT_1" x="-60.96" y="-3.81"/>
 <element name="J9" library="keiths" package="AWG18" value="RESISTOR_1" x="-132.08" y="-140.97"/>
-<element name="J10" library="keiths" package="AWG18" value="OUT_2" x="-132.08" y="-152.4"/>
+<element name="J10" library="keiths" package="AWG18" value="OUT_2" x="-8.89" y="-91.44"/>
 <element name="Q14" library="keiths" package="TO3" value="MJ10007" x="-114.3" y="-182.88">
 <attribute name="PN" value="MJ10007" x="-114.3" y="-182.88" size="1.778" layer="27" display="off"/>
@@
 <contactref element="J10" pad="P$1"/>
 <wire x1="-83.185" y1="140.97" x2="-59.69" y2="140.97" width="0" layer="19" extent="1-1"/>
-<wire x1="40.5" y1="-102.87" x2="-59.69" y2="140.97" width="0" layer="19" extent="1-1"/>
-<wire x1="-132.08" y1="-152.4" x2="40.5" y2="-102.87" width="0" layer="19" extent="1-1"/>
+<wire x1="-82.69" y1="-36.83" x2="-59.69" y2="140.97" width="0" layer="19" extent="1-1"/>
+<wire x1="-8.89" y1="-91.44" x2="-82.69" y2="-36.83" width="0" layer="19" extent="1-1"/>
 </signal>
 <signal name="N$7">
@@
 <contactref element="Q11" pad="C"/>
 <contactref element="Q11" pad="C/"/>
-<wire x1="105.41" y1="-69.723" x2="105.41" y2="-39.497" width="0" layer="19" extent="1-1"/>
-<wire x1="-113.03" y1="91.44" x2="105.41" y2="-39.497" width="0" layer="19" extent="1-1"/>
+<wire x1="-170.18" y1="-156.083" x2="-170.18" y2="-125.857" width="0" layer="19" extent="1-1"/>
+<wire x1="-163.83" y1="-101.6" x2="-170.18" y2="-125.857" width="0" layer="19" extent="1-1"/>
 </signal>
 <signal name="N$27">
@@
 <contactref element="J8" pad="P$1"/>
 <wire x1="-130.81" y1="121.92" x2="-102.235" y2="140.97" width="0" layer="19" extent="1-1"/>
-<wire x1="-132.08" y1="-129.54" x2="-130.81" y2="121.92" width="0" layer="19" extent="1-1"/>
-<wire x1="98.92" y1="-106.68" x2="-132.08" y2="-129.54" width="0" layer="19" extent="1-1"/>
+<wire x1="-60.96" y1="-3.81" x2="-130.81" y2="121.92" width="0" layer="19" extent="1-1"/>
+<wire x1="98.92" y1="-106.68" x2="-60.96" y2="-3.81" width="0" layer="19" extent="1-1"/>
 </signal>
 <signal name="N$33">
@@
 <contactref element="R9" pad="1"/>
 <contactref element="R3" pad="1"/>
-<wire x1="81.42" y1="-106.68" x2="23" y2="-102.87" width="0" layer="19" extent="1-1"/>
-<wire x1="-94.3356" y1="50.546" x2="23" y2="-102.87" width="0" layer="19" extent="16-16"/>
+<wire x1="81.42" y1="-106.68" x2="-100.19" y2="-36.83" width="0" layer="19" extent="1-1"/>
+<wire x1="-94.3356" y1="50.546" x2="-100.19" y2="-36.83" width="0" layer="19" extent="16-16"/>
 <wire x1="-82.05" y1="102.87" x2="-94.3356" y2="50.546" width="0" layer="19" extent="16-16"/>
 <wire x1="-65.54" y1="102.87" x2="-82.05" y2="102.87" width="0" layer="19" extent="1-1"/>
@@
 <contactref element="Q11" pad="B"/>
 <contactref element="J5" pad="P$1"/>
-<wire x1="99.949" y1="-56.388" x2="-132.08" y2="-118.11" width="0" layer="19" extent="1-1"/>
+<wire x1="-175.641" y1="-142.748" x2="-132.08" y2="-118.11" width="0" layer="19" extent="1-1"/>
 </signal>
 <signal name="N$28">
 <contactref element="Q11" pad="E"/>
 <contactref element="J9" pad="P$1"/>
-<wire x1="-132.08" y1="-140.97" x2="110.871" y2="-56.388" width="0" layer="19" extent="1-1"/>
+<wire x1="-132.08" y1="-140.97" x2="-164.719" y2="-142.748" width="0" layer="19" extent="1-1"/>
 </signal>
 <signal name="N$32">

Commit message: more work
Parts:
- removed J10, J13: OUT_2, keiths:AWG18
- removed J12: COIL 2, keiths:AWG18
- removed J14, J2: RESISTOR_2, keiths:AWG18
- removed J4: GND, keiths:AWG18
- removed J5, J8: OUT_1, keiths:AWG18
- removed J6: COIL 1, keiths:AWG18
- removed J7, J9: RESISTOR_1, keiths:AWG18
- removed P3: 200, keiths:3006P
- removed P7: 20, keiths:3006P
- removed Q11, Q14: MJ10007, keiths:TO3
- added J15: JST-VH-5, keiths:VHR-5N
- added P4: 20 K, keiths:3006P
- added R24: 2 K 1%, keiths:R_QUARTERWATT
- added R26: 274 K 1%, keiths:R_QUARTERWATT
- P5: value 20 K -> 200
- R23: value 274 K 1% -> 2 K 1%
- moved R23 610.7 mm to (-176.5, -486.4)
- moved R19 598.4 mm to (-176.5, -476.2)
- moved R14 570.9 mm to (-176.5, -466.1)
- moved P5 536.6 mm to (-172.7, -424.2)
- moved R21 531.6 mm to (-176.5, -412.8)
Connections:
- removed net N$18: P5.1, P7.2, P7.3, R21.2
- removed net N$24: J5.P$1, Q11.B
- removed net N$26: J6.P$1, Q11.C, Q11.C/
- removed net N$28: J9.P$1, Q11.E
- removed net N$32: J12.P$1, Q14.C, Q14.C/
- removed net N$41: J13.P$1, Q14.B
- removed net N$42: J14.P$1, Q14.E
- net GND: now also J15.P$5; no longer J4.P$1
- net N$2: now also J15.P$4, R24.2; no longer J2.P$1
- net N$22: now also P5.1, R26.1; no longer P3.1, R23.1
- net N$27: now also J15.P$2, R23.1; no longer J7.P$1
- net N$31: now also J15.P$1; no longer J8.P$1
- net N$43: now also R21.2, R23.2; no longer R19.2
- net N$44: now also P5.3; no longer P3.3
- net N$5: now also J15.P$3; no longer J10.P$1
- net N$6: now also R19.2, R24.1; no longer R21.1
- net W_IN: now also P4.2, P4.3, R21.1, R26.2; no longer P3.2, P5.3, R19.1, R23.2
- net Z_IN: now also P4.1, R19.1; no longer P7.1

Commit message: more changes
Parts:
- removed J3: GND, keiths:AWG18
Connections:
- removed net -150V: P6.V
- removed net CATHODE: P6.Z
- removed net J_IN: P6.J
- removed net P_IN: P6.P
- removed net U_IN: P6.U
- removed net X_IN: P6.X
- net GND: no longer J3.P$1
- net W_IN: now also P6.W
- net Z_IN: now also P6.Z
Changed lines of the file:
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@@
 <attribute name="PN" value="1N4736A" x="-97.79" y="123.19" size="1.778" layer="27" display="off"/>
 </element>
-<element name="J3" library="keiths" package="AWG18" value="GND" x="-120.65" y="91.44"/>
 <element name="P1" library="keiths" package="3006P" value="25 K" x="-82.55" y="78.74">
 <attribute name="PN" value="3006P-1-253LF" x="-82.55" y="78.74" size="1.778" layer="27" display="off"/>
@@
 <contactref element="R26" pad="2"/>
 <contactref element="P5" pad="2"/>
+<contactref element="P6" pad="W"/>
 <wire x1="-171.577" y1="-425.45" x2="-172.03" y2="-445.77" width="0" layer="19" extent="1-1"/>
 <wire x1="-181.03" y1="-412.75" x2="-171.577" y2="-425.45" width="0" layer="19" extent="1-1"/>
 <wire x1="-171.577" y1="-402.59" x2="-181.03" y2="-412.75" width="0" layer="19" extent="1-1"/>
 <wire x1="-166.497" y1="-400.05" x2="-171.577" y2="-402.59" width="0" layer="19" extent="1-1"/>
-<wire x1="-38.68" y1="113.03" x2="-166.497" y2="-400.05" width="0" layer="19" extent="1-1"/>
+<wire x1="-38.862" y1="50.546" x2="-166.497" y2="-400.05" width="0" layer="19" extent="16-16"/>
+<wire x1="-38.68" y1="113.03" x2="-38.862" y2="50.546" width="0" layer="19" extent="16-16"/>
 </signal>
 <signal name="N$43">
@@
 <contactref element="R13" pad="2"/>
 <contactref element="R11" pad="1"/>
-<contactref element="J3" pad="P$1"/>
+<contactref element="R14" pad="2"/>
 <contactref element="J15" pad="P$5"/>
-<contactref element="R14" pad="2"/>
 <wire x1="-6.35" y1="-14.4" x2="153.67" y2="-10.59" width="0" layer="19" extent="1-1"/>
 <wire x1="-98.298" y1="50.546" x2="-6.35" y2="-14.4" width="0" layer="19" extent="16-16"/>
@@
 <wire x1="-81.407" y1="77.47" x2="-97.917" y2="80.01" width="0" layer="19" extent="1-1"/>
 <wire x1="-76.327" y1="80.01" x2="-81.407" y2="77.47" width="0" layer="19" extent="1-1"/>
-<wire x1="-120.65" y1="91.44" x2="-102.997" y2="77.47" width="0" layer="19" extent="1-1"/>
-<wire x1="-125.15" y1="113.03" x2="-120.65" y2="91.44" width="0" layer="19" extent="1-1"/>
-<wire x1="-113.72" y1="113.03" x2="-125.15" y2="113.03" width="0" layer="19" extent="1-1"/>
+<wire x1="-113.72" y1="113.03" x2="-97.917" y2="80.01" width="0" layer="19" extent="1-1"/>
+<wire x1="-125.15" y1="113.03" x2="-113.72" y2="113.03" width="0" layer="19" extent="1-1"/>
 <wire x1="-179.18" y1="-356.51" x2="-6.35" y2="-14.4" width="0" layer="19" extent="1-1"/>
 <wire x1="-172.03" y1="-466.09" x2="-179.18" y2="-356.51" width="0" layer="19" extent="1-1"/>
 </signal>
-<signal name="J_IN">
-<contactref element="P6" pad="J"/>
-</signal>
 <signal name="-15V">
 <contactref element="P6" pad="C"/>
@@
 <contactref element="P6" pad="F"/>
 </signal>
-<signal name="U_IN">
-<contactref element="P6" pad="U"/>
-</signal>
-<signal name="X_IN">
-<contactref element="P6" pad="X"/>
-</signal>
-<signal name="P_IN">
-<contactref element="P6" pad="P"/>
-</signal>
-<signal name="-150V">
-<contactref element="P6" pad="V"/>
-</signal>
 <signal name="+10V">
 <contactref element="P6" pad="A"/>
-</signal>
-<signal name="CATHODE">
-<contactref element="P6" pad="Z"/>
 </signal>
 <signal name="+50V">
@@
 <contactref element="P4" pad="1"/>
 <contactref element="R19" pad="1"/>
+<contactref element="P6" pad="Z"/>
 <wire x1="-179.197" y1="-400.05" x2="-181.03" y2="-476.25" width="0" layer="19" extent="1-1"/>
+<wire x1="-26.9748" y1="50.546" x2="-179.197" y2="-400.05" width="0" layer="19" extent="16-16"/>
 </signal>
 </signals>

Commit message: update netlist
Parts:
- moved J15 351.8 mm to (-172.7, -12.7)
- moved P5 351.8 mm to (-175.3, -72.4)
- moved R19 351.8 mm to (-179.1, -124.5)
- moved R21 351.8 mm to (-179.1, -61.0)
- moved R23 351.8 mm to (-179.1, -134.6)
- moved R24 351.8 mm to (-179.1, -27.9)
- moved P4 351.8 mm to (-175.3, -49.5)
- moved R14 351.8 mm to (-179.1, -114.3)
- moved R26 351.8 mm to (-179.1, -94.0)
Changed lines of the file:
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@@
 <attribute name="PN" value="MFS1/2DCT52R6811F" x="-76.2" y="102.87" size="1.778" layer="27" display="off"/>
 </element>
-<element name="J15" library="keiths" package="VHR-5N" value="JST-VH-5" x="-170.18" y="-364.49"/>
-<element name="R24" library="keiths" package="R_QUARTERWATT" value="2 K 1%" x="-176.53" y="-379.73">
-<attribute name="PN" value="MFR-25FRF52-2K" x="-176.53" y="-379.73" size="1.778" layer="27" display="off"/>
-</element>
-<element name="P4" library="keiths" package="3006P" value="20 K" x="-172.72" y="-401.32">
-<attribute name="PN" value="3006P-1-203LF" x="-172.72" y="-401.32" size="1.778" layer="27" display="off"/>
-</element>
-<element name="R21" library="keiths" package="R_QUARTERWATT" value="1 K 1%" x="-176.53" y="-412.75">
-<attribute name="PN" value="MFR-25FRF52-1K" x="-176.53" y="-412.75" size="1.778" layer="27" display="off"/>
-</element>
-<element name="P5" library="keiths" package="3006P" value="200" x="-172.72" y="-424.18">
-<attribute name="PN" value="3006P-1-201LF" x="-172.72" y="-424.18" size="1.778" layer="27" display="off"/>
-</element>
-<element name="R26" library="keiths" package="R_QUARTERWATT" value="274 K 1%" x="-176.53" y="-445.77">
-<attribute name="PN" value="MFR-25FBF52-274K" x="-176.53" y="-445.77" size="1.778" layer="27" display="off"/>
-</element>
-<element name="R14" library="keiths" package="R_QUARTERWATT" value="1.96 K 1 %" x="-176.53" y="-466.09">
-<attribute name="PN" value="RNF14FTD1K96" x="-176.53" y="-466.09" size="1.778" layer="27" display="off"/>
-</element>
-<element name="R19" library="keiths" package="R_QUARTERWATT" value="1 K 1%" x="-176.53" y="-476.25">
-<attribute name="PN" value="MFR-25FRF52-1K" x="-176.53" y="-476.25" size="1.778" layer="27" display="off"/>
-</element>
-<element name="R23" library="keiths" package="R_QUARTERWATT" value="2 K 1%" x="-176.53" y="-486.41">
-<attribute name="PN" value="MFR-25FRF52-2K" x="-176.53" y="-486.41" size="1.778" layer="27" display="off"/>
+<element name="J15" library="keiths" package="VHR-5N" value="JST-VH-5" x="-172.72" y="-12.7"/>
+<element name="R24" library="keiths" package="R_QUARTERWATT" value="2 K 1%" x="-179.07" y="-27.94">
+<attribute name="PN" value="MFR-25FRF52-2K" x="-179.07" y="-27.94" size="1.778" layer="27" display="off"/>
+</element>
+<element name="P4" library="keiths" package="3006P" value="20 K" x="-175.26" y="-49.53">
+<attribute name="PN" value="3006P-1-203LF" x="-175.26" y="-49.53" size="1.778" layer="27" display="off"/>
+</element>
+<element name="R21" library="keiths" package="R_QUARTERWATT" value="1 K 1%" x="-179.07" y="-60.96">
+<attribute name="PN" value="MFR-25FRF52-1K" x="-179.07" y="-60.96" size="1.778" layer="27" display="off"/>
+</element>
+<element name="P5" library="keiths" package="3006P" value="200" x="-175.26" y="-72.39">
+<attribute name="PN" value="3006P-1-201LF" x="-175.26" y="-72.39" size="1.778" layer="27" display="off"/>
+</element>
+<element name="R26" library="keiths" package="R_QUARTERWATT" value="274 K 1%" x="-179.07" y="-93.98">
+<attribute name="PN" value="MFR-25FBF52-274K" x="-179.07" y="-93.98" size="1.778" layer="27" display="off"/>
+</element>
+<element name="R14" library="keiths" package="R_QUARTERWATT" value="1.96 K 1 %" x="-179.07" y="-114.3">
+<attribute name="PN" value="RNF14FTD1K96" x="-179.07" y="-114.3" size="1.778" layer="27" display="off"/>
+</element>
+<element name="R19" library="keiths" package="R_QUARTERWATT" value="1 K 1%" x="-179.07" y="-124.46">
+<attribute name="PN" value="MFR-25FRF52-1K" x="-179.07" y="-124.46" size="1.778" layer="27" display="off"/>
+</element>
+<element name="R23" library="keiths" package="R_QUARTERWATT" value="2 K 1%" x="-179.07" y="-134.62">
+<attribute name="PN" value="MFR-25FRF52-2K" x="-179.07" y="-134.62" size="1.778" layer="27" display="off"/>
 </element>
 </elements>
@@
 <contactref element="R24" pad="2"/>
 <contactref element="J15" pad="P$4"/>
-<wire x1="-179.18" y1="-360.51" x2="-6.35" y2="-69.669659375" width="0" layer="19" extent="1-1"/>
-<wire x1="-172.03" y1="-379.73" x2="-179.18" y2="-360.51" width="0" layer="19" extent="1-1"/>
+<wire x1="-181.72" y1="-8.72" x2="-6.35" y2="-69.669659375" width="0" layer="19" extent="1-1"/>
+<wire x1="-174.57" y1="-27.94" x2="-181.72" y2="-8.72" width="0" layer="19" extent="1-1"/>
 </signal>
 <signal name="N$3">
@@
 <wire x1="-83.185" y1="140.97" x2="-82.69" y2="-36.83" width="0" layer="19" extent="1-1"/>
 <wire x1="-59.69" y1="140.97" x2="-83.185" y2="140.97" width="0" layer="19" extent="1-1"/>
-<wire x1="-179.18" y1="-364.51" x2="-82.69" y2="-36.83" width="0" layer="19" extent="1-1"/>
+<wire x1="-181.72" y1="-12.72" x2="-82.69" y2="-36.83" width="0" layer="19" extent="1-1"/>
 </signal>
 <signal name="N$7">
@@
 <contactref element="R23" pad="1"/>
 <contactref element="J15" pad="P$2"/>
-<wire x1="-179.18" y1="-372.47" x2="-181.03" y2="-486.41" width="0" layer="19" extent="1-1"/>
-<wire x1="153.67" y1="-67.129659375" x2="-179.18" y2="-372.47" width="0" layer="19" extent="1-1"/>
+<wire x1="-181.72" y1="-20.68" x2="-183.57" y2="-134.62" width="0" layer="19" extent="1-1"/>
+<wire x1="153.67" y1="-67.129659375" x2="-181.72" y2="-20.68" width="0" layer="19" extent="1-1"/>
 </signal>
 <signal name="N$30">
@@
 <wire x1="-130.81" y1="121.92" x2="-102.235" y2="140.97" width="0" layer="19" extent="1-1"/>
 <wire x1="98.92" y1="-106.68" x2="-102.235" y2="140.97" width="0" layer="19" extent="1-1"/>
-<wire x1="-179.18" y1="-368.51" x2="98.92" y2="-106.68" width="0" layer="19" extent="1-1"/>
+<wire x1="-181.72" y1="-16.72" x2="98.92" y2="-106.68" width="0" layer="19" extent="1-1"/>
 </signal>
 <signal name="N$33">
@@
 <contactref element="R26" pad="1"/>
 <contactref element="R14" pad="1"/>
-<wire x1="-181.03" y1="-445.77" x2="-181.03" y2="-466.09" width="0" layer="19" extent="1-1"/>
-<wire x1="-179.197" y1="-422.91" x2="-181.03" y2="-445.77" width="0" layer="19" extent="1-1"/>
-<wire x1="-80.59" y1="113.03" x2="-179.197" y2="-422.91" width="0" layer="19" extent="1-1"/>
+<wire x1="-183.57" y1="-93.98" x2="-183.57" y2="-114.3" width="0" layer="19" extent="1-1"/>
+<wire x1="-181.737" y1="-71.12" x2="-183.57" y2="-93.98" width="0" layer="19" extent="1-1"/>
+<wire x1="-80.59" y1="113.03" x2="-181.737" y2="-71.12" width="0" layer="19" extent="1-1"/>
 </signal>
 <signal name="W_IN">
@@
 <contactref element="P5" pad="2"/>
 <contactref element="P6" pad="W"/>
-<wire x1="-171.577" y1="-425.45" x2="-172.03" y2="-445.77" width="0" layer="19" extent="1-1"/>
-<wire x1="-181.03" y1="-412.75" x2="-171.577" y2="-425.45" width="0" layer="19" extent="1-1"/>
-<wire x1="-171.577" y1="-402.59" x2="-181.03" y2="-412.75" width="0" layer="19" extent="1-1"/>
-<wire x1="-166.497" y1="-400.05" x2="-171.577" y2="-402.59" width="0" layer="19" extent="1-1"/>
-<wire x1="-38.862" y1="50.546" x2="-166.497" y2="-400.05" width="0" layer="19" extent="16-16"/>
+<wire x1="-174.117" y1="-73.66" x2="-174.57" y2="-93.98" width="0" layer="19" extent="1-1"/>
+<wire x1="-183.57" y1="-60.96" x2="-174.117" y2="-73.66" width="0" layer="19" extent="1-1"/>
+<wire x1="-174.117" y1="-50.8" x2="-183.57" y2="-60.96" width="0" layer="19" extent="1-1"/>
+<wire x1="-169.037" y1="-48.26" x2="-174.117" y2="-50.8" width="0" layer="19" extent="1-1"/>
+<wire x1="-38.862" y1="50.546" x2="-169.037" y2="-48.26" width="0" layer="19" extent="16-16"/>
 <wire x1="-38.68" y1="113.03" x2="-38.862" y2="50.546" width="0" layer="19" extent="16-16"/>
 </signal>
@@
 <contactref element="R21" pad="2"/>
 <contactref element="R23" pad="2"/>
-<wire x1="-172.03" y1="-412.75" x2="-172.03" y2="-486.41" width="0" layer="19" extent="1-1"/>
-<wire x1="-54.61" y1="124.46" x2="-172.03" y2="-412.75" width="0" layer="19" extent="1-1"/>
+<wire x1="-174.57" y1="-60.96" x2="-174.57" y2="-134.62" width="0" layer="19" extent="1-1"/>
+<wire x1="-54.61" y1="124.46" x2="-174.57" y2="-60.96" width="0" layer="19" extent="1-1"/>
 </signal>
 <signal name="N$44">
@@
 <wire x1="-47.68" y1="113.03" x2="-31.17" y2="113.03" width="0" layer="19" extent="1-1"/>
 <wire x1="-89.59" y1="113.03" x2="-47.68" y2="113.03" width="0" layer="19" extent="1-1"/>
-<wire x1="-166.497" y1="-422.91" x2="-89.59" y2="113.03" width="0" layer="19" extent="1-1"/>
+<wire x1="-169.037" y1="-71.12" x2="-89.59" y2="113.03" width="0" layer="19" extent="1-1"/>
 </signal>
 <signal name="GND">
@@
 <wire x1="-113.72" y1="113.03" x2="-97.917" y2="80.01" width="0" layer="19" extent="1-1"/>
 <wire x1="-125.15" y1="113.03" x2="-113.72" y2="113.03" width="0" layer="19" extent="1-1"/>
-<wire x1="-179.18" y1="-356.51" x2="-6.35" y2="-14.4" width="0" layer="19" extent="1-1"/>
-<wire x1="-172.03" y1="-466.09" x2="-179.18" y2="-356.51" width="0" layer="19" extent="1-1"/>
+<wire x1="-181.72" y1="-4.72" x2="-6.35" y2="-14.4" width="0" layer="19" extent="1-1"/>
+<wire x1="-174.57" y1="-114.3" x2="-181.72" y2="-4.72" width="0" layer="19" extent="1-1"/>
 </signal>
 <signal name="-15V">
@@
 <contactref element="R24" pad="1"/>
 <contactref element="R19" pad="2"/>
-<wire x1="-181.03" y1="-379.73" x2="-172.03" y2="-476.25" width="0" layer="19" extent="1-1"/>
-<wire x1="-24.13" y1="124.46" x2="-181.03" y2="-379.73" width="0" layer="19" extent="1-1"/>
+<wire x1="-183.57" y1="-27.94" x2="-174.57" y2="-124.46" width="0" layer="19" extent="1-1"/>
+<wire x1="-24.13" y1="124.46" x2="-183.57" y2="-27.94" width="0" layer="19" extent="1-1"/>
 </signal>
 <signal name="Z_IN">
@@
 <contactref element="R19" pad="1"/>
 <contactref element="P6" pad="Z"/>
-<wire x1="-179.197" y1="-400.05" x2="-181.03" y2="-476.25" width="0" layer="19" extent="1-1"/>
-<wire x1="-26.9748" y1="50.546" x2="-179.197" y2="-400.05" width="0" layer="19" extent="16-16"/>
+<wire x1="-181.737" y1="-48.26" x2="-183.57" y2="-124.46" width="0" layer="19" extent="1-1"/>
+<wire x1="-26.9748" y1="50.546" x2="-181.737" y2="-48.26" width="0" layer="19" extent="16-16"/>
 </signal>
 </signals>
