File: yoke/mimic1567.brd (EAGLE design)
At the start: 165.1 x 114.3 mm, 71 parts, among them J1 JST-VH-5, P1 20K, P2 25 K, P3 5K, P4 200, P5 44PINEDGE, Q1 2N2907, Q10 2N3904, Q11 2N2907, Q2 2N3904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

Commit message: end of day
Parts:
- added R31: 330, keiths:R_ONEWATT
- R1: value 274K -> 1M
- R10: value 1.96K -> 3.3; device keiths:R_QUARTERWATT -> keiths:0309/12
- R11, R9: value 3.3 -> 1.96K; device keiths:0309/12 -> keiths:R_QUARTERWATT
- R12: value 100 -> 3.3; device keiths:R_QUARTERWATT -> keiths:0309/12
- R13: value 22 -> 100
- R15: value 6.81K -> 22; device keiths:R_HALFWATT -> keiths:R_QUARTERWATT
- R16, R21: value 33.2K -> 6.81K
- R17, R22: value 100 -> 33.2K; device keiths:R_QUARTERWATT -> keiths:R_HALFWATT
- R19, R23: value 2K -> 100
- R2: value 20K -> 274K
- R20: value 6.81K -> 2K; device keiths:R_HALFWATT -> keiths:R_QUARTERWATT
- R24: value 10K -> 2K; device keiths:R_HALFWATT -> keiths:R_QUARTERWATT
- R25: value 1K -> 10K; device keiths:R_QUARTERWATT -> keiths:R_HALFWATT
- R26: value 1.2K -> 1K; device keiths:R_FIVEWATT -> keiths:R_QUARTERWATT
- R28: value 1K -> 1.2K; device keiths:R_QUARTERWATT -> keiths:R_FIVEWATT
- R29: value 330 -> 1K; device keiths:R_ONEWATT -> keiths:R_QUARTERWATT
- R4: value 3.9K -> 20K
- R5: value 4.7K -> 3.9K
- R6: value 274K -> 4.7K
- R7: value 137 -> 274K
- R8: value 1.96K -> 137
- moved R28 127.8 mm to (146.8, 26.7), turned to 0 degrees
- moved R26 116.4 mm to (30.5, 34.3)
- moved R12 92.6 mm to (151.0, 73.8)
- moved R1 82.9 mm to (16.5, 100.1), turned to 90 degrees
- moved R25 79.3 mm to (98.3, 41.1)
- moved R29 77.9 mm to (30.2, 27.9), turned to 0 degrees
- moved R20 62.6 mm to (86.4, 55.9), turned to 90 degrees
- moved R2 60.8 mm to (92.5, 99.9)
- moved R15 60.6 mm to (84.6, 71.4), turned to 180 degrees
- moved R9 56.3 mm to (88.8, 89.4)
- moved R6 31.9 mm to (68.1, 97.5), turned to 270 degrees
- moved R11 28.9 mm to (122.9, 80.8), turned to 270 degrees
- moved R17 28.1 mm to (39.9, 67.8), turned to 0 degrees
- moved R8 27.6 mm to (116.3, 90.9), turned to 270 degrees
- moved R22 26.5 mm to (39.9, 49.5), turned to 0 degrees
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Connections:
- net +50V: now also R16.1, R21.1, R28.1; no longer R15.1, R20.1, R26.1
- net -10V: now also R11.2, R15.2, R19.2, R23.2, R25.2, R31.2; no longer R10.2, R12.2, R17.2, R22.2, R24.2, R29.2
- net GND: now also R10.2, R12.2, R6.1; no longer R11.2, R2.1, R8.2
- net N$1: now also R15.1; no longer R14.1
- net N$16: now also R17.2; no longer R16.2
- net N$17: now also R16.2, R17.1; no longer R15.2, R16.1
- net N$18: now also R14.1; no longer R13.1
- net N$2: now also R20.2; no longer R19.2
- net N$20: now also R21.2, R22.1; no longer R20.2, R21.1
- net N$22: now also R7.1, R8.2, R9.1; no longer R6.1, R7.2, R8.1
- net N$23: now also R23.1; no longer R22.1
- net N$24: now also R19.1; no longer R17.1
- net N$25: now also R22.2; no longer R21.2
- net N$26: now also R13.1; no longer R12.1
- net N$27: now also R24.1; no longer R23.1
- net N$29: now also R6.2; no longer R4.2
- net N$3: now also R10.1; no longer R9.1
- net N$30: now also R12.1; no longer R11.1
- net N$31: now also R28.2; no longer R27.2
- net N$33: now also R25.1; no longer R24.1
- net N$34: now also R31.1; no longer R30.1
- net N$4: now also R4.2; no longer R2.2
- net N$43: now also R24.2, R26.2; no longer R23.2, R25.2
- net N$44: now also R11.1, R2.1, R8.1; no longer R1.1, R10.1, R7.1
- net N$5: now also R27.2; no longer R26.2
- net N$6: now also R20.1, R29.2; no longer R19.1, R28.2
- net N$8: now also R30.1; no longer R29.1
- net W_IN: now also R2.2, R26.1, R7.2; no longer R25.1, R6.2
- net Z_IN: now also R1.1, R29.1; no longer R28.1
Routing:
- net N$43: track 82.5 -> 62.8 mm
- net N$6: track 114.4 -> 96.9 mm
- net W_IN: track 186.5 -> 197.2 mm
- net -10V: track 315.4 -> 305.1 mm
- net N$40: track 79.8 -> 88.8 mm
- net N$44: track 40.3 -> 49.1 mm
- net N$39: track 12.7 -> 5.08 mm
- net N$27: track 155.3 -> 160.8 mm
- net Z_IN: track 97.1 -> 100.9 mm
- net N$20: track 12.9 -> 10.4 mm
- net N$21: track 11.3 -> 9.69 mm
- net N$24: track 6.73 -> 5.34 mm
- net N$16: track 37.1 -> 38.2 mm
- net N$29: track 80.1 -> 81.0 mm
- net N$15: track 98.5 -> 99.3 mm
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
Commit message: added logo
Other:
- board text added: "board type 1567 / preamplifier"
