File: yoke/mimic1567.brd (EAGLE design)
At the start: 165.1 x 114.3 mm, 72 parts, among them J1 JST-VH-5, P1 20K, P2 25 K, P3 5K, P4 200, P5 44PINEDGE, Q1 2N2907, Q10 2N3904, Q11 2N2907, Q2 2N3904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

Commit message: revised artwork
Parts:
- P5: value 44PINEDGE -> 44PINEDGE-M
- R26, R29: value 1K -> 1.2K; device keiths:R_QUARTERWATT -> keiths:R_FIVEWATT
- R27, R28: value 1.2K -> 1K; device keiths:R_FIVEWATT -> keiths:R_QUARTERWATT
- moved R28 116.6 mm to (30.2, 27.9)
- moved R29 116.6 mm to (146.8, 26.7)
- moved R26 116.4 mm to (146.8, 39.4)
- moved R27 116.4 mm to (30.5, 34.3)
- moved D16 59.8 mm to (34.3, 21.6), turned to 180 degrees
- moved D12 12.7 mm to (55.9, 25.4), turned to 90 degrees
- moved D14 12.7 mm to (81.3, 25.4), turned to 90 degrees
- moved D15 12.7 mm to (94.0, 25.4), turned to 270 degrees
- moved D13 12.7 mm to (68.6, 25.4), turned to 270 degrees
- moved D11 9.67 mm to (43.2, 25.4), turned to 270 degrees
Connections:
- removed net N$35 (its old number): D15.C, D16.A
- new net N$39: D11.A, D16.C
- net +50V: now also R26.1, R29.1; no longer R27.1, R28.1
- net GND: now also P5.4
- net N$31: now also R29.2; no longer R28.2
- net N$33: now also D15.C; no longer D16.C
- net N$40: now also D16.A; no longer D11.A
- net N$43: now also R27.2; no longer R26.2
- net N$5: now also R26.2; no longer R27.2
- net N$6: now also R28.2; no longer R29.2
- net W_IN: now also R27.1; no longer R26.1
- net Z_IN: now also R28.1; no longer R29.1
Routing:
- net N$35 (its old number): track 12.7 -> 0.00 mm
- net GND: track 246.7 -> 257.2 mm, vias 0 -> 2
- net N$38: track 5.08 -> 12.7 mm
- net N$39: track 0.00 -> 5.08 mm
- net +50V: track 188.5 -> 189.1 mm
