File: yoke/mimic1567.sch (EAGLE design)
At the start: 69 parts, among them J1 COIL 1, J2 LOAD RESISTOR, J6 COIL 1, J7 LOAD RESISTOR, P1 25 K, P2 10 K, P3 200, P4 100 K, P5 20 K, P6 44PINEDGE, P7 20, Q1 2N3904, Q10 2N2907, Q11 MJ10007, Q12 2N3906, Q13 MJ10007, Q2 2N3904, Q3 2N3904, Q4 2N3904, Q5 2N3904, Q6 2N3904, Q7 2N3904, Q8 2N2907, Q9 2N3906

Commit message: modifed amplifier
Parts:
- removed J1: COIL 1, keiths:AWG18
- removed P4: 100 K, keiths:POT-3006P
- removed Q13: MJ10007, keiths:MJ10007
- removed R5: 46.4K, keiths:AXIALRESISTORQUARTER_WATT
- removed R8: 29.4K, keiths:AXIALRESISTORQUARTER_WATT
- added J10, J13: OUT_2, keiths:AWG18
- added J12: COIL 2, keiths:AWG18
- added J14: RESISTOR_2, keiths:AWG18
- added J3, J4: GND, keiths:AWG18
- added J5, J8: OUT_1, keiths:AWG18
- added J9: RESISTOR_1, keiths:AWG18
- added Q14: MJ10007, keiths:MJ10007
- J2: value LOAD RESISTOR -> RESISTOR_2
- J7: value LOAD RESISTOR -> RESISTOR_1
- R20: value 137 K 1% -> 137 1%; PN MFR-25FBF52-137K -> CMF55137R00FHEB
Connections:
- net M_DIFF_IN renamed W_IN
- net P_DIFF_IN renamed Z_IN
- removed net N$1: J1.P$1, Q13.C
- new net N$24: J5.P$1, Q11.B
- new net N$28: J9.P$1, Q11.E
- new net N$32: J12.P$1, Q14.C
- new net N$41: J13.P$1, Q14.B
- new net N$42: J14.P$1, Q14.E
- net GND: now also J3.P$1, J4.P$1; no longer R5.P$1, R8.P$1
- net N$2: no longer Q13.E
- net N$22: no longer P4.A
- net N$27: no longer Q11.E
- net N$31: now also J8.P$1; no longer Q11.B
- net N$4: no longer R5.P$2, R8.P$2
- net N$44: no longer P4.E, P4.S
- net N$5: now also J10.P$1; no longer Q13.B
Other:
- moved on the sheet: C4, C5, C7, J6, J7, P1, P2, P5, P7, Q1, Q11, Q2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

Commit message: working on wire harness
Other:
- moved on the sheet: J12, J13, J14, J2, J5, J6, J9, Q11, Q14
Changed lines of the file:
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@@
 <attribute name="PN" x="307.34" y="228.6" size="1.778" layer="96" rot="MR0" display="off"/>
 </instance>
-<instance part="J2" gate="G$1" x="474.98" y="218.44" smashed="yes">
-<attribute name="NAME" x="470.916" y="221.996" size="1.9304" layer="95" font="vector" ratio="10"/>
-<attribute name="VALUE" x="470.662" y="213.106" size="1.9304" layer="96" font="vector" ratio="10"/>
+<instance part="J2" gate="G$1" x="474.98" y="223.52" smashed="yes">
+<attribute name="NAME" x="473.456" y="227.076" size="1.9304" layer="95" font="vector" ratio="10"/>
+<attribute name="VALUE" x="460.502" y="218.186" size="1.9304" layer="96" font="vector" ratio="10"/>
 </instance>
 <instance part="R2" gate="G$1" x="434.34" y="256.54">
@@
 <attribute name="PN" x="215.9" y="152.4" size="1.778" layer="96" display="off"/>
 </instance>
-<instance part="Q11" gate="G$1" x="226.06" y="60.96" rot="MR0">
-<attribute name="PN" x="226.06" y="60.96" size="1.778" layer="96" rot="MR0" display="off"/>
-</instance>
-<instance part="J6" gate="G$1" x="200.66" y="73.66" rot="MR0"/>
+<instance part="Q11" gate="G$1" x="68.58" y="238.76" rot="MR0">
+<attribute name="PN" x="68.58" y="238.76" size="1.778" layer="96" rot="MR0" display="off"/>
+</instance>
+<instance part="J6" gate="G$1" x="83.82" y="254" smashed="yes" rot="MR180">
+<attribute name="NAME" x="82.55" y="257.556" size="1.9304" layer="95" font="vector" ratio="10"/>
+<attribute name="VALUE" x="80.518" y="248.666" size="1.9304" layer="96" font="vector" ratio="10"/>
+</instance>
 <instance part="J7" gate="G$1" x="93.98" y="223.52" smashed="yes" rot="MR0">
-<attribute name="NAME" x="98.044" y="227.076" size="1.9304" layer="95" font="vector" ratio="10" rot="MR0"/>
-<attribute name="VALUE" x="89.662" y="218.694" size="1.9304" layer="96" font="vector" ratio="10" rot="MR180"/>
+<attribute name="NAME" x="92.964" y="227.076" size="1.9304" layer="95" font="vector" ratio="10"/>
+<attribute name="VALUE" x="90.678" y="218.186" size="1.9304" layer="96" font="vector" ratio="10"/>
 </instance>
 <instance part="R16" gate="G$1" x="149.86" y="137.16">
@@
 <instance part="J3" gate="G$1" x="93.98" y="147.32" rot="MR0"/>
 <instance part="J4" gate="G$1" x="472.44" y="162.56"/>
-<instance part="J5" gate="G$1" x="238.76" y="60.96" smashed="yes">
-<attribute name="NAME" x="242.316" y="61.976" size="1.9304" layer="95" font="vector" ratio="10"/>
-<attribute name="VALUE" x="242.062" y="58.166" size="1.9304" layer="96" font="vector" ratio="10"/>
+<instance part="J5" gate="G$1" x="83.82" y="238.76" smashed="yes">
+<attribute name="NAME" x="82.296" y="242.316" size="1.9304" layer="95" font="vector" ratio="10"/>
+<attribute name="VALUE" x="79.502" y="233.426" size="1.9304" layer="96" font="vector" ratio="10"/>
 </instance>
 <instance part="J8" gate="G$1" x="93.98" y="238.76" smashed="yes" rot="MR0">
-<attribute name="NAME" x="82.804" y="239.776" size="1.9304" layer="95" font="vector" ratio="10"/>
-<attribute name="VALUE" x="83.058" y="235.966" size="1.9304" layer="96" font="vector" ratio="10"/>
-</instance>
-<instance part="J9" gate="G$1" x="238.76" y="50.8" smashed="yes">
-<attribute name="NAME" x="242.316" y="51.816" size="1.9304" layer="95" font="vector" ratio="10"/>
-<attribute name="VALUE" x="242.062" y="48.006" size="1.9304" layer="96" font="vector" ratio="10"/>
+<attribute name="NAME" x="92.964" y="242.316" size="1.9304" layer="95" font="vector" ratio="10"/>
+<attribute name="VALUE" x="90.678" y="233.426" size="1.9304" layer="96" font="vector" ratio="10"/>
+</instance>
+<instance part="J9" gate="G$1" x="83.82" y="223.52" smashed="yes">
+<attribute name="NAME" x="82.296" y="227.076" size="1.9304" layer="95" font="vector" ratio="10"/>
+<attribute name="VALUE" x="69.342" y="218.186" size="1.9304" layer="96" font="vector" ratio="10"/>
 </instance>
 <instance part="J10" gate="G$1" x="474.98" y="238.76" smashed="yes">
-<attribute name="NAME" x="478.536" y="239.776" size="1.9304" layer="95" font="vector" ratio="10"/>
-<attribute name="VALUE" x="478.282" y="235.966" size="1.9304" layer="96" font="vector" ratio="10"/>
-</instance>
-<instance part="Q14" gate="G$1" x="307.34" y="60.96" rot="MR0">
-<attribute name="PN" x="307.34" y="60.96" size="1.778" layer="96" rot="MR0" display="off"/>
-</instance>
-<instance part="J12" gate="G$1" x="281.94" y="73.66" rot="MR0"/>
-<instance part="J13" gate="G$1" x="320.04" y="60.96" smashed="yes">
-<attribute name="NAME" x="323.596" y="61.976" size="1.9304" layer="95" font="vector" ratio="10"/>
-<attribute name="VALUE" x="323.342" y="58.166" size="1.9304" layer="96" font="vector" ratio="10"/>
-</instance>
-<instance part="J14" gate="G$1" x="320.04" y="50.8" smashed="yes">
-<attribute name="NAME" x="323.596" y="51.816" size="1.9304" layer="95" font="vector" ratio="10"/>
-<attribute name="VALUE" x="323.342" y="48.006" size="1.9304" layer="96" font="vector" ratio="10"/>
+<attribute name="NAME" x="472.44" y="242.316" size="1.9304" layer="95" font="vector" ratio="10"/>
+<attribute name="VALUE" x="469.138" y="233.426" size="1.9304" layer="96" font="vector" ratio="10"/>
+</instance>
+<instance part="Q14" gate="G$1" x="502.92" y="238.76">
+<attribute name="PN" x="502.92" y="238.76" size="1.778" layer="96" display="off"/>
+</instance>
+<instance part="J12" gate="G$1" x="487.68" y="254" smashed="yes" rot="MR0">
+<attribute name="NAME" x="485.14" y="257.556" size="1.9304" layer="95" font="vector" ratio="10"/>
+<attribute name="VALUE" x="484.378" y="248.666" size="1.9304" layer="96" font="vector" ratio="10"/>
+</instance>
+<instance part="J13" gate="G$1" x="487.68" y="238.76" smashed="yes" rot="MR0">
+<attribute name="NAME" x="485.14" y="242.062" size="1.9304" layer="95" font="vector" ratio="10"/>
+<attribute name="VALUE" x="485.14" y="233.426" size="1.9304" layer="96" font="vector" ratio="10"/>
+</instance>
+<instance part="J14" gate="G$1" x="487.68" y="223.52" smashed="yes" rot="MR0">
+<attribute name="NAME" x="485.394" y="227.076" size="1.9304" layer="95" font="vector" ratio="10"/>
+<attribute name="VALUE" x="485.394" y="218.186" size="1.9304" layer="96" font="vector" ratio="10"/>
 </instance>
 </instances>
@@
 <segment>
 <pinref part="J2" gate="G$1" pin="P$1"/>
-<wire x1="467.36" y1="218.44" x2="449.58" y2="218.44" width="0.1524" layer="91"/>
-<wire x1="449.58" y1="213.36" x2="449.58" y2="218.44" width="0.1524" layer="91"/>
+<wire x1="467.36" y1="223.52" x2="449.58" y2="223.52" width="0.1524" layer="91"/>
+<wire x1="449.58" y1="213.36" x2="449.58" y2="223.52" width="0.1524" layer="91"/>
 <pinref part="C1" gate="G$1" pin="1"/>
 </segment>
@@
 <segment>
 <pinref part="J6" gate="G$1" pin="P$1"/>
-<wire x1="208.28" y1="73.66" x2="220.98" y2="73.66" width="0.1524" layer="91"/>
+<wire x1="76.2" y1="254" x2="63.5" y2="254" width="0.1524" layer="91"/>
 <pinref part="Q11" gate="G$1" pin="C"/>
-<wire x1="220.98" y1="73.66" x2="220.98" y2="66.04" width="0.1524" layer="91"/>
+<wire x1="63.5" y1="254" x2="63.5" y2="243.84" width="0.1524" layer="91"/>
 </segment>
 </net>
@@
 <pinref part="R11" gate="G$1" pin="P$1"/>
 <pinref part="J3" gate="G$1" pin="P$1"/>
-<wire x1="101.6" y1="147.32" x2="114.3" y2="147.32" width="0.1524" layer="91"/>
+<wire x1="101.6" y1="147.32" x2="109.22" y2="147.32" width="0.1524" layer="91"/>
+<wire x1="109.22" y1="147.32" x2="114.3" y2="147.32" width="0.1524" layer="91"/>
 <wire x1="114.3" y1="147.32" x2="114.3" y2="162.56" width="0.1524" layer="91"/>
 <junction x="114.3" y="162.56"/>
@@
 <wire x1="215.9" y1="157.48" x2="215.9" y2="162.56" width="0.1524" layer="91"/>
 <junction x="215.9" y="162.56"/>
+<wire x1="96.52" y1="147.32" x2="109.22" y2="147.32" width="0.1524" layer="91"/>
 </segment>
 </net>
@@
 <pinref part="Q11" gate="G$1" pin="B"/>
 <pinref part="J5" gate="G$1" pin="P$1"/>
-<wire x1="231.14" y1="60.96" x2="228.6" y2="60.96" width="0.1524" layer="91"/>
+<wire x1="76.2" y1="238.76" x2="71.12" y2="238.76" width="0.1524" layer="91"/>
 </segment>
 </net>
@@
 <segment>
 <pinref part="Q11" gate="G$1" pin="E"/>
-<wire x1="220.98" y1="50.8" x2="220.98" y2="53.34" width="0.1524" layer="91"/>
+<wire x1="63.5" y1="223.52" x2="63.5" y2="231.14" width="0.1524" layer="91"/>
 <pinref part="J9" gate="G$1" pin="P$1"/>
-<wire x1="231.14" y1="50.8" x2="220.98" y2="50.8" width="0.1524" layer="91"/>
+<wire x1="76.2" y1="223.52" x2="63.5" y2="223.52" width="0.1524" layer="91"/>
 </segment>
 </net>
@@
 <segment>
 <pinref part="J12" gate="G$1" pin="P$1"/>
-<wire x1="289.56" y1="73.66" x2="302.26" y2="73.66" width="0.1524" layer="91"/>
+<wire x1="495.3" y1="254" x2="508" y2="254" width="0.1524" layer="91"/>
 <pinref part="Q14" gate="G$1" pin="C"/>
-<wire x1="302.26" y1="73.66" x2="302.26" y2="66.04" width="0.1524" layer="91"/>
+<wire x1="508" y1="254" x2="508" y2="243.84" width="0.1524" layer="91"/>
 </segment>
 </net>
@@
 <pinref part="Q14" gate="G$1" pin="B"/>
 <pinref part="J13" gate="G$1" pin="P$1"/>
-<wire x1="312.42" y1="60.96" x2="309.88" y2="60.96" width="0.1524" layer="91"/>
+<wire x1="495.3" y1="238.76" x2="500.38" y2="238.76" width="0.1524" layer="91"/>
 </segment>
 </net>
@@
 <segment>
 <pinref part="Q14" gate="G$1" pin="E"/>
-<wire x1="302.26" y1="50.8" x2="302.26" y2="53.34" width="0.1524" layer="91"/>
+<wire x1="508" y1="223.52" x2="508" y2="231.14" width="0.1524" layer="91"/>
 <pinref part="J14" gate="G$1" pin="P$1"/>
-<wire x1="312.42" y1="50.8" x2="302.26" y2="50.8" width="0.1524" layer="91"/>
-</segment>
-</net>
+<wire x1="495.3" y1="223.52" x2="508" y2="223.52" width="0.1524" layer="91"/>
+</segment>
+</net>

Commit message: more work
Parts:
- removed J10, J13: OUT_2, keiths:AWG18
- removed J12: COIL 2, keiths:AWG18
- removed J14, J2: RESISTOR_2, keiths:AWG18
- removed J4: GND, keiths:AWG18
- removed J5, J8: OUT_1, keiths:AWG18
- removed J6: COIL 1, keiths:AWG18
- removed J7, J9: RESISTOR_1, keiths:AWG18
- removed P3: 200, keiths:POT-3006P
- removed P7: 20, keiths:POT-3006P
- removed Q11, Q14: MJ10007, keiths:MJ10007
- added J15: JST-VH-5, keiths:JST-VH-5
- added P4: 20 K, keiths:POT-3006P
- added R24: 2 K 1%, keiths:AXIALRESISTORQUARTER_WATT
- added R26: 274 K 1%, keiths:AXIALRESISTORQUARTER_WATT
- P5: value 20 K -> 200; PN 3006P-1-203LF -> 3006P-1-201LF
- R23: value 274 K 1% -> 2 K 1%; PN MFR-25FBF52-274K -> MFR-25FRF52-2K
Connections:
- removed net N$18: P5.A, P7.E, P7.S, R21.P$2
- removed net N$24: J5.P$1, Q11.B
- removed net N$26: J6.P$1, Q11.C
- removed net N$28: J9.P$1, Q11.E
- removed net N$32: J12.P$1, Q14.C
- removed net N$41: J13.P$1, Q14.B
- removed net N$42: J14.P$1, Q14.E
- net GND: now also J15.5; no longer J4.P$1
- net N$2: now also J15.4, R24.P$2; no longer J2.P$1
- net N$22: now also P5.A, R26.P$1; no longer P3.A, R23.P$1
- net N$27: now also J15.2, R23.P$1; no longer J7.P$1
- net N$31: now also J15.1; no longer J8.P$1
- net N$43: now also R21.P$2, R23.P$2; no longer R19.P$2
- net N$44: now also P5.E; no longer P3.E
- net N$5: now also J15.3; no longer J10.P$1
- net N$6: now also R19.P$2, R24.P$1; no longer R21.P$1
- net W_IN: now also P4.E, P4.S, R21.P$1, R26.P$2; no longer P3.S, P5.E, R19.P$1, R23.P$2
- net Z_IN: now also P4.A, R19.P$1; no longer P7.A
Other:
- moved on the sheet: C1, C4, C5, C7, J3, P1, P2, P5, P6, Q1, Q2, Q4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

Commit message: more changes
Parts:
- removed J3: GND, keiths:AWG18
Connections:
- removed net -150V: P6.V
- removed net CATHODE: P6.Z
- removed net J_IN: P6.J
- removed net P_IN: P6.P
- removed net U_IN: P6.U
- removed net X_IN: P6.X
- net GND: no longer J3.P$1
- net W_IN: now also P6.W
- net Z_IN: now also P6.Z
Other:
- moved on the sheet: J15, P6, R19, R21

Commit message: update netlist
Connections:
- removed net +10V: P6.A
- removed net +5V: P6.F
- removed net -15V: P6.C
- net +50V: now also P6.M; no longer P6.E
- net -10V: now also P6.E
Other:
- moved on the sheet: P4, P6
Changed lines of the file:
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@@
 <attribute name="PN" x="165.1" y="101.6" size="1.778" layer="96" display="off"/>
 </instance>
-<instance part="P6" gate="G$1" x="208.28" y="335.28"/>
+<instance part="P6" gate="G$1" x="294.64" y="353.06"/>
 <instance part="R1" gate="G$1" x="391.16" y="129.54">
 <attribute name="PN" x="391.16" y="129.54" size="1.778" layer="96" display="off"/>
@@
 </instance>
 <instance part="SUPPLY2" gate="GND" x="403.86" y="106.68"/>
-<instance part="P4" gate="G$1" x="81.28" y="185.42" smashed="yes" rot="R90">
-<attribute name="NAME" x="84.328" y="192.278" size="1.9304" layer="95" font="vector" ratio="10" rot="R270"/>
-<attribute name="VALUE" x="84.328" y="182.372" size="1.9304" layer="96" font="vector" ratio="10" rot="R270"/>
-<attribute name="PN" x="81.28" y="185.42" size="1.778" layer="96" rot="R90" display="off"/>
+<instance part="P4" gate="G$1" x="182.88" y="185.42" smashed="yes" rot="R90">
+<attribute name="NAME" x="185.928" y="192.278" size="1.9304" layer="95" font="vector" ratio="10" rot="R270"/>
+<attribute name="VALUE" x="185.928" y="182.372" size="1.9304" layer="96" font="vector" ratio="10" rot="R270"/>
+<attribute name="PN" x="182.88" y="185.42" size="1.778" layer="96" rot="R90" display="off"/>
 </instance>
 <instance part="R21" gate="G$1" x="210.82" y="198.12" smashed="yes" rot="R90">
@@
 <pinref part="C5" gate="G$1" pin="1"/>
 </segment>
+<segment>
+<pinref part="P6" gate="G$1" pin="E"/>
+<wire x1="304.8" y1="368.3" x2="332.74" y2="368.3" width="0.1524" layer="91"/>
+<label x="332.74" y="368.3" size="1.9304" layer="95" font="vector" ratio="10" xref="yes"/>
+</segment>
 </net>
 <net name="N$22" class="0">
@@
 <pinref part="R17" gate="G$1" pin="P$2"/>
 <wire x1="165.1" y1="154.94" x2="165.1" y2="160.02" width="0.1524" layer="91"/>
-<wire x1="81.28" y1="198.12" x2="198.12" y2="198.12" width="0.1524" layer="91"/>
 <pinref part="P4" gate="G$1" pin="E"/>
-<wire x1="81.28" y1="193.04" x2="81.28" y2="198.12" width="0.1524" layer="91"/>
-<junction x="81.28" y="198.12"/>
-<wire x1="91.44" y1="198.12" x2="81.28" y2="198.12" width="0.1524" layer="91"/>
-<wire x1="91.44" y1="185.42" x2="91.44" y2="198.12" width="0.1524" layer="91"/>
+<wire x1="165.1" y1="198.12" x2="83.82" y2="198.12" width="0.1524" layer="91"/>
+<wire x1="190.5" y1="185.42" x2="190.5" y2="198.12" width="0.1524" layer="91"/>
 <pinref part="P4" gate="G$1" pin="S"/>
-<wire x1="86.36" y1="185.42" x2="91.44" y2="185.42" width="0.1524" layer="91"/>
-<label x="198.12" y="198.12" size="1.9304" layer="95" font="vector" ratio="10" xref="yes"/>
+<wire x1="187.96" y1="185.42" x2="190.5" y2="185.42" width="0.1524" layer="91"/>
+<label x="83.82" y="198.12" size="1.9304" layer="95" font="vector" ratio="10" rot="R180" xref="yes"/>
 <pinref part="R21" gate="G$1" pin="P$1"/>
-<junction x="91.44" y="198.12"/>
-<wire x1="205.74" y1="198.12" x2="165.1" y2="198.12" width="0.1524" layer="91"/>
+<junction x="190.5" y="198.12"/>
+<wire x1="205.74" y1="198.12" x2="190.5" y2="198.12" width="0.1524" layer="91"/>
 <pinref part="R26" gate="G$1" pin="P$2"/>
-<wire x1="165.1" y1="198.12" x2="91.44" y2="198.12" width="0.1524" layer="91"/>
+<wire x1="165.1" y1="198.12" x2="182.88" y2="198.12" width="0.1524" layer="91"/>
+<wire x1="182.88" y1="198.12" x2="190.5" y2="198.12" width="0.1524" layer="91"/>
 <wire x1="233.68" y1="154.94" x2="233.68" y2="160.02" width="0.1524" layer="91"/>
 <pinref part="P5" gate="G$1" pin="S"/>
@@
 <junction x="165.1" y="160.02"/>
 <junction x="165.1" y="198.12"/>
-</segment>
-<segment>
-<wire x1="218.44" y1="314.96" x2="246.38" y2="314.96" width="0.1524" layer="91"/>
-<label x="246.38" y="314.96" size="1.9304" layer="95" font="vector" ratio="10" xref="yes"/>
+<wire x1="182.88" y1="193.04" x2="182.88" y2="198.12" width="0.1524" layer="91"/>
+<junction x="182.88" y="198.12"/>
+</segment>
+<segment>
+<wire x1="304.8" y1="332.74" x2="332.74" y2="332.74" width="0.1524" layer="91"/>
+<label x="332.74" y="332.74" size="1.9304" layer="95" font="vector" ratio="10" xref="yes"/>
 <pinref part="P6" gate="G$1" pin="W"/>
 </segment>
@@
 <net name="Z_IN" class="0">
 <segment>
-<label x="198.12" y="172.72" size="1.9304" layer="95" font="vector" ratio="10" rot="MR180" xref="yes"/>
-<wire x1="81.28" y1="172.72" x2="198.12" y2="172.72" width="0.1524" layer="91"/>
+<label x="83.82" y="172.72" size="1.9304" layer="95" font="vector" ratio="10" rot="MR0" xref="yes"/>
 <pinref part="P4" gate="G$1" pin="A"/>
-<wire x1="81.28" y1="177.8" x2="81.28" y2="172.72" width="0.1524" layer="91"/>
-<junction x="81.28" y="172.72"/>
 <pinref part="R19" gate="G$1" pin="P$1"/>
-<wire x1="205.74" y1="172.72" x2="81.28" y2="172.72" width="0.1524" layer="91"/>
-</segment>
-<segment>
-<label x="246.38" y="307.34" size="1.9304" layer="95" font="vector" ratio="10" rot="MR180" xref="yes"/>
-<wire x1="218.44" y1="307.34" x2="246.38" y2="307.34" width="0.1524" layer="91"/>
+<wire x1="205.74" y1="172.72" x2="182.88" y2="172.72" width="0.1524" layer="91"/>
+<wire x1="182.88" y1="172.72" x2="83.82" y2="172.72" width="0.1524" layer="91"/>
+<wire x1="182.88" y1="177.8" x2="182.88" y2="172.72" width="0.1524" layer="91"/>
+<junction x="182.88" y="172.72"/>
+</segment>
+<segment>
+<label x="332.74" y="325.12" size="1.9304" layer="95" font="vector" ratio="10" rot="MR180" xref="yes"/>
+<wire x1="304.8" y1="325.12" x2="332.74" y2="325.12" width="0.1524" layer="91"/>
 <pinref part="P6" gate="G$1" pin="Z"/>
 </segment>
@@
 <segment>
 <pinref part="P6" gate="G$1" pin="D"/>
-<wire x1="218.44" y1="353.06" x2="226.06" y2="353.06" width="0.1524" layer="91"/>
-<label x="226.06" y="353.06" size="1.9304" layer="95" font="vector" ratio="10" xref="yes"/>
+<wire x1="304.8" y1="370.84" x2="312.42" y2="370.84" width="0.1524" layer="91"/>
+<label x="312.42" y="370.84" size="1.9304" layer="95" font="vector" ratio="10" xref="yes"/>
 </segment>
 <segment>
@@
 </segment>
 </net>
-<net name="-15V" class="0">
-<segment>
-<pinref part="P6" gate="G$1" pin="C"/>
-<wire x1="218.44" y1="355.6" x2="246.38" y2="355.6" width="0.1524" layer="91"/>
-<label x="246.38" y="355.6" size="1.9304" layer="95" font="vector" ratio="10" xref="yes"/>
-</segment>
-</net>
-<net name="+5V" class="0">
-<segment>
-<pinref part="P6" gate="G$1" pin="F"/>
-<wire x1="218.44" y1="347.98" x2="226.06" y2="347.98" width="0.1524" layer="91"/>
-<label x="226.06" y="347.98" size="1.9304" layer="95" font="vector" ratio="10" xref="yes"/>
-</segment>
-</net>
-<net name="+10V" class="0">
-<segment>
-<pinref part="P6" gate="G$1" pin="A"/>
-<wire x1="218.44" y1="360.68" x2="246.38" y2="360.68" width="0.1524" layer="91"/>
-<label x="246.38" y="360.68" size="1.9304" layer="95" font="vector" ratio="10" xref="yes"/>
-</segment>
-</net>
 <net name="+50V" class="0">
 <segment>
-<pinref part="P6" gate="G$1" pin="E"/>
-<wire x1="218.44" y1="350.52" x2="246.38" y2="350.52" width="0.1524" layer="91"/>
-<label x="246.38" y="350.52" size="1.9304" layer="95" font="vector" ratio="10" xref="yes"/>
-</segment>
-<segment>
+<label x="332.74" y="353.06" size="1.9304" layer="95" font="vector" ratio="10" xref="yes"/>
+<pinref part="P6" gate="G$1" pin="M"/>
+<wire x1="304.8" y1="353.06" x2="332.74" y2="353.06" width="0.1524" layer="91"/>
+</segment>
+<segment>
