File: yoke/mimic1567.sch (EAGLE design)
At the start: 62 parts, among them J15 JST-VH-5, P1 25 K, P2 10 K, P4 20 K, P5 200, P6 44PINEDGE, Q1 2N3904, Q10 2N2907, Q12 2N3906, Q2 2N3904, Q3 2N3904, Q4 2N3904, Q5 2N3904, Q6 2N3904, Q7 2N3904, Q8 2N2907, Q9 2N3906

Commit message: preamplifier card being routed
Parts:
- removed C7: 0.022 uF, keiths:ECQ-E2223JF
- removed P6: 44PINEDGE, keiths:44PINEDGE
- removed Q12: 2N3906, keiths:2N3906
- removed R26: 274 K 1%, keiths:AXIALRESISTORQUARTER_WATT
- added C2: 0.022 uF, keiths:ECQ-E2223JF
- added P3: 10 K, keiths:POT-3006P
- added Q11: 2N2907, keiths:2N2907
- added R25: 330, keiths:AXIALRESISTORONE_WATT
- added R5: 10K, keiths:AXIALRESISTORQUARTER_WATT
- added R8: 25K, keiths:AXIALRESISTORQUARTER_WATT
- C1: value 3.3UF 5% -> 3.3uF
- C3, C6: value 0.022 uF -> 0.022uF
- C4: value 3.3UF 5% -> 0.022uF; device keiths:ECQ-E2335JF -> keiths:ECQ-E2223JF; PN ECQ-E2335JF -> ECQ-E2223JFB
- C5: value 0.022 uF -> 3.3uF; device keiths:ECQ-E2223JF -> keiths:ECQ-E2335JF; PN ECQ-E2223JFB -> ECQ-E2335JF
- P1: value 25 K -> 20K; PN 3006P-1-253LF -> 3006P-1-203LF
- P2: value 10 K -> 25 K; PN 3006P-1-103LF -> 3006P-1-253LF
- P4: value 20 K -> 200; PN 3006P-1-203LF -> 3006P-1-201LF
- P5: value 200 -> 44PINEDGE; device keiths:POT-3006P -> keiths:44PINEDGE; PN 3006P-1-201LF -> (none)
- Q10: value 2N2907 -> 2N3904; device keiths:2N2907 -> keiths:2N3904; PN 2N2907A -> 2N3904
- Q4: value 2N3904 -> 2N2907; device keiths:2N3904 -> keiths:2N2907; PN 2N3904 -> 2N2907A
- Q5: value 2N3904 -> 2N3906; device keiths:2N3904 -> keiths:2N3906; PN 2N3904 -> 2N3906
- Q8: value 2N2907 -> 2N3906; device keiths:2N2907 -> keiths:2N3906; PN 2N2907A -> 2N3906
- Q9: value 2N3906 -> 2N3904; device keiths:2N3906 -> keiths:2N3904; PN 2N3906 -> 2N3904
- R1: value 3.3uF -> 274K; device keiths:AXIALRESISTORTHREE_WATT -> keiths:AXIALRESISTORQUARTER_WATT; PN ECQ-E2335JF -> MFR-25FBF52-274K
- R10: value 33.2 K 1% -> 274K; device keiths:AXIALRESISTORHALF_WATT -> keiths:AXIALRESISTORQUARTER_WATT; PN SFR16S0003322FR500 -> MFR-25FBF52-274K
- R11: value 4.64K -> 6.81K 1%; device keiths:AXIALRESISTORQUARTER_WATT -> keiths:AXIALRESISTORHALF_WATT; PN RNF14FTD4K64 -> MFS1/2DCT52R6811F
- R12: value 2.94K -> 33.2K; device keiths:AXIALRESISTORQUARTER_WATT -> keiths:AXIALRESISTORHALF_WATT; PN RNF14FTD2K94 -> SFR16S0003322FR500
- R13: value 3.3 -> 2K; device keiths:AXIALRESISTORTHREE_WATT -> keiths:AXIALRESISTORQUARTER_WATT; PN PR03000203308JAC00 -> MFR-25FRF52-2K
- R14: value 1.96 K 1 % -> 10K; device keiths:AXIALRESISTORQUARTER_WATT -> keiths:AXIALRESISTORHALF_WATT; PN RNF14FTD1K96 -> MF1/2LCT52R103J
- R15: value 330 5% -> 3.3K; device keiths:AXIALRESISTORONE_WATT -> keiths:AXIALRESISTORTWO_WATT; PN SFR16S0003300JA500 -> RR02J3K3TB
- R16: value 10 K 5% -> 6.81K; PN MF1/2LCT52R103J -> MFS1/2DCT52R6811F
- R17: value 274 K 1% -> 33.2K; device keiths:AXIALRESISTORQUARTER_WATT -> keiths:AXIALRESISTORHALF_WATT; PN MFR-25FBF52-274K -> SFR16S0003322FR500
- R18: value 1.96 K 1 % -> 2K; PN RNF14FTD1K96 -> MFR-25FRF52-2K
- R19: value 1 K 1% -> 10K; device keiths:AXIALRESISTORQUARTER_WATT -> keiths:AXIALRESISTORHALF_WATT; PN MFR-25FRF52-1K -> MF1/2LCT52R103J
- R2: value 3.3K 5% -> 137; device keiths:AXIALRESISTORTWO_WATT -> keiths:AXIALRESISTORQUARTER_WATT; PN RR02J3K3TB -> CMF55137R00FHEB
- R20: value 137 1% -> 3.3K; device keiths:AXIALRESISTORQUARTER_WATT -> keiths:AXIALRESISTORTWO_WATT; PN CMF55137R00FHEB -> RR02J3K3TB
- R21: value 1 K 1% -> 3.3; device keiths:AXIALRESISTORQUARTER_WATT -> keiths:AXIALRESISTORTHREE_WATT; PN MFR-25FRF52-1K -> PR03000203308JAC00
- R22: value 330 5% -> 1K; device keiths:AXIALRESISTORONE_WATT -> keiths:AXIALRESISTORQUARTER_WATT; PN SFR16S0003300JA500 -> MFR-25FRF52-1K
- R23: value 2 K 1% -> 1K; PN MFR-25FRF52-2K -> MFR-25FRF52-1K
- R24: value 2 K 1% -> 330; device keiths:AXIALRESISTORQUARTER_WATT -> keiths:AXIALRESISTORONE_WATT; PN MFR-25FRF52-2K -> SFR16S0003300JA500
- R3: value 3.3K 5% -> 1.96K; device keiths:AXIALRESISTORTWO_WATT -> keiths:AXIALRESISTORQUARTER_WATT; PN RR02J3K3TB -> RNF14FTD1K96
- R4: value 10 K 5% -> 10K; device keiths:AXIALRESISTORHALF_WATT -> keiths:AXIALRESISTORQUARTER_WATT; PN MF1/2LCT52R103J -> RNF14FTD2K94
- R6: value 6.81K 1% -> 1.96K; device keiths:AXIALRESISTORHALF_WATT -> keiths:AXIALRESISTORQUARTER_WATT; PN MFS1/2DCT52R6811F -> RNF14FTD1K96
- R7: value 33.2 K 1% -> 25K; device keiths:AXIALRESISTORHALF_WATT -> keiths:AXIALRESISTORQUARTER_WATT; PN SFR16S0003322FR500 -> RNF14FTD2K94
- R9: value 6.81K 1% -> 3.3uF; device keiths:AXIALRESISTORHALF_WATT -> keiths:AXIALRESISTORTHREE_WATT; PN MFS1/2DCT52R6811F -> ECQ-E2335JF
- renumbered J15 to J1
Connections:
- removed net N$13 (its old number): D11.A, D12.C
- removed net N$23: Q5.E
- new net N$37: D12.C, D13.A
- net +50V: now also P5.M, R11.P$1, R15.P$1, R16.P$1, R20.P$1; no longer P6.M, R2.P$1, R3.P$1, R6.P$1, R9.P$1
- net -10V: now also C3.1, C4.1, P5.E, Q3.E, Q9.E, R14.P$2, R19.P$2, R24.P$2, R25.P$2, R6.P$2; no longer C5.1, C7.1, P6.E, Q4.E, R15.P$2, R16.P$2, R18.P$2, R22.P$2, R4.P$2
- net GND: now also P2.2, P2.3, P3.2, P3.3, P5.D, R21.P$2, R3.P$2, R4.P$1, R5.P$1, R7.P$1, R8.P$1, R9.P$2; no longer P1.E, P1.S, P2.E, P2.S, P6.D, R1.P$2, R11.P$1, R12.P$1, R13.P$2, R14.P$2
- net N$10: now also D2.C, D6.A; no longer D14.A, D15.C
- net N$11: now also D1.C, D2.A; no longer D13.A, D14.C
- net N$12: now also D1.A, D4.C; no longer D12.A, D13.C
- net N$14: now also D3.C, D5.A; no longer D10.A, D11.C
- net N$15: now also C2.1, D3.A, Q5.E; no longer C3.1, D10.C, Q9.E
- net N$16: now also Q5.B, Q7.C, R12.P$2; no longer Q3.C, Q9.B, R7.P$2
- net N$17: now also R11.P$2, R12.P$1; no longer R7.P$1, R9.P$2
- net N$19: now also Q1.C, Q10.E; no longer Q3.E, Q5.C
- net N$2: now also R13.P$2; no longer R24.P$2
- net N$20: now also R16.P$2, R17.P$1; no longer R10.P$1, R6.P$2
- net N$21: now also Q5.C; no longer Q2.C
- net N$22: now also P4.1, R10.P$1, R2.P$2, R3.P$1; no longer P5.A, R14.P$1, R20.P$2, R26.P$1
- net N$25: now also Q10.C, Q8.B, R17.P$2; no longer Q12.B, Q7.C, R10.P$2
- net N$27: now also C5.1, R18.P$1; no longer C4.1, R23.P$1
- net N$29: now also P3.1, Q1.B, Q2.B, Q2.C, R4.P$2, R5.P$2; no longer P2.A, Q5.B, Q6.B, Q6.C, R11.P$2, R12.P$2
- net N$3: now also R9.P$1; no longer R1.P$1
- net N$30: now also C5.2, R21.P$1; no longer C4.2, R13.P$1
- net N$31: now also D16.C, Q11.E, R20.P$2; no longer D2.C, Q10.E, R3.P$2
- net N$33: now also D15.C, D16.A, Q11.B, R19.P$1; no longer D1.C, D2.A, Q10.B, R16.P$1
- net N$34: now also C4.2, Q11.C, R24.P$1; no longer C7.2, Q10.C, R15.P$1
- net N$35: now also D14.C, D15.A; no longer D1.A, D3.C
- net N$36: now also D13.C, D14.A; no longer D3.A, D4.C
- net N$38: now also D11.C, D12.A; no longer D5.A, D6.C
- net N$39: now also D10.C, D11.A; no longer D6.A, D7.C
- net N$4: now also P2.1, Q3.B, Q6.B, Q6.C, Q9.B, R7.P$2, R8.P$2; no longer P1.A, Q1.B, Q1.C, Q2.B, Q4.B
- net N$40: now also D10.A, Q8.E; no longer D7.A, Q12.E
- net N$43: now also Q10.B, R18.P$2, R22.P$2; no longer Q7.B, R21.P$2, R23.P$2
- net N$44: now also P4.3, R1.P$1, R2.P$1, R6.P$1; no longer P5.E, R17.P$1, R18.P$1, R20.P$1
- net N$5: now also D7.C, Q4.E, R15.P$2; no longer D16.A, Q8.E, R2.P$2
- net N$6: now also Q7.B, R13.P$1, R23.P$2; no longer Q3.B, R19.P$2, R24.P$1
- net N$7: now also C2.2, D6.C, D7.A, Q4.B, R14.P$1; no longer C3.2, D15.A, D16.C, Q8.B, R4.P$1
- net N$8: now also C3.2, Q4.C, R25.P$1; no longer C5.2, Q8.C, R22.P$1
- net N$9: now also Q3.C, Q8.C; no longer Q12.C, Q4.C
- net W_IN: now also P1.2, P1.3, P4.2, P5.W, R1.P$2, R10.P$2, R22.P$1; no longer P4.E, P4.S, P5.S, P6.W, R17.P$2, R21.P$1, R26.P$2
- net Z_IN: now also P1.1, P5.Z, R23.P$1; no longer P4.A, P6.Z, R19.P$1
Other:
- moved on the sheet: C3, C4, C5, C6, D1, D10, D11, D12, D13, D14, D15, D16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

Commit message: D/A being routed
Parts:
- added U$1, U$2: FIDUCIAL, adafruit:FIDUCIAL
- D10: value 1N4148 -> 1N4736A; device keiths:1N4148 -> keiths:1N4736A; PN 1N4148 -> 1N4736A
- D9: value 1N4736A -> 1N4148; device keiths:1N4736A -> keiths:1N4148; PN 1N4736A -> 1N4148
- Q1: value 2N3904 -> 2N2907; device keiths:2N3904 -> keiths:2N2907; PN 2N3904 -> 2N2907A
- Q4: value 2N2907 -> 2N3904; device keiths:2N2907 -> keiths:2N3904; PN 2N2907A -> 2N3904
- R10: value 274K -> 3.3uF; device keiths:AXIALRESISTORQUARTER_WATT -> keiths:AXIALRESISTORTHREE_WATT; PN MFR-25FBF52-274K -> ECQ-E2335JF
- R11: value 6.81K 1% -> 6.81K
- R13: value 2K -> 10K; device keiths:AXIALRESISTORQUARTER_WATT -> keiths:AXIALRESISTORHALF_WATT; PN MFR-25FRF52-2K -> MF1/2LCT52R103J
- R14: value 10K -> 2K; device keiths:AXIALRESISTORHALF_WATT -> keiths:AXIALRESISTORQUARTER_WATT; PN MF1/2LCT52R103J -> MFR-25FRF52-2K
- R15: value 3.3K -> 6.81K; device keiths:AXIALRESISTORTWO_WATT -> keiths:AXIALRESISTORHALF_WATT; PN RR02J3K3TB -> MFS1/2DCT52R6811F
- R16: value 6.81K -> 33.2K; PN MFS1/2DCT52R6811F -> SFR16S0003322FR500
- R17: value 33.2K -> 3.3K; device keiths:AXIALRESISTORHALF_WATT -> keiths:AXIALRESISTORTWO_WATT; PN SFR16S0003322FR500 -> RR02J3K3TB
- R2: value 137 -> 25K; PN CMF55137R00FHEB -> RNF14FTD2K94
- R20: value 3.3K -> 1K; device keiths:AXIALRESISTORTWO_WATT -> keiths:AXIALRESISTORQUARTER_WATT; PN RR02J3K3TB -> MFR-25FRF52-1K
- R23: value 1K -> 330; device keiths:AXIALRESISTORQUARTER_WATT -> keiths:AXIALRESISTORONE_WATT; PN MFR-25FRF52-1K -> SFR16S0003300JA500
- R25: value 330 -> 3.3K; device keiths:AXIALRESISTORONE_WATT -> keiths:AXIALRESISTORTWO_WATT; PN SFR16S0003300JA500 -> RR02J3K3TB
- R3: value 1.96K -> 25K; PN RNF14FTD1K96 -> RNF14FTD4K64
- R7: value 25K -> 274K; PN RNF14FTD2K94 -> MFR-25FBF52-274K
- R8: value 25K -> 137; PN RNF14FTD4K64 -> CMF55137R00FHEB
- R9: value 3.3uF -> 1.96K; device keiths:AXIALRESISTORTHREE_WATT -> keiths:AXIALRESISTORQUARTER_WATT; PN ECQ-E2335JF -> RNF14FTD1K96
Connections:
- removed net N$14 (its old number): D3.C, D5.A
- removed net N$39 (its old number): D10.C, D11.A
- new net N$11: D4.C, D5.A
- new net N$35: D15.C, D16.A
- net +50V: now also R17.P$1, R25.P$1; no longer R16.P$1, R20.P$1
- net -10V: now also Q4.E, R13.P$2, R23.P$2; no longer Q1.E, R14.P$2, R25.P$2
- net GND: now also R10.P$2, R2.P$1, R3.P$1; no longer R3.P$2, R7.P$1, R8.P$1
- net N$10: now also D5.C; no longer D2.C
- net N$12: now also D3.C, D4.A; no longer D1.A, D4.C
- net N$13: now also D2.C, D3.A; no longer D4.A, D5.C
- net N$15: now also D1.A; no longer D3.A
- net N$19: now also Q3.C; no longer Q1.C
- net N$2: now also R14.P$2; no longer R13.P$2
- net N$20: now also D10.C, R15.P$2, R16.P$1; no longer D9.C, R16.P$2, R17.P$1
- net N$21: now also Q6.C; no longer Q9.C
- net N$22: now also R7.P$1, R8.P$2, R9.P$1; no longer R10.P$1, R2.P$2, R3.P$1
- net N$25: now also R16.P$2; no longer R17.P$2
- net N$29: now also Q3.B, Q4.B, Q4.C; no longer Q1.B, Q2.B, Q2.C
- net N$3: now also R10.P$1; no longer R9.P$1
- net N$31: now also D9.C, R25.P$2; no longer D16.C, R20.P$2
- net N$33: now also D16.C, D9.A; no longer D15.C, D16.A
- net N$4: now also Q2.B, Q2.C, R2.P$2, R3.P$2; no longer Q3.B, Q6.C, R7.P$2, R8.P$2
- net N$40: now also D11.A; no longer D9.A
- net N$43: now also R20.P$2; no longer R22.P$2
- net N$44: now also R8.P$1; no longer R2.P$1
- net N$5: now also Q1.E, R17.P$2; no longer Q4.E, R15.P$2
- net N$6: now also R14.P$1, R22.P$2; no longer R13.P$1, R23.P$2
- net N$7: now also Q1.B, R13.P$1; no longer Q4.B, R14.P$1
- net N$8: now also Q1.C, R23.P$1; no longer Q4.C, R25.P$1
- net N$9: now also Q9.C; no longer Q3.C
- net W_IN: now also R20.P$1, R7.P$2; no longer R10.P$2, R22.P$1
- net Z_IN: now also R22.P$1; no longer R23.P$1
Other:
- moved on the sheet: D1, D11, D12, D13, D14, D15, D16, D2, D3, D4, D5, Q2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

Commit message: end of day
Parts:
- added R26, R27: 1.2K, keiths:R-5WATT
- added R28: 1K, keiths:AXIALRESISTORQUARTER_WATT
- added R29, R30: 330, keiths:AXIALRESISTORONE_WATT
- C2: value 0.022 uF -> 3.3uF; device keiths:ECQ-E2223JF -> keiths:ECQ-E2335JF; PN ECQ-E2223JFB -> ECQ-E2335JF
- C3: value 0.022uF -> 0.022 uF
- C5: value 3.3uF -> 0.022uF; device keiths:ECQ-E2335JF -> keiths:ECQ-E2223JF; PN ECQ-E2335JF -> ECQ-E2223JFB
- P3: value 10 K -> 5K
- R10: value 3.3uF -> 1.96K; device keiths:AXIALRESISTORTHREE_WATT -> keiths:AXIALRESISTORQUARTER_WATT; PN ECQ-E2335JF -> RNF14FTD1K96
- R11: value 6.81K -> 3.3; device keiths:AXIALRESISTORHALF_WATT -> keiths:R-1/2WATT; PN MFS1/2DCT52R6811F -> (none)
- R12: value 33.2K -> 100; device keiths:AXIALRESISTORHALF_WATT -> keiths:AXIALRESISTORQUARTER_WATT; PN SFR16S0003322FR500 -> RNF14FTD2K94
- R13: value 10K -> 22; device keiths:AXIALRESISTORHALF_WATT -> keiths:AXIALRESISTORQUARTER_WATT; PN MF1/2LCT52R103J -> RNF14FTD2K94
- R14: value 2K -> 22; PN MFR-25FRF52-2K -> RNF14FTD2K94
- R17: value 3.3K -> 100; device keiths:AXIALRESISTORTWO_WATT -> keiths:AXIALRESISTORQUARTER_WATT; PN RR02J3K3TB -> RNF14FTD2K94
- R18: value 2K -> 10K; device keiths:AXIALRESISTORQUARTER_WATT -> keiths:AXIALRESISTORHALF_WATT; PN MFR-25FRF52-2K -> MF1/2LCT52R103J
- R19: value 10K -> 2K; device keiths:AXIALRESISTORHALF_WATT -> keiths:AXIALRESISTORQUARTER_WATT; PN MF1/2LCT52R103J -> MFR-25FRF52-2K
- R2, R3: value 25K -> 20K
- R20: value 1K -> 6.81K; device keiths:AXIALRESISTORQUARTER_WATT -> keiths:AXIALRESISTORHALF_WATT; PN MFR-25FRF52-1K -> MFS1/2DCT52R6811F
- R21: value 3.3 -> 33.2K; device keiths:AXIALRESISTORTHREE_WATT -> keiths:AXIALRESISTORHALF_WATT; PN PR03000203308JAC00 -> SFR16S0003322FR500
- R22: value 1K -> 100; PN MFR-25FRF52-1K -> RNF14FTD2K94
- R23: value 330 -> 2K; device keiths:AXIALRESISTORONE_WATT -> keiths:AXIALRESISTORQUARTER_WATT; PN SFR16S0003300JA500 -> MFR-25FRF52-2K
- R24: value 330 -> 10K; device keiths:AXIALRESISTORONE_WATT -> keiths:AXIALRESISTORHALF_WATT; PN SFR16S0003300JA500 -> MF1/2LCT52R103J
- R25: value 3.3K -> 1K; device keiths:AXIALRESISTORTWO_WATT -> keiths:AXIALRESISTORQUARTER_WATT; PN RR02J3K3TB -> MFR-25FRF52-1K
- R4: value 10K -> 3.9K
- R5: value 10K -> 4.7K
- R6: value 1.96K -> 274K; PN RNF14FTD1K96 -> MFR-25FBF52-274K
- R7: value 274K -> 137; PN MFR-25FBF52-274K -> CMF55137R00FHEB
- R8: value 137 -> 1.96K; PN CMF55137R00FHEB -> RNF14FTD1K96
- R9: value 1.96K -> 3.3; device keiths:AXIALRESISTORQUARTER_WATT -> keiths:R-1/2WATT; PN RNF14FTD1K96 -> (none)
Connections:
- new net N$1: Q4.E, R14.P$1
- new net N$18: Q3.E, R13.P$1
- new net N$23: Q9.E, R22.P$1
- new net N$24: Q6.E, R17.P$1
- new net N$26: Q2.E, R12.P$1
- net +50V: now also R20.P$1, R26.P$1, R27.P$1; no longer R11.P$1, R17.P$1, R25.P$1
- net -10V: now also C5.1, R10.P$2, R12.P$2, R14.P$2, R17.P$2, R18.P$2, R22.P$2, R29.P$2, R30.P$2; no longer C3.1, Q2.E, Q3.E, Q4.E, Q6.E, Q9.E, R19.P$2, R23.P$2, R6.P$2
- net GND: now also R11.P$2, R8.P$2; no longer R10.P$2, R21.P$2
- net N$15: now also C3.1; no longer C2.1
- net N$16: now also R16.P$2; no longer R12.P$2
- net N$17: now also R15.P$2, R16.P$1; no longer R11.P$2, R12.P$1
- net N$2: now also C2.1, R19.P$2; no longer C1.1, R14.P$2
- net N$20: now also R20.P$2, R21.P$1; no longer R15.P$2, R16.P$1
- net N$22: now also R6.P$1, R7.P$2, R8.P$1; no longer R7.P$1, R8.P$2, R9.P$1
- net N$25: now also R21.P$2; no longer R16.P$2
- net N$27: now also C1.1, R23.P$1; no longer C5.1, R18.P$1
- net N$3: now also C2.2, R9.P$1; no longer C1.2, R10.P$1
- net N$30: now also C1.2, R11.P$1; no longer C5.2, R21.P$1
- net N$31: now also R27.P$2; no longer R25.P$2
- net N$33: now also R24.P$1; no longer R19.P$1
- net N$34: now also C5.2, R30.P$1; no longer C4.2, R24.P$1
- net N$43: now also R23.P$2, R25.P$2; no longer R18.P$2, R20.P$2
- net N$44: now also R10.P$1, R7.P$1; no longer R6.P$1, R8.P$1
- net N$5: now also R26.P$2; no longer R17.P$2
- net N$6: now also R19.P$1, R28.P$2; no longer R14.P$1, R22.P$2
- net N$7: now also C3.2, R18.P$1; no longer C2.2, R13.P$1
- net N$8: now also C4.2, R29.P$1; no longer C3.2, R23.P$1
- net W_IN: now also R25.P$1, R6.P$2; no longer R20.P$1, R7.P$2
- net Z_IN: now also R28.P$1; no longer R22.P$1
Other:
- moved on the sheet: C1, C2, C3, C4, C5, P1, P4, R1, R10, R12, R13, R14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
