File: yoke/mimic1567.sch (EAGLE design)
At the start: 71 parts, among them J1 JST-VH-5, P1 20K, P2 25 K, P3 5K, P4 200, P5 44PINEDGE, Q1 2N2907, Q10 2N3904, Q11 2N2907, Q2 2N3904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

Commit message: end of day
Parts:
- added R31: 330, keiths:AXIALRESISTORONE_WATT
- R1: value 274K -> 1M
- R10: value 1.96K -> 3.3; device keiths:AXIALRESISTORQUARTER_WATT -> keiths:R-1/2WATT; PN RNF14FTD1K96 -> (none)
- R11, R9: value 3.3 -> 1.96K; device keiths:R-1/2WATT -> keiths:AXIALRESISTORQUARTER_WATT; PN (none) -> RNF14FTD1K96
- R12: value 100 -> 3.3; device keiths:AXIALRESISTORQUARTER_WATT -> keiths:R-1/2WATT; PN RNF14FTD2K94 -> (none)
- R13: value 22 -> 100
- R15: value 6.81K -> 22; device keiths:AXIALRESISTORHALF_WATT -> keiths:AXIALRESISTORQUARTER_WATT; PN MFS1/2DCT52R6811F -> RNF14FTD2K94
- R16, R21: value 33.2K -> 6.81K; PN SFR16S0003322FR500 -> MFS1/2DCT52R6811F
- R17, R22: value 100 -> 33.2K; device keiths:AXIALRESISTORQUARTER_WATT -> keiths:AXIALRESISTORHALF_WATT; PN RNF14FTD2K94 -> SFR16S0003322FR500
- R19, R23: value 2K -> 100; PN MFR-25FRF52-2K -> RNF14FTD2K94
- R2: value 20K -> 274K; PN RNF14FTD2K94 -> MFR-25FBF52-274K
- R20: value 6.81K -> 2K; device keiths:AXIALRESISTORHALF_WATT -> keiths:AXIALRESISTORQUARTER_WATT; PN MFS1/2DCT52R6811F -> MFR-25FRF52-2K
- R24: value 10K -> 2K; device keiths:AXIALRESISTORHALF_WATT -> keiths:AXIALRESISTORQUARTER_WATT; PN MF1/2LCT52R103J -> MFR-25FRF52-2K
- R25: value 1K -> 10K; device keiths:AXIALRESISTORQUARTER_WATT -> keiths:AXIALRESISTORHALF_WATT; PN MFR-25FRF52-1K -> MF1/2LCT52R103J
- R26: value 1.2K -> 1K; device keiths:R-5WATT -> keiths:AXIALRESISTORQUARTER_WATT; PN AC05000001201JAC00 -> MFR-25FRF52-1K
- R28: value 1K -> 1.2K; device keiths:AXIALRESISTORQUARTER_WATT -> keiths:R-5WATT; PN MFR-25FRF52-1K -> AC05000001201JAC00
- R29: value 330 -> 1K; device keiths:AXIALRESISTORONE_WATT -> keiths:AXIALRESISTORQUARTER_WATT; PN SFR16S0003300JA500 -> MFR-25FRF52-1K
- R3: PN RNF14FTD4K64 -> RNF14FTD2K94
- R4: value 3.9K -> 20K; PN RNF14FTD2K94 -> RNF14FTD4K64
- R5: value 4.7K -> 3.9K; PN RNF14FTD4K64 -> RNF14FTD2K94
- R6: value 274K -> 4.7K; PN MFR-25FBF52-274K -> RNF14FTD4K64
- R7: value 137 -> 274K; PN CMF55137R00FHEB -> MFR-25FBF52-274K
- R8: value 1.96K -> 137; PN RNF14FTD1K96 -> CMF55137R00FHEB
Connections:
- net +50V: now also R16.P$1, R21.P$1, R28.P$1; no longer R15.P$1, R20.P$1, R26.P$1
- net -10V: now also R11.P$2, R15.P$2, R19.P$2, R23.P$2, R25.P$2, R31.P$2; no longer R10.P$2, R12.P$2, R17.P$2, R22.P$2, R24.P$2, R29.P$2
- net GND: now also R10.P$2, R12.P$2, R6.P$1; no longer R11.P$2, R2.P$1, R8.P$2
- net N$1: now also R15.P$1; no longer R14.P$1
- net N$16: now also R17.P$2; no longer R16.P$2
- net N$17: now also R16.P$2, R17.P$1; no longer R15.P$2, R16.P$1
- net N$18: now also R14.P$1; no longer R13.P$1
- net N$2: now also R20.P$2; no longer R19.P$2
- net N$20: now also R21.P$2, R22.P$1; no longer R20.P$2, R21.P$1
- net N$22: now also R7.P$1, R8.P$2, R9.P$1; no longer R6.P$1, R7.P$2, R8.P$1
- net N$23: now also R23.P$1; no longer R22.P$1
- net N$24: now also R19.P$1; no longer R17.P$1
- net N$25: now also R22.P$2; no longer R21.P$2
- net N$26: now also R13.P$1; no longer R12.P$1
- net N$27: now also R24.P$1; no longer R23.P$1
- net N$29: now also R6.P$2; no longer R4.P$2
- net N$3: now also R10.P$1; no longer R9.P$1
- net N$30: now also R12.P$1; no longer R11.P$1
- net N$31: now also R28.P$2; no longer R27.P$2
- net N$33: now also R25.P$1; no longer R24.P$1
- net N$34: now also R31.P$1; no longer R30.P$1
- net N$4: now also R4.P$2; no longer R2.P$2
- net N$43: now also R24.P$2, R26.P$2; no longer R23.P$2, R25.P$2
- net N$44: now also R11.P$1, R2.P$1, R8.P$1; no longer R1.P$1, R10.P$1, R7.P$1
- net N$5: now also R27.P$2; no longer R26.P$2
- net N$6: now also R20.P$1, R29.P$2; no longer R19.P$1, R28.P$2
- net N$8: now also R30.P$1; no longer R29.P$1
- net W_IN: now also R2.P$2, R26.P$1, R7.P$2; no longer R25.P$1, R6.P$2
- net Z_IN: now also R1.P$1, R29.P$1; no longer R28.P$1
Other:
- moved on the sheet: R1, R13, R14, R15, R16, R17, R19, R2, R20, R21, R22, R23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

Commit message: revised artwork
Parts:
- P5: value 44PINEDGE -> 44PINEDGE-M; device keiths:44PINEDGE -> keiths:44PINEDGE-M
- R26, R29: value 1K -> 1.2K; device keiths:AXIALRESISTORQUARTER_WATT -> keiths:R-5WATT; PN MFR-25FRF52-1K -> AC05000001201JAC00
- R27, R28: value 1.2K -> 1K; device keiths:R-5WATT -> keiths:AXIALRESISTORQUARTER_WATT; PN AC05000001201JAC00 -> MFR-25FRF52-1K
Connections:
- removed net N$35 (its old number): D15.C, D16.A
- new net N$39: D11.A, D16.C
- net +50V: now also R26.P$1, R29.P$1; no longer R27.P$1, R28.P$1
- net GND: now also P5.4
- net N$31: now also R29.P$2; no longer R28.P$2
- net N$33: now also D15.C; no longer D16.C
- net N$40: now also D16.A; no longer D11.A
- net N$43: now also R27.P$2; no longer R26.P$2
- net N$5: now also R26.P$2; no longer R27.P$2
- net N$6: now also R28.P$2; no longer R29.P$2
- net W_IN: now also R27.P$1; no longer R26.P$1
- net Z_IN: now also R28.P$1; no longer R29.P$1
Other:
- note added: "X Preamplifier"
- moved on the sheet: D11, D12, D13, D14, D15, D16, P5, R26, R27, R28, R29
