File: yoke/mimic1568_DtoA.brd (EAGLE design)
At the start: 165.1 x 114.3 mm, 23 parts, among them P1 1K, P2 1K, P3 44PINEDGE, U1 AD7533, U2 CD74HC573E, U3 CD74HCT75, U4 OPA2340N, U5 AD7533, U6 CD74HC573E

Commit message: end of day
Parts:
- moved U3 0.11 mm to (57.1, 55.6)
Routing:
- net N$44: track 152.4 -> 139.2 mm
- net D0: track 152.1 -> 151.4 mm
Changed lines of the file:
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@@
 <attribute name="VALUE" x="79.4004" y="103.632" size="1.6764" layer="27" font="vector" ratio="10"/>
 </element>
-<element name="U3" library="keiths" package="DIP-16" value="CD74HCT75" x="57.2516" y="55.6768" smashed="yes" rot="R270">
-<attribute name="NAME" x="63.754" y="60.8838" size="1.9304" layer="25" font="vector" ratio="10"/>
-<attribute name="VALUE" x="63.1952" y="50.3428" size="1.6764" layer="27" font="vector" ratio="10"/>
+<element name="U3" library="keiths" package="DIP-16" value="CD74HCT75" x="57.15" y="55.626" smashed="yes" rot="R270">
+<attribute name="NAME" x="63.6524" y="60.833" size="1.9304" layer="25" font="vector" ratio="10"/>
+<attribute name="VALUE" x="63.0936" y="50.292" size="1.6764" layer="27" font="vector" ratio="10"/>
 </element>
 <element name="U6" library="keiths" package="DIP-20" value="CD74HC573E" x="57.15" y="25.654" smashed="yes" rot="R270">
@@
 <wire x1="21.59" y1="27.432" x2="31.75" y2="37.592" width="0.4064" layer="1"/>
 <via x="31.75" y="37.592" extent="1-16" drill="0.7"/>
-<wire x1="31.75" y1="37.592" x2="50.8" y2="56.642" width="0.4064" layer="16"/>
-<wire x1="50.8" y1="56.642" x2="53.3908" y2="56.896" width="0.4064" layer="16"/>
-<wire x1="53.3908" y1="56.896" x2="53.4416" y2="56.9468" width="0.4064" layer="16"/>
+<wire x1="31.75" y1="37.592" x2="51.054" y2="56.896" width="0.4064" layer="16"/>
+<wire x1="51.054" y1="56.896" x2="53.34" y2="56.896" width="0.4064" layer="16"/>
 </signal>
 <signal name="N$3">
@@
 <wire x1="118.11" y1="76.454" x2="74.168" y2="76.454" width="0.4064" layer="16"/>
 <wire x1="74.168" y1="76.454" x2="63.754" y2="64.516" width="0.4064" layer="16"/>
-<wire x1="63.754" y1="64.516" x2="61.1124" y2="64.516" width="0.4064" layer="16"/>
-<wire x1="61.1124" y1="64.516" x2="61.0616" y2="64.5668" width="0.4064" layer="16"/>
 <wire x1="118.11" y1="76.454" x2="125.73" y2="84.074" width="0.4064" layer="16"/>
+<wire x1="60.96" y1="64.516" x2="63.754" y2="64.516" width="0.4064" layer="16"/>
 </signal>
 <signal name="N$4">
@@
 <wire x1="128.27" y1="84.074" x2="118.11" y2="73.914" width="0.4064" layer="16"/>
 <wire x1="74.168" y1="73.914" x2="63.754" y2="62.23" width="0.4064" layer="16"/>
-<wire x1="63.754" y1="62.23" x2="61.2648" y2="62.23" width="0.4064" layer="16"/>
-<wire x1="61.2648" y1="62.23" x2="61.0616" y2="62.0268" width="0.4064" layer="16"/>
 <wire x1="74.168" y1="73.914" x2="118.11" y2="73.914" width="0.4064" layer="16"/>
+<wire x1="60.96" y1="61.976" x2="63.5" y2="61.976" width="0.4064" layer="16"/>
+<wire x1="63.5" y1="61.976" x2="63.754" y2="62.23" width="0.4064" layer="16"/>
 </signal>
 <signal name="N$25">
@@
 <contactref element="U3" pad="10"/>
 <contactref element="U5" pad="12"/>
-<wire x1="61.2648" y1="49.149" x2="61.0616" y2="49.3268" width="0.254" layer="16"/>
+<wire x1="61.2648" y1="49.149" x2="60.96" y2="49.276" width="0.254" layer="16"/>
 <wire x1="118.618" y1="19.304" x2="96.3168" y2="19.304" width="0.4064" layer="1"/>
-<wire x1="66.548" y1="49.3268" x2="61.0616" y2="49.3268" width="0.4064" layer="1"/>
-<wire x1="66.548" y1="49.3268" x2="96.3168" y2="19.304" width="0.4064" layer="1"/>
+<wire x1="66.548" y1="49.276" x2="60.96" y2="49.276" width="0.4064" layer="1"/>
+<wire x1="66.548" y1="49.276" x2="96.3168" y2="19.304" width="0.4064" layer="1"/>
 <wire x1="118.618" y1="19.304" x2="122.174" y2="22.86" width="0.4064" layer="1"/>
 <wire x1="122.174" y1="22.86" x2="122.174" y2="29.718" width="0.4064" layer="1"/>
@@
 <via x="22.86" y="74.9808" extent="1-16" drill="0.7"/>
 <wire x1="4.826" y1="74.9808" x2="22.86" y2="74.9808" width="0.4064" layer="1"/>
-<wire x1="43.18" y1="37.084" x2="43.18" y2="62.0268" width="0.4064" layer="1"/>
+<wire x1="43.18" y1="37.084" x2="43.18" y2="61.976" width="0.4064" layer="1"/>
 <wire x1="22.86" y1="74.9808" x2="33.02" y2="74.9808" width="0.4064" layer="1"/>
-<wire x1="53.4416" y1="62.0268" x2="43.18" y2="62.0268" width="0.4064" layer="16"/>
-<via x="43.18" y="62.0268" extent="1-16" drill="0.7"/>
+<wire x1="53.34" y1="61.976" x2="43.18" y2="61.976" width="0.4064" layer="16"/>
+<via x="43.18" y="61.976" extent="1-16" drill="0.7"/>
 <wire x1="43.18" y1="37.084" x2="45.72" y2="34.544" width="0.4064" layer="1"/>
 <wire x1="45.72" y1="34.544" x2="53.34" y2="34.544" width="0.4064" layer="1"/>
 <wire x1="33.02" y1="74.9808" x2="43.18" y2="64.8208" width="0.4064" layer="1"/>
-<wire x1="43.18" y1="64.8208" x2="43.18" y2="62.0268" width="0.4064" layer="1"/>
-<wire x1="53.4416" y1="62.0268" x2="56.0832" y2="62.0268" width="0.4064" layer="1"/>
+<wire x1="43.18" y1="64.8208" x2="43.18" y2="61.976" width="0.4064" layer="1"/>
+<wire x1="53.34" y1="61.976" x2="56.0832" y2="61.976" width="0.4064" layer="1"/>
 <wire x1="57.15" y1="60.96" x2="57.15" y2="53.086" width="0.4064" layer="1"/>
-<wire x1="55.118" y1="51.816" x2="55.88" y2="51.816" width="0.4064" layer="1"/>
-<wire x1="55.88" y1="51.816" x2="53.4416" y2="51.8668" width="0.4064" layer="1"/>
+<wire x1="55.88" y1="51.816" x2="53.34" y2="51.816" width="0.4064" layer="1"/>
 <wire x1="55.88" y1="51.816" x2="57.15" y2="53.086" width="0.4064" layer="1"/>
-<wire x1="56.0832" y1="62.0268" x2="57.15" y2="60.96" width="0.4064" layer="1"/>
+<wire x1="56.0832" y1="61.976" x2="57.15" y2="60.96" width="0.4064" layer="1"/>
 </signal>
 <signal name="D1">
@@
 <wire x1="53.34" y1="32.004" x2="45.72" y2="32.004" width="0.4064" layer="1"/>
 <wire x1="45.72" y1="32.004" x2="41.91" y2="35.814" width="0.4064" layer="1"/>
-<wire x1="41.91" y1="35.814" x2="41.91" y2="59.4868" width="0.4064" layer="1"/>
+<wire x1="41.91" y1="35.814" x2="41.91" y2="59.436" width="0.4064" layer="1"/>
 <wire x1="24.13" y1="71.0184" x2="33.02" y2="71.0184" width="0.4064" layer="1"/>
-<wire x1="53.4416" y1="59.4868" x2="41.91" y2="59.4868" width="0.4064" layer="16"/>
-<via x="41.91" y="59.4868" extent="1-16" drill="0.7"/>
+<wire x1="53.34" y1="59.436" x2="41.91" y2="59.436" width="0.4064" layer="16"/>
+<via x="41.91" y="59.436" extent="1-16" drill="0.7"/>
 <wire x1="33.02" y1="71.0184" x2="41.91" y2="62.1284" width="0.4064" layer="1"/>
-<wire x1="41.91" y1="62.1284" x2="41.91" y2="59.4868" width="0.4064" layer="1"/>
-<wire x1="53.4416" y1="49.3268" x2="55.9308" y2="49.3268" width="0.4064" layer="16"/>
-<wire x1="55.9308" y1="49.3268" x2="57.15" y2="50.546" width="0.4064" layer="16"/>
+<wire x1="41.91" y1="62.1284" x2="41.91" y2="59.436" width="0.4064" layer="1"/>
+<wire x1="53.34" y1="49.276" x2="55.88" y2="49.276" width="0.4064" layer="16"/>
+<wire x1="55.88" y1="49.276" x2="57.15" y2="50.546" width="0.4064" layer="16"/>
 <wire x1="57.15" y1="50.546" x2="57.15" y2="58.166" width="0.4064" layer="16"/>
 <wire x1="57.15" y1="58.166" x2="55.88" y2="59.436" width="0.4064" layer="16"/>
-<wire x1="55.88" y1="59.436" x2="53.4924" y2="59.436" width="0.4064" layer="16"/>
-<wire x1="53.4924" y1="59.436" x2="53.4416" y2="59.4868" width="0.4064" layer="16"/>
+<wire x1="55.88" y1="59.436" x2="53.34" y2="59.436" width="0.4064" layer="16"/>
 </signal>
 <signal name="D2">
@@
 <wire x1="90.678" y1="43.434" x2="78.232" y2="43.434" width="0.4064" layer="1"/>
 <wire x1="78.232" y1="43.434" x2="69.596" y2="52.07" width="0.4064" layer="1"/>
-<wire x1="69.596" y1="52.07" x2="69.596" y2="102.87" width="0.4064" layer="1"/>
-<wire x1="69.596" y1="102.87" x2="65.532" y2="106.934" width="0.4064" layer="1"/>
-<wire x1="65.532" y1="106.934" x2="41.91" y2="106.934" width="0.4064" layer="1"/>
-<wire x1="41.91" y1="106.934" x2="36.576" y2="101.6" width="0.4064" layer="1"/>
 <wire x1="90.678" y1="43.434" x2="94.742" y2="47.498" width="0.4064" layer="1"/>
 <contactref element="C6" pad="2"/>
@@
 <wire x1="101.6" y1="55.9162" x2="107.6598" y2="55.9162" width="0.4064" layer="16"/>
 <wire x1="107.6598" y1="55.9162" x2="107.696" y2="55.88" width="0.4064" layer="16"/>
-<wire x1="28.194" y1="101.6" x2="36.576" y2="101.6" width="0.4064" layer="1"/>
+<wire x1="28.194" y1="101.6" x2="40.64" y2="101.6" width="0.4064" layer="1"/>
+<wire x1="69.596" y1="52.07" x2="69.596" y2="65.024" width="0.4064" layer="1"/>
+<wire x1="69.596" y1="65.024" x2="62.23" y2="72.39" width="0.4064" layer="1"/>
+<wire x1="62.23" y1="72.39" x2="46.99" y2="72.39" width="0.4064" layer="1"/>
+<wire x1="46.99" y1="72.39" x2="43.18" y2="76.2" width="0.4064" layer="1"/>
+<wire x1="43.18" y1="76.2" x2="43.18" y2="99.06" width="0.4064" layer="1"/>
+<wire x1="43.18" y1="99.06" x2="40.64" y2="101.6" width="0.4064" layer="1"/>
 </signal>
 <signal name="N$45">
@@
 <contactref element="U3" pad="9"/>
 <wire x1="119.888" y1="16.764" x2="95.8088" y2="16.764" width="0.4064" layer="1"/>
-<wire x1="65.786" y1="46.7868" x2="61.0616" y2="46.7868" width="0.4064" layer="1"/>
-<wire x1="65.786" y1="46.7868" x2="95.8088" y2="16.764" width="0.4064" layer="1"/>
+<wire x1="65.786" y1="46.736" x2="60.96" y2="46.736" width="0.4064" layer="1"/>
+<wire x1="65.786" y1="46.736" x2="95.8088" y2="16.764" width="0.4064" layer="1"/>
 <wire x1="119.888" y1="16.764" x2="124.714" y2="21.59" width="0.4064" layer="1"/>
 <wire x1="124.714" y1="21.59" x2="124.714" y2="30.734" width="0.4064" layer="1"/>
@@
 <wire x1="64.262" y1="46.736" x2="64.262" y2="55.626" width="0.4064" layer="16"/>
 <wire x1="64.262" y1="55.626" x2="62.992" y2="56.896" width="0.4064" layer="16"/>
-<wire x1="62.992" y1="56.896" x2="61.1124" y2="56.896" width="0.4064" layer="16"/>
-<wire x1="61.1124" y1="56.896" x2="61.0616" y2="56.9468" width="0.4064" layer="16"/>
+<wire x1="62.992" y1="56.896" x2="60.96" y2="56.896" width="0.4064" layer="16"/>
 </signal>
 <signal name="N$2">

Commit message: added logo
Parts:
- moved U$1 17.8 mm to (36.8, 108.0)
Other:
- board text added: "board type 1568 / X Y Digital to Analog"
