File: yoke/mimic1575.brd (EAGLE design)
At the start: 160 x 100 mm, 69 parts, among them P1 20, P6 44PINEDGE, Q1 2N3904, Q10 2N3906, Q11 2N3904, Q12 2N3904, Q13 2N3904, Q14 2N3906, Q15 2N3904, Q16 2N2222A, Q19 2N2907, Q2 2N3904, Q20 2N3904, Q21 2N3906, Q22 2N3906, Q3 2N3904, Q4 2N3904, Q5 2N2222A, Q6 2N3904, Q7 2N3906, Q8 2N3904, Q9 2N3906

Commit message: update netlist
Parts:
- Q1, Q12: value 2N3904 -> KSP05TA
- moved Q1 213.1 mm to (-157.5, -94.0)
- moved Q12 196.5 mm to (-157.5, -105.4)
Changed lines of the file:
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@@
 <element name="D2" library="keiths" package="DO35-7" value="1N4148" x="-44.45" y="85.09"/>
 <element name="P6" library="keiths" package="44PINEDGE" value="44PINEDGE" x="0" y="52.07" rot="R270"/>
-<element name="Q1" library="keiths" package="TO92" value="2N3904" x="-29.21" y="76.2">
-<attribute name="PN" value="2N3904" x="-29.21" y="76.2" size="1.778" layer="27" display="off"/>
-</element>
 <element name="Q11" library="keiths" package="TO92" value="2N3904" x="-74.93" y="76.2">
 <attribute name="PN" value="2N3904" x="-74.93" y="76.2" size="1.778" layer="27" display="off"/>
-</element>
-<element name="Q12" library="keiths" package="TO92" value="2N3904" x="-82.55" y="76.2">
-<attribute name="PN" value="2N3904" x="-82.55" y="76.2" size="1.778" layer="27" display="off"/>
 </element>
 <element name="Q13" library="keiths" package="TO92" value="2N3904" x="-90.17" y="76.2">
@@
 </element>
 <element name="Q16" library="keiths" package="TO18" value="2N2222A" x="-157.48" y="-62.23"/>
+<element name="Q1" library="keiths" package="TO92" value="KSP05TA" x="-157.48" y="-93.98"/>
+<element name="Q12" library="keiths" package="TO92" value="KSP05TA" x="-157.48" y="-105.41"/>
 </elements>
 <signals>
@@
 </signal>
 <signal name="N$15">
-<contactref element="Q12" pad="1"/>
-<contactref element="Q1" pad="3"/>
 <contactref element="Q19" pad="1"/>
 <contactref element="Q10" pad="1"/>
-<wire x1="-81.28" y1="74.93" x2="-140.97" y2="-45.72" width="0" layer="19" extent="1-1"/>
-<wire x1="-103.505" y1="95.25" x2="-81.28" y2="74.93" width="0" layer="19" extent="1-1"/>
-<wire x1="-30.48" y1="77.47" x2="-81.28" y2="74.93" width="0" layer="19" extent="1-1"/>
+<contactref element="Q1" pad="3"/>
+<contactref element="Q12" pad="1"/>
+<wire x1="-156.21" y1="-106.68" x2="-158.75" y2="-92.71" width="0" layer="19" extent="1-1"/>
+<wire x1="-140.97" y1="-45.72" x2="-158.75" y2="-92.71" width="0" layer="19" extent="1-1"/>
+<wire x1="-103.505" y1="95.25" x2="-140.97" y2="-45.72" width="0" layer="19" extent="1-1"/>
 </signal>
 <signal name="N$17">
+<contactref element="R3" pad="1"/>
 <contactref element="Q12" pad="2"/>
-<contactref element="R3" pad="1"/>
-<wire x1="-81.28" y1="77.47" x2="-80.7" y2="33.02" width="0" layer="19" extent="1-1"/>
+<wire x1="-156.21" y1="-104.14" x2="-80.7" y2="33.02" width="0" layer="19" extent="1-1"/>
 </signal>
 <signal name="N$19">
+<contactref element="R24" pad="1"/>
 <contactref element="Q1" pad="2"/>
-<contactref element="R24" pad="1"/>
-<wire x1="-46.41" y1="66.04" x2="-27.94" y2="77.47" width="0" layer="19" extent="1-1"/>
+<wire x1="-46.41" y1="66.04" x2="-156.21" y2="-92.71" width="0" layer="19" extent="1-1"/>
 </signal>
 <signal name="N$20">
-<contactref element="Q12" pad="3"/>
-<contactref element="Q1" pad="1"/>
 <contactref element="C7" pad="1"/>
 <contactref element="Q13" pad="2"/>
-<wire x1="-44.41" y1="34.29" x2="-27.94" y2="74.93" width="0" layer="19" extent="1-1"/>
-<wire x1="-83.82" y1="77.47" x2="-27.94" y2="74.93" width="0" layer="19" extent="1-1"/>
-<wire x1="-88.9" y1="77.47" x2="-83.82" y2="77.47" width="0" layer="19" extent="1-1"/>
+<contactref element="Q1" pad="1"/>
+<contactref element="Q12" pad="3"/>
+<wire x1="-158.75" y1="-104.14" x2="-156.21" y2="-95.25" width="0" layer="19" extent="1-1"/>
+<wire x1="-44.41" y1="34.29" x2="-156.21" y2="-95.25" width="0" layer="19" extent="1-1"/>
+<wire x1="-88.9" y1="77.47" x2="-44.41" y2="34.29" width="0" layer="19" extent="1-1"/>
 </signal>
 <signal name="N$16">

Commit message: backup
Parts:
- removed P6: 44PINEDGE, keiths:44PINEDGE
- removed Q21, Q22: 2N3906, keiths:TO92
- added P2: 20, keiths:3006P
- added Q17, Q18: 2N3904, keiths:TO92
- C1: value 0.001uF -> 0.022 uF; device keiths:5MM_TH -> keiths:CAP-ZERO-PT-ZERO-22UF-250V-FILM
- C10: value 0.1uF -> 3.3 UF; device keiths:5MM_TH -> keiths:ECW-FD2W335K
- C11: value 3.3 UF -> 56 pF; device keiths:ECW-FD2W335K -> keiths:5MM_TH
- C3: value 56 pF -> 120pF
- C4: value 0.022 uF -> 0.001uF; device keiths:CAP-ZERO-PT-ZERO-22UF-250V-FILM -> keiths:5MM_TH
- C5: value 680pF -> 0.022 uF; device keiths:5MM_TH -> keiths:CAP-ZERO-PT-ZERO-22UF-250V-FILM
- C6: value 330pF -> 0.022uF; device keiths:5MM_TH -> keiths:CAP-ZERO-PT-ZERO-22UF-250V-FILM
- C7: value 120pF -> 680pF
- C8: value 0.022 uF -> 330pF; device keiths:CAP-ZERO-PT-ZERO-22UF-250V-FILM -> keiths:5MM_TH
- C9: value 0.022 uF -> 0.1uF; device keiths:CAP-ZERO-PT-ZERO-22UF-250V-FILM -> keiths:5MM_TH
- P1: value 20 -> 44PINEDGE; device keiths:3006P -> keiths:44PINEDGE
- Q1: value KSP05TA -> 2N3906
- Q10, Q7: value 2N3906 -> KSP05TA
- Q12: value KSP05TA -> 2N3904
- Q14: value 2N3906 -> 2N3904
- Q19: value 2N2907 -> 2N3904; device keiths:TO18 -> keiths:TO92
- Q2, Q3, Q6: value 2N3904 -> 2N3906
- Q20: value 2N3904 -> 2N2222A; device keiths:TO92 -> keiths:TO18
- Q4: value 2N3904 -> 2N2907; device keiths:TO92 -> keiths:TO18
- Q5: value 2N2222A -> 2N3906; device keiths:TO18 -> keiths:TO92
- R1: value 220 -> 120
- R10: value 1 K -> 1K
- R11: value 1500 -> 27
- R12: value 470 -> 27
- R13: value 560 -> 470
- R14: value 27 -> 1.5K
- R15, R21, R4: value 120 -> 27
- R16: value 560 -> 220
- R17: value 560 -> 1.5K
- R18, R5: value 27 -> 120
- R19, R25: value 27 -> 560
- R2: value 560 -> 120
- R20: value 27 -> 330
- R22: value 1.5 K -> 1K
- R23: value 10 K -> 120
- R24, R3: value 680 -> 560
- R26: value 120 -> 1K
- R27: value 1 K -> 120
- R28: value 27 -> 1K
- R29: value 330 -> 560
- R30: value 1 K -> 10K
- R31: value 120 -> 560
- R6: value 1 K -> 27
- R7: value 560 -> 27
- R8: value 120 -> 680
- R9: value 560 -> 680
- ZD3: value (none) -> BAT43
- moved Q12 311.0 mm to (102.9, 64.8), turned to 315 degrees
- moved Q1 279.5 mm to (57.1, 85.1), turned to 315 degrees
- moved ZD2 278.8 mm to (115.6, 12.7), turned to 270 degrees
- moved Q7 263.6 mm to (95.2, 30.5), flipped to the bottom, turned to 135 degrees
- moved Q9 255.0 mm to (82.5, 89.2), turned to 315 degrees
- moved R29 254.1 mm to (154.9, 72.4), turned to 90 degrees
- moved C11 245.6 mm to (139.7, 15.2), turned to 270 degrees
- moved R28 244.0 mm to (154.9, 39.4), turned to 90 degrees
- moved Q15 243.5 mm to (144.8, 54.6), turned to 315 degrees
- moved Q19 242.7 mm to (130.8, 39.4), turned to 315 degrees
- moved Q10 235.7 mm to (81.3, 30.5), flipped to the bottom, turned to 315 degrees
- moved R13 226.9 mm to (120.7, 102.3), turned to 90 degrees
- moved Q16 220.4 mm to (40.6, 34.3), turned to 270 degrees
- moved R26 218.9 mm to (148.6, 17.2), turned to 90 degrees
- moved R19 214.6 mm to (133.3, 102.3), turned to 90 degrees
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Connections:
- removed net +10V1: Q5.3, R10.2, R12.2, R16.2, R19.2, R2.2, R20.2, R25.2, R5.2, R8.2, R9.2
- net +10V: now also P1.A, Q20.3, R12.2, R13.2, R17.2, R19.2, R2.2, R20.2, R24.2, R28.2, R4.2, R6.2, R7.2; no longer P6.A, R22.2
- net -15V: now also P1.C, Q15.1, Q18.1, Q19.1, R11.1, R15.1, R25.1, R3.1, R30.1, R31.1, R5.1; no longer P6.C, Q2.1, Q3.1, Q4.1, R13.1, R14.1, R17.1, R23.1, R26.1, R28.1, R7.1
- net E_IN: now also P1.E, R1.2; no longer P6.E, R31.2
- net GND: now also C1.1, C3.2, C5.1, C6.1, P1.D, R10.1; no longer C4.1, C7.2, C8.1, C9.1, P6.D, R27.1
- net H_IN: now also C9.1, P1.H, P2.1, R22.1; no longer C11.1, P1.1, P6.H, R30.1
- net K_IN: now also P1.K, Q11.2; no longer P6.K, Q20.2
- net N$1: now also C4.1, R16.1; no longer C1.1, R1.1
- net N$10: now also Q5.3, R6.1; no longer Q9.3, R20.1
- net N$11: now also Q19.3, Q20.2, R29.1, R30.2; no longer Q4.3, Q5.2, R16.1, R23.2
- net N$12: now also Q19.2, R27.2; no longer Q4.2, R15.2
- net N$13: now also C2.2, Q4.3, R5.2; no longer C4.2, Q19.3, R21.2
- net N$14: now also Q12.2, Q14.2, Q17.2, Q9.1; no longer Q11.2, Q15.2, Q21.1, Q6.2
- net N$15: now also Q10.3, Q3.1, Q4.1, Q7.1; no longer Q1.3, Q10.1, Q12.1, Q19.1
- net N$16: now also Q6.3, R7.1; no longer Q22.3, R25.1
- net N$17: now also Q7.2, R8.1; no longer Q12.2, R3.1
- net N$18: now also Q14.1, R18.2; no longer Q11.1, R26.2
- net N$19: now also Q10.2, R9.1; no longer Q1.2, R24.1
- net N$2: now also C7.1, C8.1, Q15.3, R19.1; no longer C5.1, C6.1, Q2.3, R2.1
- net N$20: now also C3.1, Q10.1, Q7.3; no longer C7.1, Q1.1, Q12.3
- net N$21: now also Q1.2, Q3.2, Q5.1, Q5.2, Q6.2, R10.2; no longer Q10.2, Q14.2, Q21.2, Q22.2, Q9.1, R27.2
- net N$22: now also Q14.3; no longer Q11.3
- net N$23: now also D1.A, Q6.1, R8.2, R9.2; no longer D2.A, Q22.1, R24.2, R3.2
- net N$24: now also Q9.3, R12.1; no longer Q21.3, R5.1
- net N$25: now also Q2.2, R1.1; no longer Q7.2, R31.1
- net N$26: now also Q1.3, R2.1; no longer Q14.3, R8.1
- net N$27: now also C5.2, R17.1; no longer C8.2, R22.1
- net N$28: now also Q12.1, R15.2; no longer Q6.1, R14.2
- net N$3: now also C4.2, Q15.2, R23.1; no longer C1.2, Q2.2, R4.1
- net N$30: now also Q1.1, Q2.3, Q4.2; no longer Q14.1, Q19.2, Q7.3
- net N$31: now also C1.2, Q2.1, R3.2; no longer C2.2, Q7.1, R13.2
- net N$33: now also Q3.3, R4.1; no longer Q10.3, R19.1
- net N$34: now also Q12.3, R14.1, R16.2; no longer Q6.3, R1.2, R11.1
- net N$36: now also Q17.1, R21.2; no longer Q15.1, R28.2
- net N$37: now also Q11.1, R14.2; no longer Q20.1, R11.2
- net N$38: now also Q11.3, R13.1; no longer Q20.3, R12.1
- net N$39: now also Q17.3, R22.2; no longer Q15.3, R30.2
- net N$4: now also C11.1, R23.2, R26.2, R27.1; no longer C3.1, R15.1, R4.2, R6.2
- net N$40: now also C6.2, R20.1; no longer C9.2, R29.1
- net N$5: now also C11.2, Q18.3, R26.1, R28.1; no longer C3.2, Q3.3, R10.1, R6.1
- net N$6: now also D1.C, Q20.1, R31.2; no longer D2.C, Q5.1, R17.2
- net N$7: now also R11.2; no longer R18.2
- net N$8: now also D2.C, Q18.2; no longer D1.C, Q3.2
- net N$9: now also C7.2, C8.2, D2.A, R24.1, R25.2; no longer C5.2, C6.2, D1.A, R7.2, R9.1
- net Z_OUT: now also C9.2, P1.Z, P2.2, P2.3; no longer C11.2, P1.2, P1.3, P6.Z
Routing:
- net +10V: track 0.00 -> 344.1 mm
- net -15V: track 0.00 -> 338.9 mm, vias 0 -> 1
- net N$14: track 0.00 -> 157.7 mm
- net GND: track 0.00 -> 152.7 mm
- net N$9: track 0.00 -> 141.6 mm
- net Z_OUT: track 0.00 -> 137.4 mm
- net K_IN: track 0.00 -> 131.5 mm, vias 0 -> 1
- net H_IN: track 0.00 -> 79.2 mm
- net N$21: track 0.00 -> 78.5 mm
- net N$15: track 0.00 -> 77.9 mm
- net N$5: track 0.00 -> 70.5 mm
- net N$23: track 0.00 -> 70.4 mm
- net N$6: track 0.00 -> 66.4 mm
- net N$3: track 0.00 -> 61.0 mm
- net N$2: track 0.00 -> 60.5 mm
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Other:
- board size 160 x 100 mm -> 165.1 x 114.3 mm

Commit message: new .brd files
Parts:
- added U$1, U$2: FIDUCIAL, adafruit:FIDUCIAL_1MM
- C1: value 0.022 uF -> 0.022uF
- C11: value 56 pF -> 56pF
Changed lines of the file:
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@@
 <board>
 <plain>
-<wire x1="2.54" y1="11.684" x2="8.89" y2="11.684" width="0.1524" layer="20"/>
-<wire x1="8.89" y1="11.684" x2="8.89" y2="3.81" width="0.1524" layer="20"/>
-<wire x1="8.89" y1="3.81" x2="12.7" y2="0" width="0.1524" layer="20"/>
-<wire x1="12.7" y1="0" x2="165.1" y2="0" width="0.1524" layer="20"/>
-<wire x1="165.1" y1="0" x2="165.1" y2="114.3" width="0.1524" layer="20"/>
-<wire x1="165.1" y1="114.3" x2="12.7" y2="114.3" width="0.1524" layer="20"/>
-<wire x1="12.7" y1="114.3" x2="8.89" y2="110.49" width="0.1524" layer="20"/>
-<wire x1="8.89" y1="110.49" x2="8.89" y2="102.616" width="0.1524" layer="20"/>
-<wire x1="8.89" y1="102.616" x2="2.54" y2="102.616" width="0.1524" layer="20"/>
-<wire x1="2.54" y1="102.616" x2="0" y2="100.076" width="0.1524" layer="20"/>
-<wire x1="0" y1="100.076" x2="0" y2="14.224" width="0.1524" layer="20"/>
-<wire x1="0" y1="14.224" x2="2.54" y2="11.684" width="0.1524" layer="20"/>
+<wire x1="2.54" y1="11.684" x2="8.89" y2="11.684" width="0.0254" layer="20"/>
+<wire x1="8.89" y1="11.684" x2="8.89" y2="3.81" width="0.0254" layer="20"/>
+<wire x1="8.89" y1="3.81" x2="12.7" y2="0" width="0.0254" layer="20"/>
+<wire x1="12.7" y1="0" x2="165.1" y2="0" width="0.0254" layer="20"/>
+<wire x1="165.1" y1="0" x2="165.1" y2="114.3" width="0.0254" layer="20"/>
+<wire x1="165.1" y1="114.3" x2="12.7" y2="114.3" width="0.0254" layer="20"/>
+<wire x1="12.7" y1="114.3" x2="8.89" y2="110.49" width="0.0254" layer="20"/>
+<wire x1="8.89" y1="110.49" x2="8.89" y2="102.616" width="0.0254" layer="20"/>
+<wire x1="8.89" y1="102.616" x2="2.54" y2="102.616" width="0.0254" layer="20"/>
+<wire x1="2.54" y1="102.616" x2="0" y2="100.076" width="0.0254" layer="20"/>
+<wire x1="0" y1="100.076" x2="0" y2="14.224" width="0.0254" layer="20"/>
+<wire x1="0" y1="14.224" x2="2.54" y2="11.684" width="0.0254" layer="20"/>
 </plain>
 <attributes>
@@
 </class>
 </classes>
-<designrules name="default *">
+<designrules name="throughhole">
 <description language="de">&lt;b&gt;EAGLE Design Rules&lt;/b&gt;
 &lt;p&gt;
@@
 <attribute name="VALUE" x="121.285" y="26.035" size="1.6764" layer="27" font="vector" ratio="10" rot="R180" align="top-center"/>
 </element>
-<element name="C1" library="keiths" package="CAP-ZERO-PT-ZERO-22UF-250V-FILM" value="0.022 uF" x="40.64" y="83.1596" smashed="yes" rot="R270">
+<element name="C1" library="keiths" package="CAP-ZERO-PT-ZERO-22UF-250V-FILM" value="0.022uF" x="40.64" y="83.1596" smashed="yes" rot="R270">
 <attribute name="PN" value="ECQ-E2223JFB" x="40.64" y="83.1596" size="1.778" layer="27" rot="R270" display="off"/>
 <attribute name="NAME" x="39.053" y="89.6314" size="1.9304" layer="25" font="vector" ratio="10"/>
 <attribute name="VALUE" x="35.386" y="74.5354" size="1.6764" layer="27" font="vector" ratio="10"/>
 </element>
-<element name="C11" library="keiths" package="5MM_TH" value="56 pF" x="139.7" y="15.24" smashed="yes" rot="R270">
+<element name="C11" library="keiths" package="5MM_TH" value="56pF" x="139.7" y="15.24" smashed="yes" rot="R270">
 <attribute name="MPN" value="68 pF" x="139.7" y="15.24" size="1.778" layer="27" rot="R270" display="off"/>
 <attribute name="NAME" x="140.208" y="20.701" size="1.9304" layer="25" font="vector" ratio="10" align="bottom-center"/>
-<attribute name="VALUE" x="139.7" y="8.255" size="1.6764" layer="27" font="vector" ratio="10" rot="R180" align="top-center"/>
+<attribute name="VALUE" x="139.7" y="8.001" size="1.6764" layer="27" font="vector" ratio="10" rot="R180" align="top-center"/>
 </element>
 <element name="C2" library="keiths" package="CAP-ZERO-PT-ZERO-22UF-250V-FILM" value="0.022 uF" x="74.93" y="68.58" smashed="yes" rot="R90">
@@
 </element>
 <element name="P1" library="keiths" package="44PINEDGE" value="44PINEDGE" x="0" y="57.15" locked="yes" smashed="yes" rot="R270">
-<attribute name="NAME" x="-16.51" y="6.096" size="1.27" layer="25"/>
+<attribute name="NAME" x="12.192" y="57.404" size="1.27" layer="25" display="off"/>
 <attribute name="VALUE" x="-16.51" y="3.556" size="1.6764" layer="27" display="off"/>
 </element>
@@
 <attribute name="PN" value="2N3904" x="107.95" y="10.033" size="1.778" layer="27" rot="R315" display="off"/>
 <attribute name="NAME" x="106.32716875" y="13.42635" size="1.9304" layer="25" font="vector" ratio="10"/>
-<attribute name="VALUE" x="104.157596875" y="5.2968" size="1.6764" layer="27" font="vector" ratio="10"/>
+<attribute name="VALUE" x="101.617596875" y="5.2968" size="1.6764" layer="27" font="vector" ratio="10"/>
 </element>
 <element name="Q19" library="keiths" package="TO92" value="2N3904" x="130.81" y="39.37" smashed="yes" rot="R315">
@@
 </element>
 <element name="Q1" library="keiths" package="TO92" value="2N3906" x="57.15" y="85.09" smashed="yes" rot="R315">
-<attribute name="NAME" x="51.92785" y="85.82936875" size="1.9304" layer="25" font="vector" ratio="10"/>
+<attribute name="NAME" x="52.18185" y="86.33736875" size="1.9304" layer="25" font="vector" ratio="10"/>
 <attribute name="VALUE" x="58.513796875" y="87.796" size="1.6764" layer="27" font="vector" ratio="10"/>
 </element>
 <element name="Q2" library="keiths" package="TO92" value="2N3906" x="57.15" y="74.93" smashed="yes" rot="R315">
-<attribute name="NAME" x="51.97116875" y="74.25935" size="1.9304" layer="25" font="vector" ratio="10"/>
+<attribute name="NAME" x="54.25716875" y="78.06935" size="1.9304" layer="25" font="vector" ratio="10"/>
 <attribute name="VALUE" x="60.469596875" y="74.3848" size="1.6764" layer="27" font="vector" ratio="10"/>
 </element>
@@
 <attribute name="PN" value="BAT43" x="115.57" y="12.7" size="1.778" layer="27" rot="R270" display="off"/>
 <attribute name="NAME" x="113.284" y="18.415" size="1.9304" layer="25" font="vector" ratio="10"/>
-<attribute name="VALUE" x="114.681" y="5.715" size="1.6764" layer="27" font="vector" ratio="10"/>
+<attribute name="VALUE" x="112.395" y="5.461" size="1.6764" layer="27" font="vector" ratio="10"/>
 </element>
 <element name="Q16" library="keiths" package="TO18" value="2N2222A" x="40.64" y="34.29" smashed="yes" rot="R270">
@@
 <element name="Q10" library="keiths" package="TO92" value="KSP05TA" x="81.28" y="30.48" smashed="yes" rot="MR315">
 <attribute name="NAME" x="78.45783125" y="33.87335" size="1.9304" layer="25" font="vector" ratio="10"/>
-<attribute name="VALUE" x="77.198403125" y="25.7438" size="1.6764" layer="27" font="vector" ratio="10"/>
+<attribute name="VALUE" x="77.198403125" y="25.4898" size="1.6764" layer="27" font="vector" ratio="10"/>
 </element>
 <element name="Q7" library="keiths" package="TO92" value="KSP05TA" x="95.25" y="30.48" smashed="yes" rot="MR135">
@@
 <attribute name="VALUE" x="90.914403125" y="25.4898" size="1.6764" layer="27" font="vector" ratio="10"/>
 </element>
+<element name="U$1" library="adafruit" package="FIDUCIAL_1MM" value="FIDUCIAL" x="19.05" y="107.95"/>
+<element name="U$2" library="adafruit" package="FIDUCIAL_1MM" value="FIDUCIAL" x="152.4" y="6.35"/>
 </elements>
 <signals>
@@
 <contactref element="P1" pad="A"/>
 <wire x1="65.532" y1="65.532" x2="55.88" y2="55.88" width="1.016" layer="16"/>
-<wire x1="4.826" y1="98.7552" x2="13.97" y2="98.7552" width="1.016" layer="16"/>
-<wire x1="13.97" y1="98.7552" x2="21.9752" y2="106.7604" width="1.016" layer="16"/>
+<wire x1="4.826" y1="98.7552" x2="17.526" y2="98.7552" width="1.016" layer="16"/>
+<wire x1="17.526" y1="98.7552" x2="25.5312" y2="106.7604" width="1.016" layer="16"/>
 <wire x1="133.35" y1="106.7604" x2="120.65" y2="106.7604" width="1.016" layer="16"/>
 <wire x1="120.65" y1="106.7604" x2="107.95" y2="106.7604" width="1.016" layer="16"/>
@@
 <wire x1="69.85" y1="106.7604" x2="65.532" y2="106.7604" width="1.016" layer="16"/>
 <wire x1="65.532" y1="106.7604" x2="57.15" y2="106.7604" width="1.016" layer="16"/>
-<wire x1="21.9752" y1="106.7604" x2="57.15" y2="106.7604" width="1.016" layer="16"/>
+<wire x1="25.5312" y1="106.7604" x2="57.15" y2="106.7604" width="1.016" layer="16"/>
 <wire x1="130.81" y1="69.7738" x2="130.81" y2="73.66" width="1.016" layer="1"/>
 <wire x1="130.81" y1="73.66" x2="134.04" y2="76.89" width="1.016" layer="1"/>
