File: yoke/mimic1575.brd (EAGLE design)
At the start: 165.1 x 114.3 mm, 71 parts, among them P1 20, P2 44PINEDGE, Q1 2N3906, Q10 2N3904, Q100 KSP05TA, Q101 KSP05TA, Q11 2N3904, Q12 2N3904, Q13 2N3904, Q14 2N3904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

Commit message: revised artwork
Parts:
- removed ZD1: BAT43, keiths:DO35-7
- added D4: 1N4148, keiths:DO35-7
- D1: value 1N4148 -> BAT43
- P2: value 44PINEDGE -> 44PINEDGE-M
- R24: value 120 -> 1K
- R25: value 1K -> 120
- moved D1 40.9 mm to (148.6, 67.9), turned to 0 degrees
- moved D2 36.4 mm to (111.8, 50.2), turned to 270 degrees
- moved R24 21.8 mm to (154.9, 25.4), turned to 270 degrees
- moved R25 21.8 mm to (133.3, 22.2), turned to 90 degrees
- turned D3 to 0 degrees
- turned D5 to 0 degrees
- renumbered ZD2 to D3, ZD3 to D5
Connections:
- net -15V: now also P2.3
- net GND: now also P2.4
- net N$12: now also R25.2; no longer R24.2
- net N$2: now also D1.C; no longer ZD1.C
- net N$23: now also D2.A; no longer D1.A
- net N$3: now also D1.A; no longer ZD1.A
- net N$4: now also R24.2, R25.1; no longer R24.1, R25.2
- net N$5: now also R24.1; no longer R25.1
- net N$6: now also D2.C; no longer D1.C
- net N$8: now also D4.C; no longer D2.C
- net N$9: now also D4.A; no longer D2.A
Routing:
- net -15V: track 346.0 -> 360.9 mm, vias 1 -> 3
- net GND: track 152.7 -> 167.4 mm, vias 0 -> 2
