File: config_register/mimic1568_DtoA.sch (EAGLE design)
At the start: 15 parts, among them P1 1K, P2 44PINEDGE, P3 1K, U1 CD74HCT75, U11 OPA2340N, U2 CD74HC573E, U3 CD74HC573E, U5 AD7533, U6 AD7533

Commit message: D/A being routed
Parts:
- added U$1, U$2: FIDUCIAL, adafruit:FIDUCIAL
- R2, R3: value 1 K -> 1K
Connections:
- net +15V: now also P2.E
- net +5V: now also P2.B
- net -15V: now also P2.C
- net D0: now also P2.7
- net D1: now also P2.8
- net D2: now also P2.9
- net D3: now also P2.10
- net D4: now also P2.11
- net D5: now also P2.12
- net D6: now also P2.13
- net D7: now also P2.14
- net GND: now also P2.D
- net XPOS: now also P2.J
- net X_LSB: now also P2.17
- net X_MSB: now also P2.16
- net YPOS: now also P2.K
- net Y_LSB: now also P2.19
- net Y_MSB: now also P2.18
Other:
- moved on the sheet: C1, C5, P1, P2, P3, R1, R10, R2, R3, U1, U11A, U11B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
