File: config_register/mimic4218_config.sch (EAGLE design)
At the start: 19 parts, among them P5 44PINEDGE, U1 CD74HCT123, U2 CD74HCT123, U3 CD74HC573E, U4 CD74HC573E

Commit message: Friday backup
Parts:
- removed P5: 44PINEDGE, keiths:44PINEDGE
- added P3: 44PINEDGE, keiths:44PINEDGE
- U5, U6: value (none) -> CD74HC00
Connections:
- removed net !WRITE: U2.1B, U5.2B, U5.4B
- new net +10V: P3.A
- new net +15V: P3.E
- new net -15V: P3.C
- new net LE3: P3.18, U2.1B, U5.2B, U5.4B
- net +5V: now also P3.B, U2.2B
- net D0: now also P3.7; no longer P5.6
- net D1: now also P3.8; no longer P5.7
- net D2: now also P3.9; no longer P5.8
- net D3: now also P3.10; no longer P5.9
- net D4: now also P3.11; no longer P5.10
- net D5: now also P3.12; no longer P5.11
- net D6: now also P3.13; no longer P5.12
- net D7: now also P3.14; no longer P5.13
- net GND: now also P3.D; no longer U2.!2A
- net HORIZ_F: now also P3.R
- net HORIZ_U: now also P3.S
- net INTENSIFY_P: now also P3.X
- net JUMP_DOWN: now also U6.2B
- net JUMP_LEFT: now also U6.3B
- net JUMP_RIGHT: now also U6.4B
- net JUMP_UP: now also U6.1B
- net J_INTEN: now also P3.V
- net J_JUMP: now also P3.J
- net K_JUMP: now also P3.K
- net LE1: now also P3.16
- net LE2: now also P3.17
- net L_JUMP: now also P3.L
- net N$15: now also U2.!2A; no longer U2.2B
- net U_INTEN: now also P3.W
- net VERT_F: now also P3.N
- net VERT_U: now also P3.P
- net X_INTEN: now also P3.U
Other:
- note added: "* The original DEC 4218 System Design Module was a data latch. It was used to capture some of the original DEC 340 configuration bits shown on this page. This resulted in the name for this card."
- note added: "High levels to direction bits enable open loop pulse steps."
- note added: "LE3 is a postive going trigger which starts the open and closed loop intensification delays. DELAY SELECT high selects 35uS and DELAY SELECT set low selects 1uS. If the INTENSIFY bit has been set high the low going intensification pulse is enabled. LE3 can be tied to the X_MSB strobe to start an intensification if X_MSB is the last position byte written."
- note added: "X_INTEN, U_INTEN, J_INTEN control cathode voltage. Low levels bring the cathode negative. INTENSITY high enables a pulse. The J_JUMP, K_JUMP, L_JUMP bits bus to the mimic_1579 cards. Low levels on these lines enable current."
- note added: "intensity"
- note removed: "* The original DEC 4218 System Design Module was a data latch. It was used to capture some of the original DEC 340 configuration bits shown on this page."
- note removed: "High levels to direction bits enable current drive."
- note removed: "POSITIVE_EDGE"
- note removed: "The DELAY_SELECT bit selects the 35 uS delay when high and the 1 uS delay when low."
- note removed: "The J_JUMP, K_JUMP, L_JUMP bits bus to the Contra_1579 cards. Low levels on these lines enable current."
- note removed: "X_INTEN, U_INTEN, J_INTEN control cathode voltage. Low levels bring the cathode negative. INTENSITY high enables a pulse."
- note removed: "output"
- moved on the sheet: C1, C2, C3, C4, R1, R2, R3, R4, R5, R6, R7, R8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
