File: config_register/mimic4218.brd (EAGLE design)
At the start: 165.1 x 114.3 mm, 19 parts, among them P3 44PINEDGE, U1 CD74HCT123, U2 CD74HCT123, U3 CD74HC573E, U4 CD74HC573E, U5 CD74HC00, U6 CD74HC00

Commit message: end of day
Parts:
- added C10, C5, C6, C7, C8, C9: 0.1uF, keiths:5MM_TH
- moved R4 217.9 mm to (147.8, 69.1), turned to 180 degrees
- moved R8 209.5 mm to (147.1, 23.1), turned to 180 degrees
- moved R3 206.2 mm to (148.3, 75.7), turned to 180 degrees
- moved C3 198.5 mm to (130.3, 28.4), turned to 90 degrees
- moved R7 195.2 mm to (147.1, 32.3), turned to 180 degrees
- moved R2 194.5 mm to (147.3, 90.9), turned to 180 degrees
- moved C2 186.4 mm to (130.3, 70.4), turned to 90 degrees
- moved R1 183.5 mm to (147.3, 98.3), turned to 180 degrees
- moved R6 181.2 mm to (147.3, 42.2), turned to 180 degrees
- moved C1 177.4 mm to (130.6, 93.5), turned to 90 degrees
- moved R5 167.3 mm to (147.3, 52.6), turned to 180 degrees
- moved U5 163.7 mm to (92.7, 62.2), turned to 270 degrees
- moved U2 158.9 mm to (111.8, 41.9), turned to 270 degrees
- moved C4 149.6 mm to (130.3, 50.3), turned to 90 degrees
- moved U1 143.0 mm to (110.5, 82.5), turned to 270 degrees
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Connections:
- net +5V: now also C10.1, C5.1, C6.1, C7.1, C8.1, C9.1
- net GND: now also C10.2, C5.2, C6.2, C7.2, C8.2, C9.2
Routing:
- net D0: track 0.00 -> 134.6 mm, vias 0 -> 1
- net D1: track 0.00 -> 134.3 mm, vias 0 -> 1
- net D2: track 0.00 -> 133.9 mm, vias 0 -> 1
- net D3: track 0.00 -> 133.5 mm, vias 0 -> 1
- net D4: track 0.00 -> 133.1 mm, vias 0 -> 1
- net D5: track 0.00 -> 132.8 mm, vias 0 -> 1
- net D6: track 0.00 -> 132.4 mm, vias 0 -> 1
- net D7: track 0.00 -> 131.9 mm, vias 0 -> 1
- net GND: track 0.00 -> 7.87 mm, vias 0 -> 1
- net +5V: track 0.00 -> 7.87 mm, vias 0 -> 1
- added copper zone on layer 2, net +5V
- added copper zone on layer 15, net GND

Commit message: end of day
Parts:
- moved C10 62.4 mm to (87.6, 101.6)
- moved C5 39.1 mm to (41.9, 76.6)
- moved U4 38.7 mm to (41.9, 61.1)
- moved U3 35.8 mm to (64.8, 61.1)
- moved U5 28.4 mm to (87.6, 90.2)
- moved U6 16.9 mm to (86.4, 59.4)
- moved R8 16.2 mm to (141.0, 38.1)
- moved C3 15.8 mm to (127.0, 43.9), turned to 270 degrees
- moved U2 15.5 mm to (109.2, 57.1)
- moved R6 15.1 mm to (141.0, 55.9)
- moved R7 14.8 mm to (141.0, 45.7)
- moved C6 14.7 mm to (109.2, 69.8)
- moved R5 12.6 mm to (141.0, 63.5)
- moved C9 10.5 mm to (64.8, 76.7)
- moved R3 10.1 mm to (141.0, 82.5)
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Routing:
- net LE3: track 0.00 -> 170.0 mm
- net INTENSIFY_P: track 0.00 -> 121.6 mm, vias 0 -> 1
- net HORIZ_F: track 0.00 -> 100.8 mm
- net VERT_F: track 0.00 -> 100.7 mm
- net HORIZ_U: track 0.00 -> 93.3 mm
- net VERT_U: track 0.00 -> 92.4 mm
- net U_INTEN: track 0.00 -> 82.9 mm, vias 0 -> 2
- net D3: track 133.5 -> 57.5 mm, vias 1 -> 0
- net D2: track 133.9 -> 58.1 mm, vias 1 -> 0
- net D4: track 133.1 -> 57.5 mm, vias 1 -> 0
- net D1: track 134.3 -> 58.7 mm, vias 1 -> 0
- net D0: track 134.6 -> 59.2 mm, vias 1 -> 0
- net D6: track 132.4 -> 58.7 mm, vias 1 -> 0
- net INTENSIFY: track 0.00 -> 72.8 mm
- net D7: track 131.9 -> 59.2 mm, vias 1 -> 0
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
Commit message: card layouts finished
Routing:
- net D5: track 67.9 -> 59.5 mm
- net N$8: track 24.7 -> 32.3 mm
Changed lines of the file:
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@@
 <wire x1="50.165" y1="57.3024" x2="48.895" y2="56.0324" width="0.4064" layer="1"/>
 <wire x1="38.1" y1="57.3024" x2="16.51" y2="57.3024" width="0.4064" layer="1"/>
-<wire x1="5.08" y1="55.1688" x2="14.3764" y2="55.1688" width="0.4064" layer="1"/>
-<wire x1="14.3764" y1="55.1688" x2="14.6558" y2="55.4482" width="0.4064" layer="1"/>
-<wire x1="14.6558" y1="55.4482" x2="16.51" y2="57.3024" width="0.4064" layer="1"/>
-<wire x1="14.732" y1="55.372" x2="5.08" y2="55.372" width="0.254" layer="1"/>
+<wire x1="5.08" y1="55.1688" x2="6.35" y2="55.1688" width="0.4064" layer="1"/>
+<wire x1="6.35" y1="55.1688" x2="14.3764" y2="55.1688" width="0.4064" layer="1"/>
 <wire x1="5.08" y1="55.372" x2="4.826" y2="55.1688" width="0.254" layer="1"/>
-<wire x1="14.732" y1="55.372" x2="14.6558" y2="55.4482" width="0.254" layer="1"/>
+<wire x1="14.3764" y1="55.1688" x2="16.51" y2="57.3024" width="0.4064" layer="1"/>
+<wire x1="5.08" y1="55.372" x2="6.1468" y2="55.372" width="0.4064" layer="1"/>
+<wire x1="6.1468" y1="55.372" x2="6.35" y2="55.1688" width="0.4064" layer="1"/>
 </signal>
 <signal name="D6">
@@
 <wire x1="22.86" y1="27.305" x2="26.67" y2="29.972" width="0.4064" layer="16"/>
 <wire x1="26.67" y1="29.972" x2="30.6832" y2="29.972" width="0.4064" layer="16"/>
-<wire x1="32.385" y1="31.75" x2="32.385" y2="32.385" width="0.4064" layer="16"/>
-<wire x1="32.385" y1="32.385" x2="32.385" y2="33.655" width="0.4064" layer="16"/>
+<wire x1="32.385" y1="31.6738" x2="32.385" y2="33.655" width="0.4064" layer="16"/>
 <wire x1="27.305" y1="35.3568" x2="30.6832" y2="35.3568" width="0.4064" layer="16"/>
 <wire x1="30.6832" y1="35.3568" x2="32.385" y2="33.655" width="0.4064" layer="16"/>
 <wire x1="30.6832" y1="29.972" x2="32.385" y2="31.6738" width="0.4064" layer="16"/>
-<wire x1="32.385" y1="31.6738" x2="32.385" y2="31.75" width="0.4064" layer="16"/>
 </signal>
 <signal name="J_INTEN">
@@
 <wire x1="127" y1="63.5" x2="113.03" y2="63.5" width="0.4064" layer="16"/>
 <wire x1="127" y1="61.682" x2="127" y2="63.5" width="0.4064" layer="16"/>
-<wire x1="135.89" y1="63.5" x2="135.89" y2="55.88" width="0" layer="19" extent="1-1"/>
+<wire x1="135.89" y1="55.88" x2="135.89" y2="63.5" width="0.4064" layer="16"/>
 </signal>
 <signal name="INTENSIFY">

Commit message: added logo
Parts:
- added U$1, U$2: FIDUCIAL, adafruit:FIDUCIAL_1MM
- C1: value .033 uF -> 0.1uF
- C10, C9: value 0.1uF -> 470 pF
- C2: value .001 uF -> 0.1uF
- C3: value 470 pF -> .033 uF
- C4: value 470 pF -> .001 uF
- U1: value CD74HCT123 -> CD74HC00; device keiths:DIP-16 -> keiths:DIP-14
- U6: value CD74HC00 -> CD74HCT123; device keiths:DIP-14 -> keiths:DIP-16
- moved C10 69.8 mm to (127.0, 43.9), turned to 270 degrees
- moved C9 64.7 mm to (127.0, 59.2), turned to 90 degrees
- moved C3 52.1 mm to (127.0, 96.0), turned to 90 degrees
- moved C2 45.3 mm to (87.6, 101.6), turned to 0 degrees
- moved C6 45.0 mm to (64.8, 76.6)
- moved C8 33.2 mm to (109.2, 69.8)
- moved U2 33.0 mm to (109.2, 90.2)
- moved U5 30.8 mm to (86.4, 59.4)
- moved U6 23.0 mm to (109.2, 57.1)
- moved U3 22.9 mm to (41.9, 61.1)
- moved U4 22.9 mm to (64.8, 61.1)
- moved U1 21.6 mm to (87.6, 90.2)
- moved C4 20.1 mm to (127.0, 79.2)
- moved C1 19.1 mm to (109.2, 103.0), turned to 0 degrees
- renumbered P3 to P1
Connections:
- net +5V: now also C1.1, C2.1, U1.14, U2.11, U2.2, U6.10, U6.16, U6.3; no longer C10.1, C9.1, U1.10, U1.11, U1.16, U1.2, U1.3, U6.14
- net DELAY_SELECT: now also U1.1, U1.12, U1.2, U3.16; no longer U4.16, U5.1, U5.12, U5.2
- net GND: now also C1.2, C2.2, U1.7, U6.1, U6.8; no longer C10.2, C9.2, U1.8, U2.1, U6.7
- net HORIZ_F: now also U5.11; no longer U6.11
- net HORIZ_U: now also U5.8; no longer U6.8
- net INTENSIFY: now also U3.15, U6.11; no longer U2.11, U4.15
- net INTENSIFY_P: now also U6.12; no longer U2.12
- net JUMP_DOWN: now also U4.18, U5.5; no longer U3.18, U6.5
- net JUMP_LEFT: now also U4.16, U5.10; no longer U3.16, U6.10
- net JUMP_RIGHT: now also U4.17, U5.13; no longer U3.17, U6.13
- net JUMP_UP: now also U4.19, U5.2; no longer U3.19, U6.2
- net J_INTEN: now also U3.17; no longer U4.17
- net J_JUMP: now also U3.14; no longer U4.14
- net K_JUMP: now also U3.13; no longer U4.13
- net LE1: now also U4.11; no longer U3.11
- net LE2: now also U3.11; no longer U4.11
- net LE3: now also U1.13, U1.5, U6.2; no longer U2.2, U5.13, U5.5
- net L_JUMP: now also U3.12; no longer U4.12
- net N$1: now also C3.1, U2.14; no longer C1.1, U1.14
- net N$10: now also U1.3, U1.4; no longer U5.3, U5.4
- net N$11: now also U5.1, U5.12, U5.4, U5.9, U6.13; no longer U2.13, U6.1, U6.12, U6.4, U6.9
- net N$12: now also U1.6, U2.9; no longer U1.9, U5.6
- net N$13: now also U1.9, U2.4; no longer U1.4, U5.9
- net N$14: now also U1.10, U2.12; no longer U1.12, U5.10
- net N$15: now also U1.8, U6.9; no longer U2.9, U5.8
- net N$2: now also C3.2, U2.15; no longer C1.2, U1.15
- net N$3: now also C4.1, U2.6; no longer C2.1, U1.6
- net N$4: now also C4.2, U2.7; no longer C2.2, U1.7
- net N$5: now also C9.1, U6.14; no longer C4.1, U2.14
- net N$6: now also C10.2, U6.7; no longer C3.2, U2.7
- net N$7: now also C10.1, U6.6; no longer C3.1, U2.6
- net N$8: now also C9.2, U6.15; no longer C4.2, U2.15
- net N$9: now also U1.11, U2.1; no longer U1.1, U5.11
- net U_INTEN: now also U3.18; no longer U4.18
- net VERT_F: now also U5.3; no longer U6.3
- net VERT_U: now also U5.6; no longer U6.6
- net X_INTEN: now also U3.19; no longer U4.19
Other:
- board text added: "board type 4218 / parameter store"
