File: config_register/mimic4218.brd (EAGLE design)
At the start: 165.1 x 114.3 mm, 27 parts, among them P1 44PINEDGE, U1 CD74HC00, U2 CD74HCT123, U3 CD74HC573E, U4 CD74HC573E, U5 CD74HC00, U6 CD74HCT123

Commit message: revised artwork
Parts:
- P13: value 44PINEDGE -> 44PINEDGE-M
- renumbered P1 to P13
Connections:
- removed net +10V: P13.A
- removed net +15V: P13.E
- removed net -15V: P13.C
- new net FF_J: P13.J
- new net FF_K: P13.K
- new net FF_L: P13.L
- net GND: now also P13.4
- net J_JUMP: no longer P13.J
- net K_JUMP: no longer P13.K
- net L_JUMP: no longer P13.L
Routing:
- net J_JUMP: track 66.1 -> 54.3 mm
- net GND: track 11.7 -> 23.4 mm
- net K_JUMP: track 62.2 -> 51.4 mm
- net L_JUMP: track 57.0 -> 50.0 mm
