File: config_register/mimic4218.sch (EAGLE design)
At the start: 19 parts, among them P3 44PINEDGE, U1 CD74HCT123, U2 CD74HCT123, U3 CD74HC573E, U4 CD74HC573E, U5 CD74HC00, U6 CD74HC00

Commit message: end of day
Parts:
- added C10, C5, C6, C7, C8, C9: 0.1uF, keiths:CAP0.1UF100V
Connections:
- net +5V: now also C10.1, C5.1, C6.1, C7.1, C8.1, C9.1
- net GND: now also C10.2, C5.2, C6.2, C7.2, C8.2, C9.2
Changed lines of the file:
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@@
 <part name="SUPPLY28" library="supply2" deviceset="+10V" device=""/>
 <part name="SUPPLY29" library="keiths" deviceset="+5V" device=""/>
+<part name="C5" library="keiths" deviceset="CAP0.1UF100V" device="" value="0.1uF"/>
+<part name="C6" library="keiths" deviceset="CAP0.1UF100V" device="" value="0.1uF"/>
+<part name="SUPPLY30" library="keiths" deviceset="GND" device=""/>
+<part name="SUPPLY31" library="keiths" deviceset="GND" device=""/>
+<part name="SUPPLY32" library="keiths" deviceset="+5V" device=""/>
+<part name="SUPPLY33" library="keiths" deviceset="+5V" device=""/>
+<part name="C8" library="keiths" deviceset="CAP0.1UF100V" device="" value="0.1uF"/>
+<part name="SUPPLY34" library="keiths" deviceset="GND" device=""/>
+<part name="SUPPLY35" library="keiths" deviceset="+5V" device=""/>
+<part name="C7" library="keiths" deviceset="CAP0.1UF100V" device="" value="0.1uF"/>
+<part name="C9" library="keiths" deviceset="CAP0.1UF100V" device="" value="0.1uF"/>
+<part name="SUPPLY36" library="keiths" deviceset="GND" device=""/>
+<part name="SUPPLY37" library="keiths" deviceset="GND" device=""/>
+<part name="SUPPLY38" library="keiths" deviceset="+5V" device=""/>
+<part name="SUPPLY39" library="keiths" deviceset="+5V" device=""/>
+<part name="C10" library="keiths" deviceset="CAP0.1UF100V" device="" value="0.1uF"/>
+<part name="SUPPLY40" library="keiths" deviceset="GND" device=""/>
+<part name="SUPPLY41" library="keiths" deviceset="+5V" device=""/>
 </parts>
 <sheets>
@@
 <text x="361.188" y="169.164" size="2.1844" layer="91">500 nS</text>
 <text x="361.188" y="184.404" size="2.1844" layer="91">400 nS</text>
-<text x="226.06" y="81.28" size="2.1844" layer="91" font="vector" ratio="10">* The original DEC 4218 System Design Module
+<text x="330.2" y="15.24" size="2.1844" layer="91" font="vector" ratio="10">* The original DEC 4218 System Design Module
 was a data latch.  It was used to capture some
 of the original DEC 340 configuration bits shown
@@
 <attribute name="VALUE" x="293.751" y="166.497" size="1.9304" layer="96" font="vector" ratio="10" rot="MR0"/>
 </instance>
+<instance part="C5" gate="G$1" x="139.7" y="78.74"/>
+<instance part="C6" gate="G$1" x="160.02" y="78.74"/>
+<instance part="SUPPLY30" gate="GND" x="139.7" y="68.58"/>
+<instance part="SUPPLY31" gate="GND" x="160.02" y="68.58"/>
+<instance part="SUPPLY32" gate="+5V" x="139.7" y="88.9" smashed="yes">
+<attribute name="VALUE" x="138.303" y="92.329" size="1.9304" layer="96" font="vector" ratio="10"/>
+</instance>
+<instance part="SUPPLY33" gate="+5V" x="160.02" y="88.9" smashed="yes">
+<attribute name="VALUE" x="158.623" y="92.329" size="1.9304" layer="96" font="vector" ratio="10"/>
+</instance>
+<instance part="C8" gate="G$1" x="180.34" y="78.74"/>
+<instance part="SUPPLY34" gate="GND" x="180.34" y="68.58"/>
+<instance part="SUPPLY35" gate="+5V" x="180.34" y="88.9" smashed="yes">
+<attribute name="VALUE" x="178.943" y="92.329" size="1.9304" layer="96" font="vector" ratio="10"/>
+</instance>
+<instance part="C7" gate="G$1" x="203.2" y="78.74"/>
+<instance part="C9" gate="G$1" x="223.52" y="78.74"/>
+<instance part="SUPPLY36" gate="GND" x="203.2" y="68.58"/>
+<instance part="SUPPLY37" gate="GND" x="223.52" y="68.58"/>
+<instance part="SUPPLY38" gate="+5V" x="203.2" y="88.9" smashed="yes">
+<attribute name="VALUE" x="201.803" y="92.329" size="1.9304" layer="96" font="vector" ratio="10"/>
+</instance>
+<instance part="SUPPLY39" gate="+5V" x="223.52" y="88.9" smashed="yes">
+<attribute name="VALUE" x="222.123" y="92.329" size="1.9304" layer="96" font="vector" ratio="10"/>
+</instance>
+<instance part="C10" gate="G$1" x="243.84" y="78.74"/>
+<instance part="SUPPLY40" gate="GND" x="243.84" y="68.58"/>
+<instance part="SUPPLY41" gate="+5V" x="243.84" y="88.9" smashed="yes">
+<attribute name="VALUE" x="242.443" y="92.329" size="1.9304" layer="96" font="vector" ratio="10"/>
+</instance>
 </instances>
 <busses>
@@
 <wire x1="309.88" y1="167.64" x2="299.72" y2="167.64" width="0.1524" layer="91"/>
 </segment>
+<segment>
+<pinref part="C5" gate="G$1" pin="1"/>
+<pinref part="SUPPLY32" gate="+5V" pin="+5V"/>
+<wire x1="139.7" y1="86.36" x2="139.7" y2="83.82" width="0.1524" layer="91"/>
+</segment>
+<segment>
+<pinref part="C6" gate="G$1" pin="1"/>
+<pinref part="SUPPLY33" gate="+5V" pin="+5V"/>
+<wire x1="160.02" y1="86.36" x2="160.02" y2="83.82" width="0.1524" layer="91"/>
+</segment>
+<segment>
+<pinref part="C8" gate="G$1" pin="1"/>
+<pinref part="SUPPLY35" gate="+5V" pin="+5V"/>
+<wire x1="180.34" y1="86.36" x2="180.34" y2="83.82" width="0.1524" layer="91"/>
+</segment>
+<segment>
+<pinref part="C7" gate="G$1" pin="1"/>
+<pinref part="SUPPLY38" gate="+5V" pin="+5V"/>
+<wire x1="203.2" y1="86.36" x2="203.2" y2="83.82" width="0.1524" layer="91"/>
+</segment>
+<segment>
+<pinref part="C9" gate="G$1" pin="1"/>
+<pinref part="SUPPLY39" gate="+5V" pin="+5V"/>
+<wire x1="223.52" y1="86.36" x2="223.52" y2="83.82" width="0.1524" layer="91"/>
+</segment>
+<segment>
+<pinref part="C10" gate="G$1" pin="1"/>
+<pinref part="SUPPLY41" gate="+5V" pin="+5V"/>
+<wire x1="243.84" y1="86.36" x2="243.84" y2="83.82" width="0.1524" layer="91"/>
+</segment>
 </net>
 <net name="GND" class="0">
@@
 <wire x1="157.48" y1="292.1" x2="132.08" y2="292.1" width="0.1524" layer="91"/>
 </segment>
-</net>
+<segment>
+<pinref part="C5" gate="G$1" pin="2"/>
+<pinref part="SUPPLY30" gate="GND" pin="GND"/>
+<wire x1="139.7" y1="71.12" x2="139.7" y2="73.66" width="0.1524" layer="91"/>
+</segment>
+<segment>
+<pinref part="C6" gate="G$1" pin="2"/>
+<pinref part="SUPPLY31" gate="GND" pin="GND"/>
+<wire x1="160.02" y1="71.12" x2="160.02" y2="73.66" width="0.1524" layer="91"/>
+</segment>
+<segment>
+<pinref part="C8" gate="G$1" pin="2"/>
+<pinref part="SUPPLY34" gate="GND" pin="GND"/>
+<wire x1="180.34" y1="71.12" x2="180.34" y2="73.66" width="0.1524" layer="91"/>
+</segment>
+<segment>
+<pinref part="C7" gate="G$1" pin="2"/>
+<pinref part="SUPPLY36" gate="GND" pin="GND"/>
+<wire x1="203.2" y1="71.12" x2="203.2" y2="73.66" width="0.1524" layer="91"/>
+</segment>
+<segment>
+<pinref part="C9" gate="G$1" pin="2"/>
+<pinref part="SUPPLY37" gate="GND" pin="GND"/>
+<wire x1="223.52" y1="71.12" x2="223.52" y2="73.66" width="0.1524" layer="91"/>
+</segment>
+<segment>
+<pinref part="C10" gate="G$1" pin="2"/>
+<pinref part="SUPPLY40" gate="GND" pin="GND"/>
+<wire x1="243.84" y1="71.12" x2="243.84" y2="73.66" width="0.1524" layer="91"/>
+</segment>
+</net>

Commit message: added logo
Parts:
- added U$1, U$2: FIDUCIAL, adafruit:FIDUCIAL
- C1: value .033 uF -> 0.1uF; device keiths:CAP_5MM -> keiths:CAP0.1UF100V
- C10, C9: value 0.1uF -> 470 pF; device keiths:CAP0.1UF100V -> keiths:CAP_5MM
- C2: value .001 uF -> 0.1uF; device keiths:CAP_5MM -> keiths:CAP0.1UF100V
- C3: value 470 pF -> .033 uF
- C4: value 470 pF -> .001 uF
- U1: value CD74HCT123 -> CD74HC00; device keiths:CD74HCT123 -> keiths:CD74HC00
- U6: value CD74HC00 -> CD74HCT123; device keiths:CD74HC00 -> keiths:CD74HCT123
- renumbered P3 to P1
Connections:
- net +5V: now also C1.1, C2.1, U2.!2CLR, U2.1B, U6.!1CLR, U6.2B; no longer C10.1, C9.1, U1.!1CLR, U1.!2CLR, U1.1B, U1.2B
- net DELAY_SELECT: now also U1.1A, U1.1B, U1.4A, U3.Q3; no longer U4.Q3, U5.1A, U5.1B, U5.4A
- net GND: now also C1.2, C2.2, U6.!1A; no longer C10.2, C9.2, U2.!1A
- net HORIZ_F: now also U5.4Y; no longer U6.4Y
- net HORIZ_U: now also U5.3Y; no longer U6.3Y
- net INTENSIFY: now also U3.Q4, U6.!2CLR; no longer U2.!2CLR, U4.Q4
- net INTENSIFY_P: now also U6.!2Q; no longer U2.!2Q
- net JUMP_DOWN: now also U4.Q1, U5.2B; no longer U3.Q1, U6.2B
- net JUMP_LEFT: now also U4.Q3, U5.3B; no longer U3.Q3, U6.3B
- net JUMP_RIGHT: now also U4.Q2, U5.4B; no longer U3.Q2, U6.4B
- net JUMP_UP: now also U4.Q0, U5.1B; no longer U3.Q0, U6.1B
- net J_INTEN: now also U3.Q2; no longer U4.Q2
- net J_JUMP: now also U3.Q5; no longer U4.Q5
- net K_JUMP: now also U3.Q6; no longer U4.Q6
- net LE1: now also U4.LE; no longer U3.LE
- net LE2: now also U3.LE; no longer U4.LE
- net LE3: now also U1.2B, U1.4B, U6.1B; no longer U2.1B, U5.2B, U5.4B
- net L_JUMP: now also U3.Q7; no longer U4.Q7
- net N$1: now also C3.1, U2.1C; no longer C1.1, U1.1C
- net N$10: now also U1.1Y, U1.2A; no longer U5.1Y, U5.2A
- net N$11: now also U5.1A, U5.2A, U5.3A, U5.4A, U6.1Q; no longer U2.1Q, U6.1A, U6.2A, U6.3A, U6.4A
- net N$12: now also U1.2Y, U2.!2A; no longer U1.!2A, U5.2Y
- net N$13: now also U1.3A, U2.!1Q; no longer U1.!1Q, U5.3A
- net N$14: now also U1.3B, U2.!2Q; no longer U1.!2Q, U5.3B
- net N$15: now also U1.3Y, U6.!2A; no longer U2.!2A, U5.3Y
- net N$2: now also C3.2, U2.1R/C; no longer C1.2, U1.1R/C
- net N$3: now also C4.1, U2.2C; no longer C2.1, U1.2C
- net N$4: now also C4.2, U2.2R/C; no longer C2.2, U1.2R/C
- net N$5: now also C9.1, U6.1C; no longer C4.1, U2.1C
- net N$6: now also C10.2, U6.2R/C; no longer C3.2, U2.2R/C
- net N$7: now also C10.1, U6.2C; no longer C3.1, U2.2C
- net N$8: now also C9.2, U6.1R/C; no longer C4.2, U2.1R/C
- net N$9: now also U1.4Y, U2.!1A; no longer U1.!1A, U5.4Y
- net U_INTEN: now also U3.Q1; no longer U4.Q1
- net VERT_F: now also U5.1Y; no longer U6.1Y
- net VERT_U: now also U5.2Y; no longer U6.2Y
- net X_INTEN: now also U3.Q0; no longer U4.Q0
Other:
- moved on the sheet: C3, C4, C6, C8, U2, U3, U4, U5

Commit message: revised artwork
Parts:
- removed P1: 44PINEDGE, keiths:44PINEDGE
- added P13: 44PINEDGE-M, keiths:44PINEDGE-M
Connections:
- removed net +10V: P1.A
- removed net +15V: P1.E
- removed net -15V: P1.C
- new net FF_J: P13.J
- new net FF_K: P13.K
- new net FF_L: P13.L
- net +5V: now also P13.B; no longer P1.B
- net D0: now also P13.7; no longer P1.7
- net D1: now also P13.8; no longer P1.8
- net D2: now also P13.9; no longer P1.9
- net D3: now also P13.10; no longer P1.10
- net D4: now also P13.11; no longer P1.11
- net D5: now also P13.12; no longer P1.12
- net D6: now also P13.13; no longer P1.13
- net D7: now also P13.14; no longer P1.14
- net GND: now also P13.4, P13.D; no longer P1.D
- net HORIZ_F: now also P13.R; no longer P1.R
- net HORIZ_U: now also P13.S; no longer P1.S
- net INTENSIFY_P: now also P13.X; no longer P1.X
- net J_INTEN: now also P13.V; no longer P1.V
- net J_JUMP: no longer P1.J
- net K_JUMP: no longer P1.K
- net LE1: now also P13.16; no longer P1.16
- net LE2: now also P13.17; no longer P1.17
- net LE3: now also P13.18; no longer P1.18
- net L_JUMP: no longer P1.L
- net U_INTEN: now also P13.W; no longer P1.W
- net VERT_F: now also P13.N; no longer P1.N
- net VERT_U: now also P13.P; no longer P1.P
- net X_INTEN: now also P13.U; no longer P1.U
Other:
- note added: "Parameter Store"
- note removed: "intensity"
- note removed: "scale"
- moved on the sheet: C1, C10, C2, C3, C4, C5, C6, C7, C8, C9, R1, R2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
