File: config_register/system_input.brd (EAGLE design)
At the start: 165.1 x 114.3 mm, 0 parts

Commit message: added logo
Parts:
- added U$1, U$2: FIDUCIAL, adafruit:FIDUCIAL_1MM

Commit message: revised artwork
Parts:
- added P1: 44PINEDGE-M, keiths:44PINEDGE
Connections:
- new net +5V: P1.B
- new net D0: P1.7
- new net D1: P1.8
- new net D2: P1.9
- new net D3: P1.10
- new net D4: P1.11
- new net D5: P1.12
- new net D6: P1.13
- new net D7: P1.14
- new net GND: P1.4, P1.D
- new net LE1: P1.16
- new net LE2: P1.17
- new net LE3: P1.18
- new net X_LSB: P1.20
- new net X_MSB: P1.19
- new net Y_LSB: P1.22
- new net Y_MSB: P1.21
Changed lines of the file:
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@@
 <element name="U$1" library="adafruit" package="FIDUCIAL_1MM" value="FIDUCIAL" x="152.4" y="6.35"/>
 <element name="U$2" library="adafruit" package="FIDUCIAL_1MM" value="FIDUCIAL" x="36.83" y="107.95"/>
+<element name="P1" library="keiths" package="44PINEDGE" value="44PINEDGE-M" x="0" y="57.15" rot="R270"/>
 </elements>
 <signals>
+<signal name="LE1">
+<contactref element="P1" pad="16"/>
+</signal>
+<signal name="D0">
+<contactref element="P1" pad="7"/>
+</signal>
+<signal name="D1">
+<contactref element="P1" pad="8"/>
+</signal>
+<signal name="D2">
+<contactref element="P1" pad="9"/>
+</signal>
+<signal name="D3">
+<contactref element="P1" pad="10"/>
+</signal>
+<signal name="D4">
+<contactref element="P1" pad="11"/>
+</signal>
+<signal name="D5">
+<contactref element="P1" pad="12"/>
+</signal>
+<signal name="D6">
+<contactref element="P1" pad="13"/>
+</signal>
+<signal name="D7">
+<contactref element="P1" pad="14"/>
+</signal>
+<signal name="LE2">
+<contactref element="P1" pad="17"/>
+</signal>
+<signal name="+5V">
+<contactref element="P1" pad="B"/>
+</signal>
+<signal name="GND">
+<contactref element="P1" pad="D"/>
+<contactref element="P1" pad="4"/>
+<wire x1="4.826" y1="86.868" x2="4.826" y2="86.868" width="0" layer="19" extent="1-16"/>
+</signal>
+<signal name="LE3">
+<contactref element="P1" pad="18"/>
+</signal>
+<signal name="Y_LSB">
+<contactref element="P1" pad="22"/>
+</signal>
+<signal name="X_MSB">
+<contactref element="P1" pad="19"/>
+</signal>
+<signal name="Y_MSB">
+<contactref element="P1" pad="21"/>
+</signal>
+<signal name="X_LSB">
+<contactref element="P1" pad="20"/>
+</signal>
 </signals>
 </board>
