File: config_register/system_input.sch (EAGLE design)
At the start: 0 parts

Commit message: added logo
Parts:
- added U$1, U$2: FIDUCIAL, adafruit:FIDUCIAL
Changed lines of the file:
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@@
 <parts>
 <part name="FRAME1" library="frames" deviceset="FRAME_C_L" device=""/>
+<part name="U$1" library="adafruit" deviceset="FIDUCIAL" device=""/>
+<part name="U$2" library="adafruit" deviceset="FIDUCIAL" device=""/>
 </parts>
 <sheets>
@@
 <instance part="FRAME1" gate="G$1" x="0" y="0"/>
 <instance part="FRAME1" gate="G$2" x="452.12" y="0"/>
+<instance part="U$1" gate="G$1" x="454.66" y="401.32"/>
+<instance part="U$2" gate="G$1" x="472.44" y="401.32"/>
 </instances>
 <busses>

Commit message: revised artwork
Parts:
- added P1: 44PINEDGE-M, keiths:44PINEDGE-M
Connections:
- new net +5V: P1.B
- new net D0: P1.7
- new net D1: P1.8
- new net D2: P1.9
- new net D3: P1.10
- new net D4: P1.11
- new net D5: P1.12
- new net D6: P1.13
- new net D7: P1.14
- new net GND: P1.4, P1.D
- new net LE1: P1.16
- new net LE2: P1.17
- new net LE3: P1.18
- new net X_LSB: P1.20
- new net X_MSB: P1.19
- new net Y_LSB: P1.22
- new net Y_MSB: P1.21
Other:
- note added: "Brain Bus"
Changed lines of the file:
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@@
 <part name="U$1" library="adafruit" deviceset="FIDUCIAL" device=""/>
 <part name="U$2" library="adafruit" deviceset="FIDUCIAL" device=""/>
+<part name="SUPPLY19" library="keiths" deviceset="+5V" device=""/>
+<part name="SUPPLY20" library="keiths" deviceset="GND" device=""/>
+<part name="SUPPLY24" library="keiths" deviceset="GND" device=""/>
+<part name="P1" library="keiths" deviceset="44PINEDGE-M" device=""/>
 </parts>
 <sheets>
 <sheet>
 <plain>
+<text x="109.22" y="317.5" size="2.1844" layer="91" font="vector" ratio="10">Brain Bus</text>
 </plain>
 <instances>
@@
 <instance part="U$1" gate="G$1" x="454.66" y="401.32"/>
 <instance part="U$2" gate="G$1" x="472.44" y="401.32"/>
+<instance part="SUPPLY19" gate="+5V" x="152.4" y="378.46" smashed="yes" rot="R270">
+<attribute name="VALUE" x="155.829" y="377.317" size="1.9304" layer="96" font="vector" ratio="10"/>
+</instance>
+<instance part="SUPPLY20" gate="GND" x="152.4" y="373.38" smashed="yes" rot="R90">
+<attribute name="VALUE" x="155.829" y="372.745" size="1.9304" layer="96" font="vector" ratio="10"/>
+</instance>
+<instance part="SUPPLY24" gate="GND" x="81.28" y="373.38" smashed="yes" rot="MR90">
+<attribute name="VALUE" x="77.851" y="372.745" size="1.9304" layer="96" font="vector" ratio="10" rot="MR0"/>
+</instance>
+<instance part="P1" gate="G$1" x="116.84" y="355.6"/>
 </instances>
 <busses>
 </busses>
 <nets>
+<net name="LE1" class="0">
+<segment>
+<wire x1="99.06" y1="342.9" x2="106.68" y2="342.9" width="0.1524" layer="91"/>
+<label x="99.06" y="342.9" size="1.9304" layer="95" font="vector" ratio="10" rot="MR0" xref="yes"/>
+<pinref part="P1" gate="G$1" pin="16"/>
+</segment>
+</net>
+<net name="D0" class="0">
+<segment>
+<label x="83.82" y="365.76" size="1.9304" layer="95" font="vector" ratio="10" rot="MR0" xref="yes"/>
+<wire x1="83.82" y1="365.76" x2="106.68" y2="365.76" width="0.1524" layer="91"/>
+<pinref part="P1" gate="G$1" pin="7"/>
+</segment>
+</net>
+<net name="D1" class="0">
+<segment>
+<label x="99.06" y="363.22" size="1.9304" layer="95" font="vector" ratio="10" rot="MR0" xref="yes"/>
+<wire x1="99.06" y1="363.22" x2="106.68" y2="363.22" width="0.1524" layer="91"/>
+<pinref part="P1" gate="G$1" pin="8"/>
+</segment>
+</net>
+<net name="D2" class="0">
+<segment>
+<label x="83.82" y="360.68" size="1.9304" layer="95" font="vector" ratio="10" rot="MR0" xref="yes"/>
+<wire x1="83.82" y1="360.68" x2="106.68" y2="360.68" width="0.1524" layer="91"/>
+<pinref part="P1" gate="G$1" pin="9"/>
+</segment>
+</net>
+<net name="D3" class="0">
+<segment>
+<label x="99.06" y="358.14" size="1.9304" layer="95" font="vector" ratio="10" rot="MR0" xref="yes"/>
+<wire x1="99.06" y1="358.14" x2="106.68" y2="358.14" width="0.1524" layer="91"/>
+<pinref part="P1" gate="G$1" pin="10"/>
+</segment>
+</net>
+<net name="D4" class="0">
+<segment>
+<wire x1="106.68" y1="355.6" x2="83.82" y2="355.6" width="0.1524" layer="91"/>
+<label x="83.82" y="355.6" size="1.9304" layer="95" font="vector" ratio="10" rot="MR0" xref="yes"/>
+<pinref part="P1" gate="G$1" pin="11"/>
+</segment>
+</net>
+<net name="D5" class="0">
+<segment>
+<wire x1="99.06" y1="353.06" x2="106.68" y2="353.06" width="0.1524" layer="91"/>
+<label x="99.06" y="353.06" size="1.9304" layer="95" font="vector" ratio="10" rot="MR0" xref="yes"/>
+<pinref part="P1" gate="G$1" pin="12"/>
+</segment>
+</net>
+<net name="D6" class="0">
+<segment>
+<wire x1="83.82" y1="350.52" x2="106.68" y2="350.52" width="0.1524" layer="91"/>
+<label x="83.82" y="350.52" size="1.9304" layer="95" font="vector" ratio="10" rot="MR0" xref="yes"/>
+<pinref part="P1" gate="G$1" pin="13"/>
+</segment>
+</net>
+<net name="D7" class="0">
+<segment>
+<label x="99.06" y="347.98" size="1.9304" layer="95" font="vector" ratio="10" rot="MR0" xref="yes"/>
+<wire x1="99.06" y1="347.98" x2="106.68" y2="347.98" width="0.1524" layer="91"/>
+<pinref part="P1" gate="G$1" pin="14"/>
+</segment>
+</net>
+<net name="LE2" class="0">
+<segment>
+<wire x1="106.68" y1="340.36" x2="83.82" y2="340.36" width="0.1524" layer="91"/>
+<label x="83.82" y="340.36" size="1.9304" layer="95" font="vector" ratio="10" rot="MR0" xref="yes"/>
+<pinref part="P1" gate="G$1" pin="17"/>
+</segment>
+</net>
+<net name="+5V" class="0">
+<segment>
+<pinref part="SUPPLY19" gate="+5V" pin="+5V"/>
+<wire x1="149.86" y1="378.46" x2="127" y2="378.46" width="0.1524" layer="91"/>
+<pinref part="P1" gate="G$1" pin="B"/>
+</segment>
+</net>
+<net name="GND" class="0">
+<segment>
+<pinref part="SUPPLY20" gate="GND" pin="GND"/>
+<wire x1="149.86" y1="373.38" x2="127" y2="373.38" width="0.1524" layer="91"/>
+<pinref part="P1" gate="G$1" pin="D"/>
+</segment>
+<segment>
+<pinref part="SUPPLY24" gate="GND" pin="GND"/>
+<wire x1="83.82" y1="373.38" x2="106.68" y2="373.38" width="0.1524" layer="91"/>
+<pinref part="P1" gate="G$1" pin="4"/>
+</segment>
+</net>
+<net name="LE3" class="0">
+<segment>
+<wire x1="106.68" y1="337.82" x2="99.06" y2="337.82" width="0.1524" layer="91"/>
+<label x="99.06" y="337.82" size="1.9304" layer="95" font="vector" ratio="10" rot="MR0" xref="yes"/>
+<pinref part="P1" gate="G$1" pin="18"/>
+</segment>
+</net>
+<net name="Y_LSB" class="0">
+<segment>
+<wire x1="106.68" y1="327.66" x2="99.06" y2="327.66" width="0.1524" layer="91"/>
+<label x="99.06" y="327.66" size="1.9304" layer="95" font="vector" ratio="10" rot="MR0" xref="yes"/>
+<pinref part="P1" gate="G$1" pin="22"/>
+</segment>
+</net>
+<net name="X_MSB" class="0">
+<segment>
+<wire x1="83.82" y1="335.28" x2="106.68" y2="335.28" width="0.1524" layer="91"/>
+<label x="83.82" y="335.28" size="1.9304" layer="95" font="vector" ratio="10" rot="MR0" xref="yes"/>
+<pinref part="P1" gate="G$1" pin="19"/>
+</segment>
+</net>
+<net name="Y_MSB" class="0">
+<segment>
+<wire x1="106.68" y1="330.2" x2="83.82" y2="330.2" width="0.1524" layer="91"/>
+<label x="83.82" y="330.2" size="1.9304" layer="95" font="vector" ratio="10" rot="MR0" xref="yes"/>
+<pinref part="P1" gate="G$1" pin="21"/>
+</segment>
+</net>
+<net name="X_LSB" class="0">
+<segment>
+<wire x1="106.68" y1="332.74" x2="99.06" y2="332.74" width="0.1524" layer="91"/>
+<label x="99.06" y="332.74" size="1.9304" layer="95" font="vector" ratio="10" rot="MR0" xref="yes"/>
+<pinref part="P1" gate="G$1" pin="20"/>
+</segment>
+</net>
 </nets>
 </sheet>
