File: tube_neck/mimic1705.sch (EAGLE design)
At the start: 25 parts, among them J1 WM5238, J2 WM5235, J3 WM5236, P1 44PINEDGE, P3 1M

Commit message: EOD backup
Parts:
- removed P3: 1M, keiths:POT-3006P
- removed ZD2, ZD3: 1N5271, keiths:1N754A
- removed ZD4, ZD5: BZX79-C56, keiths:1N754A
- added D1, D4: 1N4764, keiths:1N4764A
- added D5, D6: BZV85-C56,113, keiths:BZV85-C56,113
- added J5: JST-VH-3, keiths:JST-VH-3
- added P2: 1 M, keiths:POT-3006P
- J1: value WM5238 -> JST-VH-2; device keiths:WM5238 -> keiths:JST-VH-2
- J2: value WM5235 -> JST-VH-5; device keiths:WM5235 -> keiths:JST-VH-5
- J3: value WM5236 -> JST-VH-3; device keiths:WM5236 -> keiths:JST-VH-3
Connections:
- removed net +50V: P1.E
- removed net BASE: P1.K
- net -150V: now also J5.3; no longer P1.V
- net 6.3_VAC_1: now also J1.1; no longer J2.1
- net 6.3_VAC_2: now also J1.2, J2.5; no longer J1.5, J2.2
- net CATHODE: now also J2.2, J5.1; no longer J1.2, P1.Y
- net GND: now also D4.A, D6.C, J5.2, P2.1; no longer P3.A, ZD2.A, ZD5.C
- net GRID1: now also J2.3, P2.2; no longer J1.3, P3.S
- net GRID2: now also D1.C, J2.1; no longer J1.1, ZD3.C
- net HEATER: now also J2.4; no longer J1.4
- net N$1: now also D5.C, D6.A; no longer ZD4.C, ZD5.A
- net N$2: now also D1.A, D4.C; no longer ZD2.C, ZD3.A
- net N$7: now also D5.A, P2.3; no longer P3.E, ZD4.A
Other:
- note added: "100 Volt Zeners"
- note added: "60 Volt Zeners"
- note added: "Tube Socket"
- note added: "mimic4688"
- note removed: "Tube Neck"
- note removed: "set for 2mA"
- moved on the sheet: C1, C4, D2, D3, J3, P1, R10, R11, R12, R13, R4, R5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

Commit message: end of day
Parts:
- P2: value 1 M -> 1M
- renumbered P1 to P20
Changed lines of the file:
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@@
 <part name="FRAME1" library="frames" deviceset="FRAME_C_L" device=""/>
 <part name="FRAME2" library="frames" deviceset="FRAME_C_L" device=""/>
-<part name="P1" library="keiths" deviceset="44PINEDGE" device=""/>
+<part name="P20" library="keiths" deviceset="44PINEDGE" device=""/>
 <part name="R4" library="keiths" deviceset="RES-V" device="" value="220K"/>
 <part name="SUPPLY1" library="keiths" deviceset="GND" device=""/>
@@
 <part name="J3" library="keiths" deviceset="JST-VH-3" device=""/>
 <part name="J1" library="keiths" deviceset="JST-VH-2" device=""/>
-<part name="P2" library="keiths" deviceset="POT-3006P" device="" value="1 M"/>
+<part name="P2" library="keiths" deviceset="POT-3006P" device="" value="1M"/>
 <part name="J2" library="keiths" deviceset="JST-VH-5" device=""/>
 <part name="D1" library="keiths" deviceset="1N4764A" device="" value="1N4764"/>
@@
 <instance part="FRAME1" gate="G$1" x="0" y="0"/>
 <instance part="FRAME2" gate="G$2" x="452.12" y="0"/>
-<instance part="P1" gate="G$1" x="271.78" y="345.44"/>
+<instance part="P20" gate="G$1" x="271.78" y="345.44"/>
 <instance part="R4" gate="G$1" x="299.72" y="106.68"/>
 <instance part="SUPPLY1" gate="GND" x="299.72" y="60.96"/>
@@
 <wire x1="281.94" y1="363.22" x2="289.56" y2="363.22" width="0.1524" layer="91"/>
 <label x="289.56" y="363.22" size="1.9304" layer="95" font="vector" ratio="10" xref="yes"/>
-<pinref part="P1" gate="G$1" pin="D"/>
+<pinref part="P20" gate="G$1" pin="D"/>
 </segment>
 <segment>
