File: tube_neck/mimic1705.brd (EAGLE design)
At the start: 152.4 x 114.3 mm, 25 parts, among them J1 WM5238, J2 WM5235, J3 WM5236, P1 44PINEDGE, P3 1M

Commit message: EOD backup
Parts:
- removed P3: 1M, keiths:3006P
- removed ZD2, ZD3: 1N5271, keiths:DO35-7
- removed ZD4, ZD5: BZX79-C56, keiths:DO35-7
- added D1, D4: 1N4764, keiths:DO-41-10
- added D5, D6: BZV85-C56,113, keiths:DO-41-10
- added J5: JST-VH-3, keiths:VHR-3N
- added P2: 1 M, keiths:3006P
- J1: value WM5238 -> JST-VH-2; device keiths:MOLEX-WM5238 -> keiths:VHR-2N
- J2: value WM5235 -> JST-VH-5; device keiths:MOLEX-WM5235 -> keiths:VHR-5N
- J3: value WM5236 -> JST-VH-3; device keiths:MOLEX-WM5236 -> keiths:VHR-3N
- moved J1 30.2 mm to (141.0, 68.6), turned to 0 degrees
- moved J3 11.7 mm to (141.0, 83.8), turned to 0 degrees
- moved J2 11.5 mm to (141.0, 15.2), turned to 0 degrees
Connections:
- removed net +50V: P1.E
- removed net BASE: P1.K
- net +265V: now also J3.P$1; no longer J3.1
- net -150V: now also J3.P$3, J5.P$3; no longer J3.3, P1.V
- net 6.3_VAC_1: now also J1.P$1; no longer J2.1
- net 6.3_VAC_2: now also J1.P$2, J2.P$5; no longer J1.5, J2.2
- net CATHODE: now also J2.P$2, J5.P$1; no longer J1.2, P1.Y
- net GND: now also D4.A, D6.C, J3.P$2, J5.P$2, P2.1; no longer J3.2, P3.1, ZD2.A, ZD5.C
- net GRID1: now also J2.P$3, P2.2; no longer J1.3, P3.2
- net GRID2: now also D1.C, J2.P$1; no longer J1.1, ZD3.C
- net HEATER: now also J2.P$4; no longer J1.4
- net N$1: now also D5.C, D6.A; no longer ZD4.C, ZD5.A
- net N$2: now also D1.A, D4.C; no longer ZD2.C, ZD3.A
- net N$7: now also D5.A, P2.3; no longer P3.3, ZD4.A

Commit message: end of day
Parts:
- P2: value 1 M -> 1M
- moved D3 115.4 mm to (135.9, 93.8), turned to 90 degrees
- moved R4 103.4 mm to (123.2, 101.6), turned to 270 degrees
- moved D2 98.5 mm to (125.7, 54.6), turned to 180 degrees
- moved D4 97.4 mm to (102.9, 101.6), turned to 270 degrees
- moved D1 96.7 mm to (113.0, 101.6), turned to 90 degrees
- moved C1 86.5 mm to (127.0, 82.3), turned to 270 degrees
- moved R10 85.1 mm to (35.6, 86.4), turned to 180 degrees
- moved R11 79.3 mm to (55.9, 86.4), turned to 180 degrees
- moved J2 78.5 mm to (153.7, 92.7)
- moved R6 75.0 mm to (96.5, 77.5), turned to 0 degrees
- moved R12 73.9 mm to (76.2, 86.4), turned to 180 degrees
- moved R9 72.6 mm to (35.6, 77.5), turned to 0 degrees
- moved R13 70.3 mm to (96.5, 86.4), turned to 180 degrees
- moved R5 70.0 mm to (76.2, 101.6), turned to 90 degrees
- moved R7 60.7 mm to (76.2, 77.5), turned to 0 degrees
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- renumbered P1 to P20
Routing:
- net GND: track 0.00 -> 320.6 mm
- net +265V: track 0.00 -> 88.6 mm
- net N$8: track 0.00 -> 78.9 mm
- net CATHODE: track 0.00 -> 68.0 mm
- net HEATER: track 0.00 -> 67.4 mm
- net GRID1: track 0.00 -> 62.7 mm
- net GRID2: track 0.00 -> 48.2 mm
- net 6.3_VAC_1: track 0.00 -> 44.2 mm
- net -150V: track 0.00 -> 34.9 mm
- net 6.3_VAC_2: track 0.00 -> 27.4 mm
- net N$1: track 0.00 -> 27.3 mm
- net N$7: track 0.00 -> 24.1 mm
- net N$2: track 0.00 -> 10.2 mm
- net N$11: track 0.00 -> 8.39 mm
- net N$5: track 0.00 -> 7.62 mm
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Other:
- board size 152.4 x 114.3 mm -> 165.1 x 114.3 mm

Commit message: end of day
Parts:
- moved C3 29.7 mm to (99.1, 66.0), turned to 0 degrees
- moved C2 18.9 mm to (99.1, 50.8), turned to 0 degrees
- moved D2 8.52 mm to (118.1, 58.4)
Routing:
- net GND: track 320.6 -> 309.7 mm
- net -150V: track 34.9 -> 42.5 mm
- net +265V: track 88.6 -> 85.7 mm
- net HEATER: track 67.4 -> 66.6 mm
- net 6.3_VAC_2: track 27.4 -> 27.9 mm
