File: tube_neck/mimic4688.brd (EAGLE design)
At the start: 160 x 100 mm, 56 parts, among them P1 44PINEDGE, Q1 2N3906, Q10 2N3906, Q11 2N3906, Q5 2N3904, Q7 2N3906, Q8 2N3906, Q9 2N3906

Commit message: EOD backup
Parts:
- added J1: JST-VH-3, keiths:VHR-3N
Connections:
- net +5V: now also P1.B; no longer P1.F
- net -150V: now also J1.P$3; no longer P1.V
- net CATHODE: now also J1.P$1
- net GND: now also J1.P$2
Changed lines of the file:
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@@
 <element name="R8" library="keiths" package="0207/10" value="2.2K" x="-43.18" y="63.5"/>
 <element name="R9" library="keiths" package="0207/10" value="3.3K" x="-67.31" y="63.5"/>
+<element name="J1" library="keiths" package="VHR-3N" value="JST-VH-3" x="-101.6" y="-15.24"/>
 </elements>
 <signals>
@@
 <contactref element="R28" pad="1"/>
 <contactref element="P1" pad="D"/>
+<contactref element="J1" pad="P$2"/>
+<wire x1="-98.298" y1="6.096" x2="-110.6" y2="-15.24" width="0" layer="19" extent="16-16"/>
 <wire x1="-95.25" y1="21.59" x2="-98.298" y2="6.096" width="0" layer="19" extent="16-16"/>
 <wire x1="-87.63" y1="21.59" x2="-95.25" y2="21.59" width="0" layer="19" extent="1-1"/>
@@
 <contactref element="R6" pad="1"/>
 <contactref element="Q9" pad="3"/>
-<contactref element="P1" pad="F"/>
-<wire x1="-80.01" y1="21.59" x2="-90.3732" y2="6.096" width="0" layer="19" extent="16-16"/>
+<contactref element="P1" pad="B"/>
+<wire x1="-80.01" y1="21.59" x2="-106.2228" y2="6.096" width="0" layer="19" extent="16-16"/>
 <wire x1="-72.39" y1="21.59" x2="-80.01" y2="21.59" width="0" layer="19" extent="1-1"/>
 <wire x1="-64.77" y1="21.59" x2="-72.39" y2="21.59" width="0" layer="19" extent="1-1"/>
@@
 <contactref element="R20" pad="2"/>
 <contactref element="R21" pad="2"/>
-<contactref element="P1" pad="V"/>
-<wire x1="-29.21" y1="21.59" x2="-42.8244" y2="6.096" width="0" layer="19" extent="16-16"/>
+<contactref element="J1" pad="P$3"/>
+<wire x1="-29.21" y1="21.59" x2="-110.6" y2="-11.27125" width="0" layer="19" extent="1-1"/>
 <wire x1="-13.97" y1="21.59" x2="-29.21" y2="21.59" width="0" layer="19" extent="1-1"/>
 </signal>
@@
 <contactref element="R28" pad="2"/>
 <contactref element="P1" pad="Z"/>
-<wire x1="-30.44" y1="31.75" x2="-17.78" y2="49.53" width="0" layer="19" extent="1-1"/>
-<wire x1="-26.9748" y1="6.096" x2="-30.44" y2="31.75" width="0" layer="19" extent="16-16"/>
+<contactref element="J1" pad="P$1"/>
+<wire x1="-26.9748" y1="6.096" x2="-110.6" y2="-19.20875" width="0" layer="19" extent="16-16"/>
+<wire x1="-30.44" y1="31.75" x2="-26.9748" y2="6.096" width="0" layer="19" extent="16-16"/>
+<wire x1="-17.78" y1="49.53" x2="-30.44" y2="31.75" width="0" layer="19" extent="1-1"/>
 <wire x1="-86.36" y1="93.98" x2="-17.78" y2="49.53" width="0" layer="19" extent="1-1"/>
 </signal>

Commit message: end of day
Parts:
- removed D10, D12, D14, D15, D4, D5: 1N4148, keiths:DO35-7
- removed Q8: 2N3906, keiths:TO92
- removed R32, R33: 4.7K, keiths:0207/10
- added Q2, Q4: 2N3904, keiths:TO92
- added Q3, Q6: 2N3906, keiths:TO92
- added R29: 12.7K, keiths:0207/10
- added R30: 23.7K, keiths:0207/10
- Q7: value 2N3906 -> 2N3904
- R1: value 11K -> 11.3K
- R16: value 12.1K -> 20K
- R17: value 11.5K -> 11.3K
- R2: value 4.7K -> 10K
- R22: value 23.2K -> 10K
- R23: value 22.6K -> 60.4K
- R24: value 47.5K -> 95.3K
- R25: value 48.7K -> 10.7K
- R26: value 86.6K -> 12.1K
- R27: value 14.7K -> 20K
- R3: value 4.7K -> 18.7K
- R4: value 5.6K -> 60.4K
- R5: value 4.7K -> 20K
- R6: value 4.7K -> 11.3K
- R7: value 27K -> 10K
- moved J1 280.7 mm to (153.7, 101.6)
- moved R6 218.7 mm to (118.1, 47.0), turned to 90 degrees
- moved R28 217.5 mm to (125.7, 106.7)
- moved Q11 217.3 mm to (111.8, 90.2), turned to 45 degrees
- moved Q9 215.9 mm to (134.6, 53.3), turned to 45 degrees
- moved R18 204.5 mm to (113.0, 78.7)
- moved D1 204.3 mm to (161.3, 53.3), turned to 270 degrees
- moved R5 200.8 mm to (133.3, 63.5)
- moved R26 186.4 mm to (134.6, 38.1), turned to 90 degrees
- moved C3 184.9 mm to (149.9, 82.5)
- moved D11 182.6 mm to (87.6, 76.2)
- moved R2 177.8 mm to (92.7, 48.3), turned to 270 degrees
- moved R21 175.1 mm to (130.8, 76.2)
- moved R25 174.7 mm to (146.1, 36.8), turned to 90 degrees
- moved D2 167.9 mm to (111.8, 40.6), turned to 270 degrees
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Connections:
- removed net +5V: P1.B, Q7.3, Q8.3, Q9.3, R3.1, R33.1, R6.1
- removed net N$31: D10.C, Q8.2, R32.2, R33.2
- removed net N$4: D2.A, D3.C, Q7.1, R4.1
- new net N$16: D3.A, Q6.3, R23.2, R24.2
- new net N$22: Q7.1, R27.1
- net +10V: now also Q2.3, Q4.3, Q7.3, R1.1, R29.1, R3.1, R30.1, R4.1, R6.1; no longer R16.2, R22.1, R27.2
- net -15V: now also Q3.1, Q6.1, Q9.1, R2.2, R22.2; no longer R1.2, R4.2
- net J_IN: now also Q7.2; no longer R2.1
- net N$10: now also Q4.1, R16.1; no longer D12.A, D3.A, R17.2, R22.2
- net N$11: now also Q5.1; no longer Q5.3
- net N$13: now also Q6.2, R17.2, R22.1, R27.2; no longer D14.A, D15.A, R23.2, R24.2
- net N$17: now also Q9.3; no longer D5.A
- net N$2: now also Q3.2, R1.2, R16.2, R2.1; no longer D2.C, Q7.2, R2.2, R3.2
- net N$21: now also D2.C, D3.C, R29.2, R30.2; no longer D12.C, D15.C, R16.1, R27.1
- net N$3: now also D2.A, Q3.3, R3.2, R4.2; no longer D10.A, D14.C, Q8.1, R1.1
- net N$5: now also R7.1; no longer D4.C
- net N$6: now also Q2.1, R5.1; no longer D4.A, D5.C, Q9.1, R7.1
- net N$9: now also Q5.3; no longer Q5.1
- net U_IN: now also Q4.2; no longer R32.1
- net X_IN: now also Q2.2; no longer R5.1
Routing:
- net +10V: track 0.00 -> 57.4 mm
- net N$13: track 0.00 -> 33.8 mm
- net N$16: track 0.00 -> 21.1 mm
- net N$21: track 0.00 -> 15.2 mm
- net N$22: track 0.00 -> 11.5 mm
- net J_IN: track 0.00 -> 9.89 mm
- net -15V: track 0.00 -> 8.91 mm
Other:
- board size 160 x 100 mm -> 165.1 x 114.3 mm
