File: tube_neck/mimic4688.sch (EAGLE design)
At the start: 56 parts, among them P1 44PINEDGE, Q1 2N3906, Q10 2N3906, Q11 2N3906, Q5 2N3904, Q7 2N3906, Q8 2N3906, Q9 2N3906

Commit message: EOD backup
Parts:
- added J1: JST-VH-3, keiths:JST-VH-3
Connections:
- net +5V: now also P1.B; no longer P1.F
- net -150V: now also J1.3; no longer P1.V
- net CATHODE: now also J1.1
- net GND: now also J1.2
Other:
- note added: "Connector to mimic1705 bias."
- note added: "Plus 5 Volts on P_IN sets CATHODE to 0 volts placing the CATHODE in cut-off. GRID ONE being negative at about 80 volts requires the cathode be moved negative from ground to reduce cut-off bias between CATHODE and grid and enable emission."
- note removed: "+5 Volts on P_IN will cause CATHODE to be set to 0 volts."
- moved on the sheet: C1, C2, C3, D1, D10, D11, D12, D13, D14, D15, D2, D3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

Commit message: end of day
Parts:
- removed D10, D12, D14, D15, D4, D5: 1N4148, keiths:1N4148
- removed Q8: 2N3906, keiths:2N3906
- removed R32, R33: 4.7K, keiths:R-1/4WATT
- added Q2, Q4: 2N3904, keiths:2N3904
- added Q3, Q6: 2N3906, keiths:2N3906
- added R29: 12.7K, keiths:R-1/4WATT
- added R30: 23.7K, keiths:R-1/4WATT
- Q7: value 2N3906 -> 2N3904; device keiths:2N3906 -> keiths:2N3904
- R1: value 11K -> 11.3K
- R16: value 12.1K -> 20K
- R17: value 11.5K -> 11.3K
- R2: value 4.7K -> 10K
- R22: value 23.2K -> 10K
- R23: value 22.6K -> 60.4K
- R24: value 47.5K -> 95.3K
- R25: value 48.7K -> 10.7K
- R26: value 86.6K -> 12.1K
- R27: value 14.7K -> 20K
- R3: value 4.7K -> 18.7K
- R4: value 5.6K -> 60.4K
- R5: value 4.7K -> 20K
- R6: value 4.7K -> 11.3K
- R7: value 27K -> 10K
Connections:
- removed net +5V: P1.B, Q7.E, Q8.E, Q9.E, R3.P$1, R33.P$1, R6.P$1
- removed net N$31: D10.C, Q8.B, R32.P$2, R33.P$2
- removed net N$4: D2.A, D3.C, Q7.C, R4.P$1
- new net N$16: D3.A, Q6.E, R23.P$2, R24.P$2
- new net N$22: Q7.E, R27.P$1
- net +10V: now also Q2.C, Q4.C, Q7.C, R1.P$1, R29.P$1, R3.P$1, R30.P$1, R4.P$1, R6.P$1; no longer R16.P$2, R22.P$1, R27.P$2
- net -15V: now also Q3.C, Q6.C, Q9.C, R2.P$2, R22.P$2; no longer R1.P$2, R4.P$2
- net J_IN: now also Q7.B; no longer R2.P$1
- net N$10: now also Q4.E, R16.P$1; no longer D12.A, D3.A, R17.P$2, R22.P$2
- net N$13: now also Q6.B, R17.P$2, R22.P$1, R27.P$2; no longer D14.A, D15.A, R23.P$2, R24.P$2
- net N$17: now also Q9.E; no longer D5.A
- net N$2: now also Q3.B, R1.P$2, R16.P$2, R2.P$1; no longer D2.C, Q7.B, R2.P$2, R3.P$2
- net N$21: now also D2.C, D3.C, R29.P$2, R30.P$2; no longer D12.C, D15.C, R16.P$1, R27.P$1
- net N$3: now also D2.A, Q3.E, R3.P$2, R4.P$2; no longer D10.A, D14.C, Q8.C, R1.P$1
- net N$5: now also R7.P$1; no longer D4.C
- net N$6: now also Q2.E, R5.P$1; no longer D4.A, D5.C, Q9.C, R7.P$1
- net U_IN: now also Q4.B; no longer R32.P$1
- net X_IN: now also Q2.B; no longer R5.P$1
Other:
- note added: "+5V +5V +5V GND -26.1 Volts"
- note added: "+5V +5V GND GND -25.4 Volts"
- note added: "+5V GND +5V GND -24.4 Volts"
- note added: "+5V GND GND GND -23.4 Volts"
- note added: "GND +5V +5V GND -21.3 Volts"
- note added: "GND +5V GND GND -19.9 Volts"
- note added: "GND GND +5V GND -18.2 Volts"
- note added: "GND GND GND GND -16.4 Volts"
- note added: "Plus 5 Volts on P_IN sets CATHODE to ground and cuts-off CATHODE. GRID ONE being negative requires the cathode be moved negative from ground to reduce cut-off bias to enable emission."
- note removed: "+5V +5V +5V GND -18.2 Volts"
- note removed: "+5V +5V GND GND -21.8 Volts"
- note removed: "+5V GND +5V GND -25.5 Volts"
- note removed: "+5V GND GND GND -29.1 Volts"
- note removed: "GND +5V +5V GND -32.7 Volts"
- note removed: "GND +5V GND GND -36.2 Volts"
- note removed: "GND GND +5V GND -40.0 Volts"
- note removed: "GND GND GND GND -43.6 Volts"
- note removed: "Plus 5 Volts on P_IN sets CATHODE to 0 volts placing the CATHODE in cut-off. GRID ONE being negative at about 80 volts requires the cathode be moved negative from ground to reduce cut-off bias between CATHODE and grid and enable emission."
- moved on the sheet: C1, C2, D1, D2, D3, D6, D7, D8, D9, Q10, Q11, Q9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
