File: neck/mimic1705.brd (EAGLE design)
At the start: 165.1 x 114.3 mm, 26 parts, among them J1 JST-VH-2, J2 JST-VH-5, J3 JST-VH-3, J5 JST-VH-3, P2 1M, P20 44PINEDGE

Commit message: card layouts finished
Parts:
- removed P20: 44PINEDGE, keiths:44PINEDGE
- removed R11, R12, R13: 0.33, keiths:0309/12
- added P1: 1M, keiths:3006P
- added R1: 18K, keiths:0207/10
- added R2: 220K, keiths:0207/10
- added R3: 0.33, keiths:0309/12
- C2: value 22 uF -> 0.01UF; device keiths:AXIAL10X26 -> keiths:5MM_TH
- C4: value 0.01UF -> 22 uF; device keiths:5MM_TH -> keiths:AXIAL10X26
- D1, D4: value 1N4764 -> BZV85-C56,113
- D2, D3: value 1N4005 -> 1N4764
- D5, D6: value BZV85-C56,113 -> 1N4005
- J1: value JST-VH-2 -> JST-VH-5; device keiths:VHR-2N -> keiths:VHR-5N
- J2: value JST-VH-5 -> JST-VH-2; device keiths:VHR-5N -> keiths:VHR-2N
- P2: value 1M -> 44PINEDGE; device keiths:3006P -> keiths:44PINEDGE
- R4: value 220K -> 0.33; device keiths:0207/10 -> keiths:0309/12
- R5: value 18K -> 0.33; device keiths:0207/10 -> keiths:0309/12
- moved P2 98.9 mm to (0.00, 57.1), turned to 270 degrees
- moved D6 88.7 mm to (118.1, 58.4), turned to 180 degrees
- moved D5 71.9 mm to (135.9, 93.8)
- moved R4 69.0 mm to (55.9, 86.4), turned to 180 degrees
- moved D4 62.3 mm to (40.6, 99.1), turned to 90 degrees
- moved R10 61.6 mm to (96.5, 77.5), turned to 0 degrees
- moved C4 54.8 mm to (99.1, 50.8), turned to 0 degrees
- moved D1 48.3 mm to (64.8, 104.1)
- moved D2 45.8 mm to (102.9, 101.6), turned to 270 degrees
- moved C2 42.1 mm to (127.0, 82.3), turned to 270 degrees
- moved R7 40.6 mm to (35.6, 77.5)
- moved R9 40.6 mm to (76.2, 77.5)
- moved D3 25.4 mm to (111.8, 101.6)
- moved J1 19.0 mm to (153.7, 92.7)
- moved J2 19.0 mm to (153.7, 73.7)
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- renumbered J5 to J4
Connections:
- net +265V: now also R2.2; no longer R4.1
- net -150V: now also D6.C; no longer D2.C
- net 6.3_VAC_1: now also J2.P$1, R10.2; no longer J1.P$1, R6.2
- net 6.3_VAC_2: now also J1.P$5, J2.P$2; no longer J1.P$2, J2.P$5
- net CATHODE: now also D5.C, J1.P$2; no longer D3.C, J2.P$2
- net GND: now also C2.2, C4.P$1, D2.A, D4.C, P1.1, P2.D; no longer C2.P$1, C4.2, D4.A, D6.C, P2.1, P20.D
- net GRID1: now also C1.1, D5.A, J1.P$3, P1.2; no longer C4.1, D3.A, J2.P$3, P2.2
- net GRID2: now also C2.1, D3.C, J1.P$1, R2.1; no longer C1.1, D1.C, J2.P$1, R4.2
- net HEATER: now also J1.P$4, R6.1; no longer J2.P$4, R13.1
- net N$1: now also D1.C, D4.A; no longer D5.C, D6.A
- net N$10: now also R7.2; no longer R9.2
- net N$11: now also R3.2, R7.1; no longer R10.2, R9.1
- net N$12: now also R3.1, R4.2; no longer R10.1, R11.2
- net N$13: now also R4.1, R5.2; no longer R11.1, R12.2
- net N$14: now also R5.1, R6.2; no longer R12.1, R13.2
- net N$2: now also D2.C, D3.A; no longer D1.A, D4.C
- net N$5: now also R10.1, R9.2; no longer R6.1, R7.2
- net N$7: now also D1.A, P1.3, R1.2; no longer D5.A, P2.3, R5.2
- net N$8: now also C4.P$2, D6.A, R1.1; no longer C2.P$2, D2.A, R5.1
- net N$9: now also R9.1; no longer R7.1
Routing:
- net +265V: track 85.7 -> 89.5 mm
- net GRID2: track 48.2 -> 44.6 mm
- net N$2: track 10.2 -> 8.89 mm
- net N$1: track 27.3 -> 26.2 mm

Commit message: added logo
Parts:
- added U$1, U$2: FIDUCIAL, adafruit:FIDUCIAL_1MM
Other:
- board text added: "board type 1705 / bias and focus"
