File: neck/mimic1705.brd (EAGLE design)
At the start: 165.1 x 114.3 mm, 28 parts, among them J1 JST-VH-5, J2 JST-VH-2, J3 JST-VH-3, J4 JST-VH-3, P1 1M, P2 44PINEDGE

Commit message: revised artwork
Parts:
- P2: value 44PINEDGE -> 44PINEDGE-M
- moved U$1 153.9 mm to (36.8, 108.0)
- moved U$2 153.9 mm to (152.4, 6.35)
Connections:
- net GND: now also P2.4
Routing:
- net GND: track 309.7 -> 323.3 mm, vias 0 -> 2
- net HEATER: track 66.6 -> 69.5 mm
- net N$11: track 8.39 -> 8.93 mm
