File: neck/mimic4688.brd (EAGLE design)
At the start: 165.1 x 114.3 mm, 54 parts, among them J1 JST-VH-3, P1 44PINEDGE, Q1 2N3906, Q10 2N3906, Q2 2N3906, Q3 2N3906, Q4 2N3904, Q5 2N3904, Q6 2N3904, Q7 2N3904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

Commit message: added logo
Parts:
- added U$1, U$2: FIDUCIAL, adafruit:FIDUCIAL_1MM
Routing:
- net N$8: track 25.4 -> 30.5 mm
Other:
- board text added: "board type 4688 / variable intensifier"
