File: neck/mimic4688.brd (EAGLE design)
At the start: 165.1 x 114.3 mm, 56 parts, among them J1 JST-VH-3, P1 44PINEDGE, Q1 2N3906, Q10 2N3906, Q2 2N3906, Q3 2N3906, Q4 2N3904, Q5 2N3904, Q6 2N3904, Q7 2N3904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

Commit message: revised artwork
Parts:
- P1: value 44PINEDGE -> 44PINEDGE-M
- moved U$1 153.9 mm to (36.8, 108.0)
- moved U$2 153.9 mm to (152.4, 6.35)
Connections:
- net GND: now also P1.4
Routing:
- net +10V: track 330.6 -> 320.6 mm
- net GND: track 181.0 -> 190.2 mm, vias 1 -> 3
- net -15V: track 233.0 -> 237.1 mm
- net CATHODE: track 197.0 -> 196.3 mm
