File: neck/mimic1705.sch (EAGLE design)
At the start: 26 parts, among them J1 JST-VH-2, J2 JST-VH-5, J3 JST-VH-3, J5 JST-VH-3, P2 1M, P20 44PINEDGE

Commit message: card layouts finished
Parts:
- removed P20: 44PINEDGE, keiths:44PINEDGE
- removed R11, R12, R13: 0.33, keiths:R-1/2WATT
- added P1: 1M, keiths:POT-3006P
- added R1: 18K, keiths:RES-V
- added R2: 220K, keiths:RES-V
- added R3: 0.33, keiths:R-1/2WATT
- C2: value 22 uF -> 0.01UF; device keiths:CAP100UF200V -> keiths:CAP_5MM; PN TVX2C220MCD -> (none)
- C4: value 0.01UF -> 22 uF; device keiths:CAP_5MM -> keiths:CAP100UF200V; PN (none) -> TVX2C220MCD
- D1, D4: value 1N4764 -> BZV85-C56,113; device keiths:1N4764A -> keiths:BZV85-C56,113
- D2, D3: value 1N4005 -> 1N4764; device keiths:1N400X -> keiths:1N4764A
- D5, D6: value BZV85-C56,113 -> 1N4005; device keiths:BZV85-C56,113 -> keiths:1N400X
- J1: value JST-VH-2 -> JST-VH-5; device keiths:JST-VH-2 -> keiths:JST-VH-5
- J2: value JST-VH-5 -> JST-VH-2; device keiths:JST-VH-5 -> keiths:JST-VH-2
- P2: value 1M -> 44PINEDGE; device keiths:POT-3006P -> keiths:44PINEDGE
- R4: value 220K -> 0.33; device keiths:RES-V -> keiths:R-1/2WATT
- R5: value 18K -> 0.33; device keiths:RES-V -> keiths:R-1/2WATT
- renumbered J5 to J4
Connections:
- net +265V: now also R2.P$2; no longer R4.P$1
- net -150V: now also D6.C; no longer D2.C
- net 6.3_VAC_1: now also J2.1, R10.P$2; no longer J1.1, R6.P$2
- net 6.3_VAC_2: now also J1.5, J2.2; no longer J1.2, J2.5
- net CATHODE: now also D5.C, J1.2; no longer D3.C, J2.2
- net GND: now also C2.2, C4.1, D2.A, D4.C, P1.1, P2.D; no longer C2.1, C4.2, D4.A, D6.C, P2.1, P20.D
- net GRID1: now also C1.1, D5.A, J1.3, P1.2; no longer C4.1, D3.A, J2.3, P2.2
- net GRID2: now also C2.1, D3.C, J1.1, R2.P$1; no longer C1.1, D1.C, J2.1, R4.P$2
- net HEATER: now also J1.4, R6.P$1; no longer J2.4, R13.P$1
- net N$1: now also D1.C, D4.A; no longer D5.C, D6.A
- net N$10: now also R7.P$2; no longer R9.P$2
- net N$11: now also R3.P$2, R7.P$1; no longer R10.P$2, R9.P$1
- net N$12: now also R3.P$1, R4.P$2; no longer R10.P$1, R11.P$2
- net N$13: now also R4.P$1, R5.P$2; no longer R11.P$1, R12.P$2
- net N$14: now also R5.P$1, R6.P$2; no longer R12.P$1, R13.P$2
- net N$2: now also D2.C, D3.A; no longer D1.A, D4.C
- net N$5: now also R10.P$1, R9.P$2; no longer R6.P$1, R7.P$2
- net N$7: now also D1.A, P1.3, R1.P$2; no longer D5.A, P2.3, R5.P$2
- net N$8: now also C4.2, D6.A, R1.P$1; no longer C2.2, D2.A, R5.P$1
- net N$9: now also R9.P$1; no longer R7.P$1
Other:
- moved on the sheet: C1, D1, D4, R10, R6, R7, R9

Commit message: added logo
Parts:
- added U$1, U$2: FIDUCIAL, adafruit:FIDUCIAL
Changed lines of the file:
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@@
 <part name="D1" library="keiths" deviceset="BZV85-C56,113" device="" value="BZV85-C56,113"/>
 <part name="D4" library="keiths" deviceset="BZV85-C56,113" device="" value="BZV85-C56,113"/>
+<part name="U$1" library="adafruit" deviceset="FIDUCIAL" device=""/>
+<part name="U$2" library="adafruit" deviceset="FIDUCIAL" device=""/>
 </parts>
 <sheets>
@@
 <attribute name="VALUE" x="322.58" y="226.06" size="1.9304" layer="96" font="vector" ratio="10"/>
 </instance>
+<instance part="U$1" gate="G$1" x="477.52" y="398.78"/>
+<instance part="U$2" gate="G$1" x="497.84" y="398.78"/>
 </instances>
 <busses>

Commit message: revised artwork
Parts:
- P2: value 44PINEDGE -> 44PINEDGE-M; device keiths:44PINEDGE -> keiths:44PINEDGE-M
Connections:
- net GND: now also P2.4
Other:
- note added: "Bias and Focus"
- moved on the sheet: P2
Changed lines of the file:
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@@
 <part name="FRAME1" library="frames" deviceset="FRAME_C_L" device=""/>
 <part name="FRAME2" library="frames" deviceset="FRAME_C_L" device=""/>
-<part name="P2" library="keiths" deviceset="44PINEDGE" device=""/>
 <part name="R2" library="keiths" deviceset="RES-V" device="" value="220K"/>
 <part name="SUPPLY1" library="keiths" deviceset="GND" device=""/>
@@
 <part name="D1" library="keiths" deviceset="BZV85-C56,113" device="" value="BZV85-C56,113"/>
 <part name="D4" library="keiths" deviceset="BZV85-C56,113" device="" value="BZV85-C56,113"/>
+<part name="U$2" library="adafruit" deviceset="FIDUCIAL" device=""/>
 <part name="U$1" library="adafruit" deviceset="FIDUCIAL" device=""/>
-<part name="U$2" library="adafruit" deviceset="FIDUCIAL" device=""/>
+<part name="P2" library="keiths" deviceset="44PINEDGE-M" device=""/>
+<part name="SUPPLY40" library="keiths" deviceset="GND" device=""/>
+<part name="SUPPLY45" library="keiths" deviceset="GND" device=""/>
 </parts>
 <sheets>
@@
 <text x="292.1" y="233.68" size="3.81" layer="91" font="vector" ratio="10">60 Volt
 Zeners</text>
+<text x="271.78" y="307.34" size="2.1844" layer="91" font="vector" ratio="10">Bias and Focus</text>
 </plain>
 <instances>
 <instance part="FRAME1" gate="G$1" x="0" y="0"/>
 <instance part="FRAME2" gate="G$2" x="452.12" y="0"/>
-<instance part="P2" gate="G$1" x="271.78" y="345.44"/>
 <instance part="R2" gate="G$1" x="299.72" y="106.68" smashed="yes" rot="R180">
 <attribute name="NAME" x="301.752" y="107.95" size="1.9304" layer="95" font="vector" ratio="10"/>
@@
 <attribute name="VALUE" x="322.58" y="226.06" size="1.9304" layer="96" font="vector" ratio="10"/>
 </instance>
-<instance part="U$1" gate="G$1" x="477.52" y="398.78"/>
-<instance part="U$2" gate="G$1" x="497.84" y="398.78"/>
+<instance part="U$2" gate="G$1" x="510.54" y="53.34"/>
+<instance part="U$1" gate="G$1" x="530.86" y="53.34"/>
+<instance part="P2" gate="G$1" x="284.48" y="345.44"/>
+<instance part="SUPPLY40" gate="GND" x="248.92" y="363.22" smashed="yes" rot="MR90">
+<attribute name="VALUE" x="245.491" y="362.585" size="1.9304" layer="96" font="vector" ratio="10" rot="MR0"/>
+</instance>
+<instance part="SUPPLY45" gate="GND" x="320.04" y="363.22" smashed="yes" rot="R90">
+<attribute name="VALUE" x="323.469" y="362.585" size="1.9304" layer="96" font="vector" ratio="10"/>
+</instance>
 </instances>
 <busses>
@@
 </segment>
 <segment>
-<wire x1="281.94" y1="363.22" x2="289.56" y2="363.22" width="0.1524" layer="91"/>
-<label x="289.56" y="363.22" size="1.9304" layer="95" font="vector" ratio="10" xref="yes"/>
-<pinref part="P2" gate="G$1" pin="D"/>
-</segment>
-<segment>
 <pinref part="SUPPLY2" gate="GND" pin="GND"/>
 <wire x1="137.16" y1="177.8" x2="157.48" y2="177.8" width="0.1524" layer="91"/>
@@
 <pinref part="J3" gate="G$1" pin="2"/>
 </segment>
+<segment>
+<wire x1="294.64" y1="363.22" x2="317.5" y2="363.22" width="0.1524" layer="91"/>
+<pinref part="SUPPLY45" gate="GND" pin="GND"/>
+<pinref part="P2" gate="G$1" pin="D"/>
+</segment>
+<segment>
+<pinref part="SUPPLY40" gate="GND" pin="GND"/>
+<wire x1="251.46" y1="363.22" x2="274.32" y2="363.22" width="0.1524" layer="91"/>
+<pinref part="P2" gate="G$1" pin="4"/>
+</segment>
 </net>
