File: neck/mimic4688.sch (EAGLE design)
At the start: 54 parts, among them J1 JST-VH-3, P1 44PINEDGE, Q1 2N3906, Q10 2N3906, Q11 2N3906, Q2 2N3904, Q3 2N3906, Q4 2N3904, Q5 2N3904, Q6 2N3906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

Commit message: card layouts finished
Parts:
- removed D13: 1N4148, keiths:1N4148
- removed Q11: 2N3906, keiths:2N3906
- added D4: 1N4148, keiths:1N4148
- added Q8: 2N3906, keiths:2N3906
- Q2: value 2N3904 -> 2N3906; device keiths:2N3904 -> keiths:2N3906
- Q6: value 2N3906 -> 2N3904; device keiths:2N3906 -> keiths:2N3904
- R1: value 11.3K -> 33K; device keiths:R-1/4WATT -> keiths:RES33K2W
- R10: value 1.5K -> 2.2K
- R11: value 470 -> 5.1K
- R12: value 470 -> 22K
- R13: value 100K -> 3.3K
- R14: value 22K -> 20K
- R15: value 100K -> 12.7K
- R16: value 20K -> 23.7K
- R17: value 11.3K -> 10K
- R18, R19: value 5.1K -> 20K
- R2: value 10K -> 470
- R20, R21: value 33K -> 10K; device keiths:RES33K2W -> keiths:R-1/4WATT
- R22: value 10K -> 11.3K
- R25: value 10.7K -> 11.3K
- R26: value 12.1K -> 60.4K
- R27: value 20K -> 18.7K
- R28: value 100K -> 11.3K
- R29: value 12.7K -> 12.1K
- R3: value 18.7K -> 470
- R30: value 23.7K -> 10.7K
- R4: value 60.4K -> 33K; device keiths:R-1/4WATT -> keiths:RES33K2W
- R5: value 20K -> 100K
- R6: value 11.3K -> 5.1K
- R7: value 10K -> 3K
- R8: value 2.2K -> 100K
- R9: value 3.3K -> 100K
- renumbered D11 to D5
Connections:
- removed net N$22: Q7.E, R27.P$1
- new net N$4: Q7.E, R18.P$2
- net +10V: now also Q5.C, Q6.C, R15.P$1, R16.P$1, R22.P$1, R27.P$1, R28.P$1; no longer Q2.C, Q4.C, R1.P$1, R17.P$1, R3.P$1, R4.P$1, R6.P$1
- net -150V: now also R1.P$2, R4.P$2; no longer R20.P$2, R21.P$2
- net -15V: now also Q10.C, Q8.C, R12.P$2, R13.P$2, R17.P$2, R20.P$2, R21.P$2, R7.P$1; no longer Q3.C, Q6.C, R10.P$2, R14.P$2, R2.P$2, R22.P$2, R7.P$2, R9.P$2
- net CATHODE: now also D6.A, R9.P$1; no longer D13.A, R28.P$2
- net GND: now also D6.C, Q1.E, Q2.E, R5.P$1, R8.P$2, R9.P$2; no longer D13.C, Q10.E, Q11.E, R13.P$1, R15.P$1, R28.P$1
- net J_IN: now also Q5.B; no longer Q7.B
- net N$1: now also Q1.B, R2.P$1; no longer Q10.B, R11.P$1
- net N$10: now also Q5.E, R19.P$2; no longer Q4.E, R16.P$1
- net N$11: now also Q4.E, R13.P$1; no longer Q5.E, R9.P$1
- net N$12: now also Q4.B, R12.P$1, R8.P$1; no longer Q5.B, R13.P$2, R14.P$1
- net N$13: now also Q8.B, R17.P$1, R19.P$1, R22.P$2; no longer Q6.B, R17.P$2, R22.P$1, R27.P$2
- net N$14: now also D2.C, D3.A; no longer D8.C, D9.A
- net N$15: now also Q2.C, Q3.E; no longer Q1.E, Q11.C
- net N$16: now also D9.A, Q8.E; no longer D3.A, Q6.E
- net N$17: now also D7.A, Q10.E, R29.P$2, R30.P$2; no longer D1.A, Q9.E, R25.P$2, R26.P$2
- net N$18: now also Q3.B, R11.P$2, R6.P$1; no longer Q1.B, R18.P$1, R19.P$2
- net N$2: now also Q9.B, R14.P$1, R20.P$1, R25.P$2; no longer Q3.B, R1.P$2, R16.P$2, R2.P$1
- net N$20: now also D2.A, Q2.B, R5.P$2; no longer D8.A, Q11.B, R15.P$2
- net N$21: now also D4.A, D7.C, D8.C, R11.P$1, R15.P$2, R16.P$2; no longer D1.C, D2.C, D7.A, R19.P$1, R29.P$2, R30.P$2
- net N$3: now also D8.A, Q9.E, R26.P$2, R27.P$2; no longer D2.A, Q3.E, R3.P$2, R4.P$2
- net N$5: now also Q10.B, R18.P$1, R21.P$1, R28.P$2; no longer Q9.B, R5.P$2, R6.P$2, R7.P$1
- net N$6: now also Q6.E, R14.P$2; no longer Q2.E, R5.P$1
- net N$7: now also D1.A, D4.C, Q1.C, R7.P$2; no longer D6.A, D7.C, Q10.C, R10.P$1
- net N$8: now also D1.C, R2.P$2, R3.P$2; no longer D6.C, R11.P$2, R12.P$1
- net N$9: now also Q4.C, R10.P$1, R3.P$1; no longer Q5.C, R12.P$2, R8.P$2
- net P_IN: now also R10.P$2; no longer R8.P$1
- net U_IN: now also Q6.B; no longer Q4.B
- net X_IN: now also Q7.B; no longer Q2.B
- net Y_OUT: now also Q3.C, R1.P$1, R4.P$1, R6.P$2; no longer Q1.C, R18.P$2, R20.P$1, R21.P$1
Other:
- moved on the sheet: D1, D2, D3, D6, D7, D8, D9, Q1, Q10, Q3, Q4, Q5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

Commit message: added logo
Parts:
- added U$1, U$2: FIDUCIAL, adafruit:FIDUCIAL
Changed lines of the file:
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@@
 <grid distance="0.1" unitdist="inch" unit="inch" style="lines" multiple="1" display="no" altdistance="0.01" altunitdist="inch" altunit="inch"/>
 <layers>
-<layer number="1" name="Top" color="4" fill="1" visible="yes" active="no"/>
-<layer number="2" name="Route2" color="1" fill="3" visible="yes" active="no"/>
-<layer number="3" name="Route3" color="4" fill="3" visible="yes" active="no"/>
-<layer number="4" name="Route4" color="1" fill="4" visible="yes" active="no"/>
-<layer number="5" name="Route5" color="4" fill="4" visible="yes" active="no"/>
-<layer number="6" name="Route6" color="1" fill="8" visible="yes" active="no"/>
-<layer number="7" name="Route7" color="4" fill="8" visible="yes" active="no"/>
-<layer number="8" name="Route8" color="1" fill="2" visible="yes" active="no"/>
-<layer number="9" name="Route9" color="4" fill="2" visible="yes" active="no"/>
-<layer number="10" name="Route10" color="1" fill="7" visible="yes" active="no"/>
-<layer number="11" name="Route11" color="4" fill="7" visible="yes" active="no"/>
-<layer number="12" name="Route12" color="1" fill="5" visible="yes" active="no"/>
-<layer number="13" name="Route13" color="4" fill="5" visible="yes" active="no"/>
-<layer number="14" name="Route14" color="1" fill="6" visible="yes" active="no"/>
-<layer number="15" name="Route15" color="4" fill="6" visible="yes" active="no"/>
-<layer number="16" name="Bottom" color="1" fill="1" visible="yes" active="no"/>
-<layer number="17" name="Pads" color="2" fill="1" visible="yes" active="no"/>
-<layer number="18" name="Vias" color="2" fill="1" visible="yes" active="no"/>
-<layer number="19" name="Unrouted" color="6" fill="1" visible="yes" active="no"/>
-<layer number="20" name="Dimension" color="15" fill="1" visible="yes" active="no"/>
-<layer number="21" name="tPlace" color="7" fill="1" visible="yes" active="no"/>
-<layer number="22" name="bPlace" color="7" fill="1" visible="yes" active="no"/>
-<layer number="23" name="tOrigins" color="15" fill="1" visible="yes" active="no"/>
-<layer number="24" name="bOrigins" color="15" fill="1" visible="yes" active="no"/>
-<layer number="25" name="tNames" color="7" fill="1" visible="yes" active="no"/>
-<layer number="26" name="bNames" color="7" fill="1" visible="yes" active="no"/>
-<layer number="27" name="tValues" color="7" fill="1" visible="yes" active="no"/>
-<layer number="28" name="bValues" color="7" fill="1" visible="yes" active="no"/>
+<layer number="1" name="Top" color="4" fill="1" visible="no" active="no"/>
+<layer number="2" name="Route2" color="1" fill="3" visible="no" active="no"/>
+<layer number="3" name="Route3" color="4" fill="3" visible="no" active="no"/>
+<layer number="4" name="Route4" color="1" fill="4" visible="no" active="no"/>
+<layer number="5" name="Route5" color="4" fill="4" visible="no" active="no"/>
+<layer number="6" name="Route6" color="1" fill="8" visible="no" active="no"/>
+<layer number="7" name="Route7" color="4" fill="8" visible="no" active="no"/>
+<layer number="8" name="Route8" color="1" fill="2" visible="no" active="no"/>
+<layer number="9" name="Route9" color="4" fill="2" visible="no" active="no"/>
+<layer number="10" name="Route10" color="1" fill="7" visible="no" active="no"/>
+<layer number="11" name="Route11" color="4" fill="7" visible="no" active="no"/>
+<layer number="12" name="Route12" color="1" fill="5" visible="no" active="no"/>
+<layer number="13" name="Route13" color="4" fill="5" visible="no" active="no"/>
+<layer number="14" name="Route14" color="1" fill="6" visible="no" active="no"/>
+<layer number="15" name="Route15" color="4" fill="6" visible="no" active="no"/>
+<layer number="16" name="Bottom" color="1" fill="1" visible="no" active="no"/>
+<layer number="17" name="Pads" color="2" fill="1" visible="no" active="no"/>
+<layer number="18" name="Vias" color="2" fill="1" visible="no" active="no"/>
+<layer number="19" name="Unrouted" color="6" fill="1" visible="no" active="no"/>
+<layer number="20" name="Dimension" color="15" fill="1" visible="no" active="no"/>
+<layer number="21" name="tPlace" color="7" fill="1" visible="no" active="no"/>
+<layer number="22" name="bPlace" color="7" fill="1" visible="no" active="no"/>
+<layer number="23" name="tOrigins" color="15" fill="1" visible="no" active="no"/>
+<layer number="24" name="bOrigins" color="15" fill="1" visible="no" active="no"/>
+<layer number="25" name="tNames" color="7" fill="1" visible="no" active="no"/>
+<layer number="26" name="bNames" color="7" fill="1" visible="no" active="no"/>
+<layer number="27" name="tValues" color="7" fill="1" visible="no" active="no"/>
+<layer number="28" name="bValues" color="7" fill="1" visible="no" active="no"/>
 <layer number="29" name="tStop" color="7" fill="3" visible="no" active="no"/>
 <layer number="30" name="bStop" color="7" fill="6" visible="no" active="no"/>
@@
 <layer number="35" name="tGlue" color="7" fill="4" visible="no" active="no"/>
 <layer number="36" name="bGlue" color="7" fill="5" visible="no" active="no"/>
-<layer number="37" name="tTest" color="7" fill="1" visible="yes" active="no"/>
-<layer number="38" name="bTest" color="7" fill="1" visible="yes" active="no"/>
+<layer number="37" name="tTest" color="7" fill="1" visible="no" active="no"/>
+<layer number="38" name="bTest" color="7" fill="1" visible="no" active="no"/>
 <layer number="39" name="tKeepout" color="4" fill="11" visible="no" active="no"/>
 <layer number="40" name="bKeepout" color="1" fill="11" visible="no" active="no"/>
@@
 <layer number="44" name="Drills" color="7" fill="1" visible="no" active="no"/>
 <layer number="45" name="Holes" color="7" fill="1" visible="no" active="no"/>
-<layer number="46" name="Milling" color="3" fill="1" visible="yes" active="no"/>
-<layer number="47" name="Measures" color="7" fill="1" visible="yes" active="no"/>
-<layer number="48" name="Document" color="7" fill="1" visible="yes" active="no"/>
-<layer number="49" name="Reference" color="7" fill="1" visible="yes" active="no"/>
-<layer number="50" name="dxf" color="7" fill="1" visible="yes" active="no"/>
-<layer number="51" name="tDocu" color="7" fill="1" visible="yes" active="no"/>
-<layer number="52" name="bDocu" color="7" fill="1" visible="yes" active="no"/>
-<layer number="53" name="tGND_GNDA" color="7" fill="1" visible="yes" active="no"/>
-<layer number="54" name="bGND_GNDA" color="7" fill="1" visible="yes" active="no"/>
-<layer number="56" name="wert" color="7" fill="1" visible="yes" active="no"/>
-<layer number="57" name="tCAD" color="7" fill="1" visible="yes" active="no"/>
-<layer number="59" name="tCarbon" color="7" fill="1" visible="yes" active="no"/>
-<layer number="60" name="bCarbon" color="7" fill="1" visible="yes" active="no"/>
+<layer number="46" name="Milling" color="3" fill="1" visible="no" active="no"/>
+<layer number="47" name="Measures" color="7" fill="1" visible="no" active="no"/>
+<layer number="48" name="Document" color="7" fill="1" visible="no" active="no"/>
+<layer number="49" name="Reference" color="7" fill="1" visible="no" active="no"/>
+<layer number="50" name="dxf" color="7" fill="1" visible="no" active="no"/>
+<layer number="51" name="tDocu" color="7" fill="1" visible="no" active="no"/>
+<layer number="52" name="bDocu" color="7" fill="1" visible="no" active="no"/>
+<layer number="53" name="tGND_GNDA" color="7" fill="1" visible="no" active="no"/>
+<layer number="54" name="bGND_GNDA" color="7" fill="1" visible="no" active="no"/>
+<layer number="56" name="wert" color="7" fill="1" visible="no" active="no"/>
+<layer number="57" name="tCAD" color="7" fill="1" visible="no" active="no"/>
+<layer number="59" name="tCarbon" color="7" fill="1" visible="no" active="no"/>
+<layer number="60" name="bCarbon" color="7" fill="1" visible="no" active="no"/>
 <layer number="90" name="Modules" color="5" fill="1" visible="yes" active="yes"/>
 <layer number="91" name="Nets" color="2" fill="1" visible="yes" active="yes"/>
@@
 <part name="R16" library="keiths" deviceset="R-1/4WATT" device="" value="23.7K"/>
 <part name="D5" library="keiths" deviceset="1N4148" device="" value="1N4148"/>
+<part name="U$1" library="adafruit" deviceset="FIDUCIAL" device=""/>
+<part name="U$2" library="adafruit" deviceset="FIDUCIAL" device=""/>
 </parts>
 <sheets>
@@
 <attribute name="VALUE" x="320.04" y="226.06" size="1.9304" layer="96" font="vector" ratio="10"/>
 </instance>
+<instance part="U$1" gate="G$1" x="485.14" y="398.78"/>
+<instance part="U$2" gate="G$1" x="500.38" y="398.78"/>
 </instances>
 <busses>

Commit message: revised artwork
Parts:
- P1: value 44PINEDGE -> 44PINEDGE-M; device keiths:44PINEDGE -> keiths:44PINEDGE-M
Connections:
- net GND: now also P1.4
Other:
- note added: "Variable Intensifier"
- moved on the sheet: P1
Changed lines of the file:
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@@
 <part name="FRAME1" library="frames" deviceset="FRAME_C_L" device=""/>
 <part name="FRAME2" library="frames" deviceset="FRAME_C_L" device=""/>
-<part name="P1" library="keiths" deviceset="44PINEDGE" device=""/>
 <part name="SUPPLY1" library="keiths" deviceset="GND" device=""/>
 <part name="R28" library="keiths" deviceset="R-1/4WATT" device="" value="11.3K"/>
@@
 <part name="R16" library="keiths" deviceset="R-1/4WATT" device="" value="23.7K"/>
 <part name="D5" library="keiths" deviceset="1N4148" device="" value="1N4148"/>
+<part name="U$2" library="adafruit" deviceset="FIDUCIAL" device=""/>
 <part name="U$1" library="adafruit" deviceset="FIDUCIAL" device=""/>
-<part name="U$2" library="adafruit" deviceset="FIDUCIAL" device=""/>
+<part name="P1" library="keiths" deviceset="44PINEDGE-M" device=""/>
+<part name="SUPPLY40" library="keiths" deviceset="GND" device=""/>
+<part name="SUPPLY45" library="keiths" deviceset="GND" device=""/>
+<part name="SUPPLY46" library="keiths" deviceset="-15V" device=""/>
+<part name="SUPPLY47" library="supply2" deviceset="+10V" device=""/>
 </parts>
 <sheets>
@@
 <text x="459.74" y="195.58" size="3.81" layer="91" font="vector" ratio="10">Connector to
 mimic1705 bias.</text>
+<text x="73.66" y="180.34" size="2.1844" layer="91" font="vector" ratio="10">Variable Intensifier</text>
 </plain>
 <instances>
 <instance part="FRAME1" gate="G$1" x="0" y="0"/>
 <instance part="FRAME2" gate="G$2" x="452.12" y="0"/>
-<instance part="P1" gate="G$1" x="66.04" y="215.9"/>
 <instance part="SUPPLY1" gate="GND" x="368.3" y="358.14" rot="MR180"/>
 <instance part="R28" gate="&gt;NAME" x="226.06" y="96.52" smashed="yes" rot="MR90">
@@
 <attribute name="VALUE" x="320.04" y="226.06" size="1.9304" layer="96" font="vector" ratio="10"/>
 </instance>
-<instance part="U$1" gate="G$1" x="485.14" y="398.78"/>
-<instance part="U$2" gate="G$1" x="500.38" y="398.78"/>
+<instance part="U$2" gate="G$1" x="485.14" y="398.78"/>
+<instance part="U$1" gate="G$1" x="500.38" y="398.78"/>
+<instance part="P1" gate="G$1" x="88.9" y="218.44"/>
+<instance part="SUPPLY40" gate="GND" x="55.88" y="236.22" smashed="yes" rot="MR90">
+<attribute name="VALUE" x="52.451" y="235.585" size="1.9304" layer="96" font="vector" ratio="10" rot="MR0"/>
+</instance>
+<instance part="SUPPLY45" gate="GND" x="127" y="236.22" smashed="yes" rot="R90">
+<attribute name="VALUE" x="130.429" y="235.585" size="1.9304" layer="96" font="vector" ratio="10"/>
+</instance>
+<instance part="SUPPLY46" gate="G$1" x="111.76" y="238.76" smashed="yes" rot="R90">
+<attribute name="VALUE" x="115.697" y="237.871" size="1.9304" layer="96" font="vector" ratio="10"/>
+</instance>
+<instance part="SUPPLY47" gate="G$1" x="111.76" y="243.84" smashed="yes" rot="MR90">
+<attribute name="VALUE" x="115.824" y="244.729" size="1.9304" layer="96" font="vector" ratio="10" rot="MR180"/>
+</instance>
 </instances>
 <busses>
@@
 </segment>
 <segment>
-<pinref part="P1" gate="G$1" pin="D"/>
-<wire x1="76.2" y1="233.68" x2="83.82" y2="233.68" width="0.1524" layer="91"/>
-<label x="83.82" y="233.68" size="1.9304" layer="95" font="vector" ratio="10" xref="yes"/>
-</segment>
-<segment>
 <wire x1="436.88" y1="200.66" x2="429.26" y2="200.66" width="0.1524" layer="91"/>
 <wire x1="429.26" y1="200.66" x2="429.26" y2="190.5" width="0.1524" layer="91"/>
@@
 <wire x1="210.82" y1="274.32" x2="210.82" y2="281.94" width="0.1524" layer="91"/>
 </segment>
+<segment>
+<wire x1="99.06" y1="236.22" x2="124.46" y2="236.22" width="0.1524" layer="91"/>
+<pinref part="SUPPLY45" gate="GND" pin="GND"/>
+<pinref part="P1" gate="G$1" pin="D"/>
+</segment>
+<segment>
+<pinref part="SUPPLY40" gate="GND" pin="GND"/>
+<wire x1="58.42" y1="236.22" x2="78.74" y2="236.22" width="0.1524" layer="91"/>
+<pinref part="P1" gate="G$1" pin="4"/>
+</segment>
 </net>
 <net name="J_IN" class="0">
@@
 </segment>
 <segment>
+<label x="109.22" y="226.06" size="1.9304" layer="95" font="vector" ratio="10" xref="yes"/>
 <pinref part="P1" gate="G$1" pin="J"/>
-<wire x1="76.2" y1="223.52" x2="83.82" y2="223.52" width="0.1524" layer="91"/>
-<label x="83.82" y="223.52" size="1.9304" layer="95" font="vector" ratio="10" xref="yes"/>
+<wire x1="99.06" y1="226.06" x2="109.22" y2="226.06" width="0.1524" layer="91"/>
 </segment>
 </net>
@@
 </segment>
 <segment>
-<pinref part="P1" gate="G$1" pin="C"/>
-<wire x1="76.2" y1="236.22" x2="111.76" y2="236.22" width="0.1524" layer="91"/>
-<label x="111.76" y="236.22" size="1.9304" layer="95" font="vector" ratio="10" xref="yes"/>
-</segment>
-<segment>
 <label x="185.42" y="114.3" size="1.9304" layer="95" font="vector" ratio="10" rot="MR0" xref="yes"/>
 <pinref part="Q9" gate="G$1" pin="C"/>
@@
 <wire x1="226.06" y1="162.56" x2="226.06" y2="160.02" width="0.1524" layer="91"/>
 <junction x="226.06" y="160.02"/>
+</segment>
+<segment>
+<pinref part="SUPPLY46" gate="G$1" pin="-15V"/>
+<pinref part="P1" gate="G$1" pin="C"/>
+<wire x1="99.06" y1="238.76" x2="109.22" y2="238.76" width="0.1524" layer="91"/>
 </segment>
 </net>
@@
 </segment>
 <segment>
+<label x="124.46" y="203.2" size="1.9304" layer="95" font="vector" ratio="10" xref="yes"/>
 <pinref part="P1" gate="G$1" pin="U"/>
-<wire x1="76.2" y1="200.66" x2="111.76" y2="200.66" width="0.1524" layer="91"/>
-<label x="111.76" y="200.66" size="1.9304" layer="95" font="vector" ratio="10" xref="yes"/>
+<wire x1="99.06" y1="203.2" x2="124.46" y2="203.2" width="0.1524" layer="91"/>
 </segment>
 </net>
@@
 </segment>
 <segment>
+<label x="109.22" y="195.58" size="1.9304" layer="95" font="vector" ratio="10" xref="yes"/>
 <pinref part="P1" gate="G$1" pin="X"/>
-<wire x1="76.2" y1="193.04" x2="83.82" y2="193.04" width="0.1524" layer="91"/>
-<label x="83.82" y="193.04" size="1.9304" layer="95" font="vector" ratio="10" xref="yes"/>
+<wire x1="99.06" y1="195.58" x2="109.22" y2="195.58" width="0.1524" layer="91"/>
 </segment>
 </net>
@@
 </segment>
 <segment>
+<label x="124.46" y="213.36" size="1.9304" layer="95" font="vector" ratio="10" xref="yes"/>
 <pinref part="P1" gate="G$1" pin="P"/>
-<wire x1="76.2" y1="210.82" x2="111.76" y2="210.82" width="0.1524" layer="91"/>
-<label x="111.76" y="210.82" size="1.9304" layer="95" font="vector" ratio="10" xref="yes"/>
+<wire x1="99.06" y1="213.36" x2="124.46" y2="213.36" width="0.1524" layer="91"/>
 </segment>
 </net>
@@
 <net name="+10V" class="0">
 <segment>
-<pinref part="P1" gate="G$1" pin="A"/>
-<wire x1="76.2" y1="241.3" x2="111.76" y2="241.3" width="0.1524" layer="91"/>
-<label x="111.76" y="241.3" size="1.9304" layer="95" font="vector" ratio="10" xref="yes"/>
-</segment>
-<segment>
 <pinref part="R28" gate="&gt;NAME" pin="P$1"/>
 <wire x1="226.06" y1="106.68" x2="226.06" y2="101.6" width="0.1524" layer="91"/>
@@
 <pinref part="R16" gate="&gt;NAME" pin="P$1"/>
 <wire x1="264.16" y1="205.74" x2="241.3" y2="205.74" width="0.1524" layer="91"/>
+</segment>
+<segment>
+<pinref part="SUPPLY47" gate="G$1" pin="+10V"/>
+<pinref part="P1" gate="G$1" pin="A"/>
+<wire x1="99.06" y1="243.84" x2="109.22" y2="243.84" width="0.1524" layer="91"/>
 </segment>
 </net>
@@
 </segment>
 <segment>
-<wire x1="76.2" y1="187.96" x2="111.76" y2="187.96" width="0.1524" layer="91"/>
-<label x="111.76" y="187.96" size="1.9304" layer="95" font="vector" ratio="10" xref="yes"/>
+<wire x1="99.06" y1="190.5" x2="124.46" y2="190.5" width="0.1524" layer="91"/>
+<label x="124.46" y="190.5" size="1.9304" layer="95" font="vector" ratio="10" xref="yes"/>
 <pinref part="P1" gate="G$1" pin="Z"/>
 </segment>
