File: processor.sch (EAGLE design)
At the start: 1 part, among them P5 44PINEDGE

Commit message: revised artwork
Parts:
- removed P5: 44PINEDGE, keiths:44PINEDGE
- added P1: 44PINEDGE-M, keiths:44PINEDGE-M
Connections:
- new net LE3: P1.18
- net +5V: now also P1.B; no longer P5.B
- net D0: now also P1.7; no longer P5.1
- net D1: now also P1.8; no longer P5.2
- net D2: now also P1.9; no longer P5.3
- net D3: now also P1.10; no longer P5.4
- net D4: now also P1.11; no longer P5.5
- net D5: now also P1.12; no longer P5.6
- net D6: now also P1.13; no longer P5.7
- net D7: now also P1.14; no longer P5.8
- net GND: now also P1.4, P1.D; no longer P5.D
- net LE1: now also P1.16; no longer P5.9
- net LE2: now also P1.17; no longer P5.10
- net X_LSB: now also P1.20; no longer P5.12
- net X_MSB: now also P1.19; no longer P5.11
- net Y_LSB: now also P1.22; no longer P5.14
- net Y_MSB: now also P1.21; no longer P5.13
Other:
- note added: "Brain Bus"
Changed lines of the file:
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@@
 <parts>
 <part name="FRAME1" library="frames" deviceset="FRAME_C_L" device=""/>
-<part name="P5" library="keiths" deviceset="44PINEDGE" device=""/>
+<part name="SUPPLY19" library="keiths" deviceset="+5V" device=""/>
+<part name="SUPPLY20" library="keiths" deviceset="GND" device=""/>
+<part name="SUPPLY24" library="keiths" deviceset="GND" device=""/>
+<part name="P1" library="keiths" deviceset="44PINEDGE-M" device=""/>
 </parts>
 <sheets>
 <sheet>
 <plain>
+<text x="274.32" y="187.96" size="2.1844" layer="91" font="vector" ratio="10">Brain Bus</text>
 </plain>
 <instances>
 <instance part="FRAME1" gate="G$1" x="0" y="0"/>
 <instance part="FRAME1" gate="G$2" x="452.12" y="0"/>
-<instance part="P5" gate="G$1" x="281.94" y="226.06"/>
+<instance part="SUPPLY19" gate="+5V" x="317.5" y="248.92" smashed="yes" rot="R270">
+<attribute name="VALUE" x="320.929" y="247.777" size="1.9304" layer="96" font="vector" ratio="10"/>
+</instance>
+<instance part="SUPPLY20" gate="GND" x="317.5" y="243.84" smashed="yes" rot="R90">
+<attribute name="VALUE" x="320.929" y="243.205" size="1.9304" layer="96" font="vector" ratio="10"/>
+</instance>
+<instance part="SUPPLY24" gate="GND" x="246.38" y="243.84" smashed="yes" rot="MR90">
+<attribute name="VALUE" x="242.951" y="243.205" size="1.9304" layer="96" font="vector" ratio="10" rot="MR0"/>
+</instance>
+<instance part="P1" gate="G$1" x="281.94" y="226.06"/>
 </instances>
 <busses>
@@
 <net name="LE1" class="0">
 <segment>
-<wire x1="264.16" y1="231.14" x2="271.78" y2="231.14" width="0.1524" layer="91"/>
-<label x="264.16" y="231.14" size="1.9304" layer="95" font="vector" ratio="10" rot="MR0" xref="yes"/>
-<pinref part="P5" gate="G$1" pin="9"/>
+<wire x1="264.16" y1="213.36" x2="271.78" y2="213.36" width="0.1524" layer="91"/>
+<label x="264.16" y="213.36" size="1.9304" layer="95" font="vector" ratio="10" rot="MR0" xref="yes"/>
+<pinref part="P1" gate="G$1" pin="16"/>
 </segment>
 </net>
 <net name="D0" class="0">
 <segment>
-<label x="264.16" y="251.46" size="1.9304" layer="95" font="vector" ratio="10" rot="MR0" xref="yes"/>
-<wire x1="264.16" y1="251.46" x2="271.78" y2="251.46" width="0.1524" layer="91"/>
-<pinref part="P5" gate="G$1" pin="1"/>
+<label x="248.92" y="236.22" size="1.9304" layer="95" font="vector" ratio="10" rot="MR0" xref="yes"/>
+<wire x1="248.92" y1="236.22" x2="271.78" y2="236.22" width="0.1524" layer="91"/>
+<pinref part="P1" gate="G$1" pin="7"/>
 </segment>
 </net>
 <net name="D1" class="0">
 <segment>
-<label x="251.46" y="248.92" size="1.9304" layer="95" font="vector" ratio="10" rot="MR0" xref="yes"/>
-<wire x1="251.46" y1="248.92" x2="271.78" y2="248.92" width="0.1524" layer="91"/>
-<pinref part="P5" gate="G$1" pin="2"/>
+<label x="264.16" y="233.68" size="1.9304" layer="95" font="vector" ratio="10" rot="MR0" xref="yes"/>
+<wire x1="264.16" y1="233.68" x2="271.78" y2="233.68" width="0.1524" layer="91"/>
+<pinref part="P1" gate="G$1" pin="8"/>
 </segment>
 </net>
 <net name="D2" class="0">
 <segment>
-<label x="264.16" y="246.38" size="1.9304" layer="95" font="vector" ratio="10" rot="MR0" xref="yes"/>
-<wire x1="264.16" y1="246.38" x2="271.78" y2="246.38" width="0.1524" layer="91"/>
-<pinref part="P5" gate="G$1" pin="3"/>
+<label x="248.92" y="231.14" size="1.9304" layer="95" font="vector" ratio="10" rot="MR0" xref="yes"/>
+<wire x1="248.92" y1="231.14" x2="271.78" y2="231.14" width="0.1524" layer="91"/>
+<pinref part="P1" gate="G$1" pin="9"/>
 </segment>
 </net>
 <net name="D3" class="0">
 <segment>
-<label x="251.46" y="243.84" size="1.9304" layer="95" font="vector" ratio="10" rot="MR0" xref="yes"/>
-<wire x1="271.78" y1="243.84" x2="251.46" y2="243.84" width="0.1524" layer="91"/>
-<pinref part="P5" gate="G$1" pin="4"/>
+<label x="264.16" y="228.6" size="1.9304" layer="95" font="vector" ratio="10" rot="MR0" xref="yes"/>
+<wire x1="264.16" y1="228.6" x2="271.78" y2="228.6" width="0.1524" layer="91"/>
+<pinref part="P1" gate="G$1" pin="10"/>
 </segment>
 </net>
 <net name="D4" class="0">
 <segment>
-<label x="264.16" y="241.3" size="1.9304" layer="95" font="vector" ratio="10" rot="MR0" xref="yes"/>
-<wire x1="271.78" y1="241.3" x2="264.16" y2="241.3" width="0.1524" layer="91"/>
-<pinref part="P5" gate="G$1" pin="5"/>
+<wire x1="271.78" y1="226.06" x2="248.92" y2="226.06" width="0.1524" layer="91"/>
+<label x="248.92" y="226.06" size="1.9304" layer="95" font="vector" ratio="10" rot="MR0" xref="yes"/>
+<pinref part="P1" gate="G$1" pin="11"/>
 </segment>
 </net>
 <net name="D5" class="0">
 <segment>
-<label x="251.46" y="238.76" size="1.9304" layer="95" font="vector" ratio="10" rot="MR0" xref="yes"/>
-<wire x1="271.78" y1="238.76" x2="251.46" y2="238.76" width="0.1524" layer="91"/>
-<pinref part="P5" gate="G$1" pin="6"/>
+<wire x1="264.16" y1="223.52" x2="271.78" y2="223.52" width="0.1524" layer="91"/>
+<label x="264.16" y="223.52" size="1.9304" layer="95" font="vector" ratio="10" rot="MR0" xref="yes"/>
+<pinref part="P1" gate="G$1" pin="12"/>
 </segment>
 </net>
 <net name="D6" class="0">
 <segment>
-<label x="264.16" y="236.22" size="1.9304" layer="95" font="vector" ratio="10" rot="MR0" xref="yes"/>
-<wire x1="264.16" y1="236.22" x2="271.78" y2="236.22" width="0.1524" layer="91"/>
-<pinref part="P5" gate="G$1" pin="7"/>
+<wire x1="248.92" y1="220.98" x2="271.78" y2="220.98" width="0.1524" layer="91"/>
+<label x="248.92" y="220.98" size="1.9304" layer="95" font="vector" ratio="10" rot="MR0" xref="yes"/>
+<pinref part="P1" gate="G$1" pin="13"/>
 </segment>
 </net>
 <net name="D7" class="0">
 <segment>
-<label x="251.46" y="233.68" size="1.9304" layer="95" font="vector" ratio="10" rot="MR0" xref="yes"/>
-<wire x1="271.78" y1="233.68" x2="251.46" y2="233.68" width="0.1524" layer="91"/>
-<pinref part="P5" gate="G$1" pin="8"/>
+<label x="264.16" y="218.44" size="1.9304" layer="95" font="vector" ratio="10" rot="MR0" xref="yes"/>
+<wire x1="264.16" y1="218.44" x2="271.78" y2="218.44" width="0.1524" layer="91"/>
+<pinref part="P1" gate="G$1" pin="14"/>
 </segment>
 </net>
 <net name="LE2" class="0">
 <segment>
-<wire x1="271.78" y1="228.6" x2="251.46" y2="228.6" width="0.1524" layer="91"/>
-<label x="251.46" y="228.6" size="1.9304" layer="95" font="vector" ratio="10" rot="MR0" xref="yes"/>
-<pinref part="P5" gate="G$1" pin="10"/>
+<wire x1="271.78" y1="210.82" x2="248.92" y2="210.82" width="0.1524" layer="91"/>
+<label x="248.92" y="210.82" size="1.9304" layer="95" font="vector" ratio="10" rot="MR0" xref="yes"/>
+<pinref part="P1" gate="G$1" pin="17"/>
 </segment>
 </net>
 <net name="X_MSB" class="0">
 <segment>
-<pinref part="P5" gate="G$1" pin="11"/>
-<wire x1="271.78" y1="226.06" x2="264.16" y2="226.06" width="0.1524" layer="91"/>
-<label x="264.16" y="226.06" size="1.9304" layer="95" font="vector" ratio="10" rot="MR0" xref="yes"/>
+<wire x1="248.92" y1="205.74" x2="271.78" y2="205.74" width="0.1524" layer="91"/>
+<label x="248.92" y="205.74" size="1.9304" layer="95" font="vector" ratio="10" rot="MR0" xref="yes"/>
+<pinref part="P1" gate="G$1" pin="19"/>
 </segment>
 </net>
 <net name="X_LSB" class="0">
 <segment>
-<pinref part="P5" gate="G$1" pin="12"/>
-<wire x1="271.78" y1="223.52" x2="251.46" y2="223.52" width="0.1524" layer="91"/>
-<label x="251.46" y="223.52" size="1.9304" layer="95" font="vector" ratio="10" rot="MR0" xref="yes"/>
+<wire x1="271.78" y1="203.2" x2="264.16" y2="203.2" width="0.1524" layer="91"/>
+<label x="264.16" y="203.2" size="1.9304" layer="95" font="vector" ratio="10" rot="MR0" xref="yes"/>
+<pinref part="P1" gate="G$1" pin="20"/>
 </segment>
 </net>
 <net name="Y_MSB" class="0">
 <segment>
-<pinref part="P5" gate="G$1" pin="13"/>
-<wire x1="271.78" y1="220.98" x2="264.16" y2="220.98" width="0.1524" layer="91"/>
-<label x="264.16" y="220.98" size="1.9304" layer="95" font="vector" ratio="10" rot="MR0" xref="yes"/>
+<wire x1="271.78" y1="200.66" x2="248.92" y2="200.66" width="0.1524" layer="91"/>
+<label x="248.92" y="200.66" size="1.9304" layer="95" font="vector" ratio="10" rot="MR0" xref="yes"/>
+<pinref part="P1" gate="G$1" pin="21"/>
 </segment>
 </net>
 <net name="Y_LSB" class="0">
 <segment>
-<pinref part="P5" gate="G$1" pin="14"/>
-<wire x1="271.78" y1="218.44" x2="251.46" y2="218.44" width="0.1524" layer="91"/>
-<label x="251.46" y="218.44" size="1.9304" layer="95" font="vector" ratio="10" rot="MR0" xref="yes"/>
+<wire x1="271.78" y1="198.12" x2="264.16" y2="198.12" width="0.1524" layer="91"/>
+<label x="264.16" y="198.12" size="1.9304" layer="95" font="vector" ratio="10" rot="MR0" xref="yes"/>
+<pinref part="P1" gate="G$1" pin="22"/>
 </segment>
 </net>
 <net name="GND" class="0">
 <segment>
-<wire x1="292.1" y1="243.84" x2="299.72" y2="243.84" width="0.1524" layer="91"/>
-<label x="299.72" y="243.84" size="1.9304" layer="95" font="vector" ratio="10" xref="yes"/>
-<pinref part="P5" gate="G$1" pin="D"/>
+<pinref part="SUPPLY20" gate="GND" pin="GND"/>
+<wire x1="314.96" y1="243.84" x2="292.1" y2="243.84" width="0.1524" layer="91"/>
+<pinref part="P1" gate="G$1" pin="D"/>
+</segment>
+<segment>
+<pinref part="SUPPLY24" gate="GND" pin="GND"/>
+<wire x1="248.92" y1="243.84" x2="271.78" y2="243.84" width="0.1524" layer="91"/>
+<pinref part="P1" gate="G$1" pin="4"/>
 </segment>
 </net>
 <net name="+5V" class="0">
 <segment>
-<label x="299.72" y="248.92" size="1.9304" layer="95" font="vector" ratio="10" xref="yes"/>
-<wire x1="292.1" y1="248.92" x2="299.72" y2="248.92" width="0.1524" layer="91"/>
-<pinref part="P5" gate="G$1" pin="B"/>
+<pinref part="SUPPLY19" gate="+5V" pin="+5V"/>
+<wire x1="314.96" y1="248.92" x2="292.1" y2="248.92" width="0.1524" layer="91"/>
+<pinref part="P1" gate="G$1" pin="B"/>
 </segment>
 </net>
+<net name="LE3" class="0">
+<segment>
+<wire x1="271.78" y1="208.28" x2="264.16" y2="208.28" width="0.1524" layer="91"/>
+<label x="264.16" y="208.28" size="1.9304" layer="95" font="vector" ratio="10" rot="MR0" xref="yes"/>
+<pinref part="P1" gate="G$1" pin="18"/>
+</segment>
+</net>
