File: backplane/backplane.brd (EAGLE design)
At the start: 431.8 x 127 mm, 14 parts, among them J1 44PINEDGECONNECTOR, J2 44PINEDGECONNECTOR, P1 44PINEDGECONNECTOR, P10 44PINEDGECONNECTOR, P11 44PINEDGECONNECTOR, P12 44PINEDGECONNECTOR, P2 44PINEDGECONNECTOR, P3 44PINEDGECONNECTOR, P4 44PINEDGECONNECTOR, P5 44PINEDGECONNECTOR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

Commit message: added missing connector on bckplane
Parts:
- removed P10: 44PINEDGECONNECTOR, keiths:44PINEDGECONN
- added P13: PASSTHROUGH, keiths:PASSTHROUGH
Connections:
- net +10V: now also P13.P$1
- net +15V: now also P13.P$6
- net +50V: now also P13.P$7
- net +5V: now also P13.P$2
- net -10V: now also P13.P$5
- net -15V: now also P13.P$3
- net GND: now also P13.P$4
Routing:
- net +50V: track 30.3 -> 264.9 mm
- net -10V: track 91.7 -> 263.7 mm
- net +15V: track 0.00 -> 93.7 mm
- net -15V: track 228.4 -> 313.0 mm
- net +10V: track 209.0 -> 293.6 mm
- net +5V: track 63.4 -> 96.1 mm
- net GND: track 334.4 -> 365.1 mm
Other:
- board text added: "Power"
