File: backplane/backplane.sch (EAGLE design)
At the start: 14 parts, among them J1 44PINEDGE, J2 44PINEDGE, P1 44PINEDGE, P10 44PINEDGE, P11 44PINEDGE, P12 44PINEDGE, P2 44PINEDGE, P3 44PINEDGE, P4 44PINEDGE, P5 44PINEDGE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

Commit message: revised artwork
Parts:
- J1, J2, P1, P10, P11, P12, P2, P3, P4, P5, P6, P7, P8: value 44PINEDGE -> 44PINEDGECONNECTOR; device keiths:44PINEDGE -> keiths:44PINEDGECONNECTOR
- P9: value 44PINEDGE -> 44PINEDGE-FCONNECTOR; device keiths:44PINEDGE -> keiths:44PINEDGE-FCONNECTOR
Connections:
- net X_FF_OUT renamed X_FF_OUT_P
- net Y_FF_OUT renamed Y_FF_OUT_P
- removed net H_IN: P4.H, P5.H
- removed net H_OUT: J1.H, J2.H
- removed net J_IN: P12.J
- removed net K_IN: P4.K, P5.K
- removed net P_IN: P12.P
- removed net U_IN: P12.U
- removed net X_IN: P12.X
- new net N$1: P1.C
- new net X_FF_OUT_H: J1.H, P4.H
- new net Y_FF_OUT_H: J2.H, P5.H
- net +10V: no longer P1.A
- net +15V: now also P3.5; no longer P1.E, P3.E
- net +5V: now also P2.B
- net -15V: now also J1.3, J2.3, P12.3, P3.3, P4.3, P5.3; no longer P1.C
- net D0: now also P2.7
- net D1: now also P2.8
- net D2: now also P2.9
- net D3: now also P2.10
- net D4: now also P2.11
- net D5: now also P2.12
- net D6: now also P2.13
- net D7: now also P2.14
- net GND: now also J1.4, J2.4, P1.4, P11.4, P12.4, P2.4, P2.D, P3.4, P4.4, P5.4, P6.4, P7.4
- net INTENSIFY_P: now also P12.P
- net J_INTEN: now also P12.J
- net LE1: now also P2.16
- net LE2: now also P2.17
- net LE3: now also P2.18
- net U_INTEN: now also P12.U
- net X_INTEN: now also P12.X
- net X_LSB: now also P2.20
- net X_MSB: now also P2.19, P4.K
- net Y_LSB: now also P2.22
- net Y_MSB: now also P2.21, P5.K
Other:
- note removed: "intensity"
- note removed: "scale"

Commit message: added missing connector on bckplane
Parts:
- removed P10: 44PINEDGECONNECTOR, keiths:44PINEDGECONNECTOR
- added P13: PASSTHROUGH, keiths:PASSTHROUGH
Connections:
- net +10V: now also P13.1
- net +15V: now also P13.6
- net +50V: now also P13.7
- net +5V: now also P13.2
- net -10V: now also P13.5
- net -15V: now also P13.3
- net GND: now also P13.4
Other:
- note added: "Power"
Changed lines of the file:
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@@
 <part name="P8" library="keiths" deviceset="44PINEDGE" device="CONNECTOR"/>
 <part name="P9" library="keiths" deviceset="44PINEDGE-F" device="CONNECTOR"/>
-<part name="P10" library="keiths" deviceset="44PINEDGE" device="CONNECTOR"/>
 <part name="P11" library="keiths" deviceset="44PINEDGE" device="CONNECTOR"/>
 <part name="P12" library="keiths" deviceset="44PINEDGE" device="CONNECTOR"/>
@@
 <part name="SUPPLY50" library="keiths" deviceset="-15V" device=""/>
 <part name="SUPPLY51" library="keiths" deviceset="+15V" device=""/>
+<part name="SUPPLY3" library="keiths" deviceset="+50V" device=""/>
+<part name="SUPPLY25" library="keiths" deviceset="+50V" device=""/>
+<part name="SUPPLY27" library="keiths" deviceset="+50V" device=""/>
+<part name="SUPPLY28" library="keiths" deviceset="+5V" device=""/>
+<part name="SUPPLY45" library="keiths" deviceset="GND" device=""/>
+<part name="SUPPLY52" library="supply2" deviceset="+10V" device=""/>
+<part name="SUPPLY53" library="keiths" deviceset="-15V" device=""/>
+<part name="SUPPLY56" library="keiths" deviceset="+15V" device=""/>
+<part name="SUPPLY57" library="supply2" deviceset="-10V" device=""/>
+<part name="P13" library="keiths" deviceset="PASSTHROUGH" device=""/>
 </parts>
 <sheets>
@@
 <text x="325.12" y="149.86" size="2.1844" layer="91" font="vector" ratio="10">Variable Intensifier</text>
 <text x="457.2" y="149.86" size="2.1844" layer="91" font="vector" ratio="10">Bias and Focus</text>
+<text x="73.66" y="322.58" size="2.1844" layer="91" font="vector" ratio="10">Power</text>
 </plain>
 <instances>
@@
 <attribute name="VALUE" x="205.74" y="69.85" size="1.778" layer="96"/>
 </instance>
-<instance part="P10" gate="G$1" x="78.74" y="360.68" smashed="yes">
-<attribute name="NAME" x="74.93" y="388.62" size="1.778" layer="95"/>
-<attribute name="VALUE" x="73.66" y="328.93" size="1.778" layer="96" display="off"/>
-</instance>
 <instance part="P11" gate="G$1" x="469.9" y="187.96" smashed="yes">
 <attribute name="NAME" x="466.09" y="215.9" size="1.778" layer="95"/>
@@
 <instance part="SUPPLY51" gate="+15V" x="449.58" y="375.92" smashed="yes" rot="R90">
 <attribute name="VALUE" x="445.516" y="376.809" size="1.9304" layer="96" font="vector" ratio="10" rot="R180"/>
+</instance>
+<instance part="SUPPLY3" gate="+50V" x="114.3" y="360.68" smashed="yes" rot="R270">
+<attribute name="VALUE" x="117.729" y="359.791" size="1.9304" layer="96" font="vector" ratio="10"/>
+</instance>
+<instance part="SUPPLY25" gate="+50V" x="114.3" y="187.96" smashed="yes" rot="R270">
+<attribute name="VALUE" x="117.729" y="187.071" size="1.9304" layer="96" font="vector" ratio="10"/>
+</instance>
+<instance part="SUPPLY27" gate="+50V" x="246.38" y="187.96" smashed="yes" rot="R270">
+<attribute name="VALUE" x="249.809" y="187.071" size="1.9304" layer="96" font="vector" ratio="10"/>
+</instance>
+<instance part="SUPPLY28" gate="+5V" x="99.06" y="383.54" smashed="yes" rot="R270">
+<attribute name="VALUE" x="102.489" y="382.397" size="1.9304" layer="96" font="vector" ratio="10"/>
+</instance>
+<instance part="SUPPLY45" gate="GND" x="99.06" y="378.46" smashed="yes" rot="R90">
+<attribute name="VALUE" x="102.489" y="377.825" size="1.9304" layer="96" font="vector" ratio="10"/>
+</instance>
+<instance part="SUPPLY52" gate="G$1" x="114.3" y="386.08" smashed="yes" rot="MR90">
+<attribute name="VALUE" x="118.364" y="386.969" size="1.9304" layer="96" font="vector" ratio="10" rot="MR180"/>
+</instance>
+<instance part="SUPPLY53" gate="G$1" x="114.3" y="381" smashed="yes" rot="R90">
+<attribute name="VALUE" x="118.237" y="380.111" size="1.9304" layer="96" font="vector" ratio="10"/>
+</instance>
+<instance part="SUPPLY56" gate="+15V" x="99.06" y="373.38" smashed="yes" rot="MR90">
+<attribute name="VALUE" x="103.124" y="374.269" size="1.9304" layer="96" font="vector" ratio="10" rot="MR180"/>
+</instance>
+<instance part="SUPPLY57" gate="G$1" x="114.3" y="375.92" smashed="yes" rot="R90">
+<attribute name="VALUE" x="118.237" y="374.777" size="1.9304" layer="96" font="vector" ratio="10"/>
+</instance>
+<instance part="P13" gate="G$1" x="78.74" y="360.68" smashed="yes">
+<attribute name="NAME" x="74.93" y="388.62" size="1.778" layer="95"/>
+<attribute name="VALUE" x="73.66" y="328.93" size="1.778" layer="96" display="off"/>
 </instance>
 </instances>
@@
 <pinref part="P2" gate="G$1" pin="B"/>
 </segment>
+<segment>
+<pinref part="P13" gate="G$1" pin="2"/>
+<pinref part="SUPPLY28" gate="+5V" pin="+5V"/>
+<wire x1="96.52" y1="383.54" x2="88.9" y2="383.54" width="0.1524" layer="91"/>
+</segment>
 </net>
 <net name="GND" class="0">
@@
 <wire x1="45.72" y1="205.74" x2="68.58" y2="205.74" width="0.1524" layer="91"/>
 </segment>
+<segment>
+<pinref part="P13" gate="G$1" pin="4"/>
+<pinref part="SUPPLY45" gate="GND" pin="GND"/>
+<wire x1="96.52" y1="378.46" x2="88.9" y2="378.46" width="0.1524" layer="91"/>
+</segment>
 </net>
 <net name="X_INTEN" class="0">
@@
 <wire x1="452.12" y1="375.92" x2="459.74" y2="375.92" width="0.1524" layer="91"/>
 </segment>
+<segment>
+<pinref part="P13" gate="G$1" pin="6"/>
+<pinref part="SUPPLY56" gate="+15V" pin="+15V"/>
+<wire x1="96.52" y1="373.38" x2="88.9" y2="373.38" width="0.1524" layer="91"/>
+</segment>
 </net>
 <net name="-15V" class="0">
@@
 <wire x1="60.96" y1="294.64" x2="68.58" y2="294.64" width="0.1524" layer="91"/>
 </segment>
+<segment>
+<pinref part="P13" gate="G$1" pin="3"/>
+<pinref part="SUPPLY53" gate="G$1" pin="-15V"/>
+<wire x1="111.76" y1="381" x2="88.9" y2="381" width="0.1524" layer="91"/>
+</segment>
 </net>
 <net name="+10V" class="0">
@@
 <pinref part="SUPPLY44" gate="G$1" pin="+10V"/>
 </segment>
+<segment>
+<pinref part="P13" gate="G$1" pin="1"/>
+<pinref part="SUPPLY52" gate="G$1" pin="+10V"/>
+<wire x1="111.76" y1="386.08" x2="88.9" y2="386.08" width="0.1524" layer="91"/>
+</segment>
 </net>
 <net name="Y_LSB" class="0">
@@
 <wire x1="353.06" y1="289.56" x2="360.68" y2="289.56" width="0.1524" layer="91"/>
 </segment>
-</net>
-<net name="+50V" class="0">
-<segment>
-<label x="111.76" y="187.96" size="1.9304" layer="95" font="vector" ratio="10" xref="yes"/>
-<pinref part="P6" gate="G$1" pin="M"/>
-<wire x1="88.9" y1="187.96" x2="111.76" y2="187.96" width="0.1524" layer="91"/>
-</segment>
-<segment>
-<label x="243.84" y="187.96" size="1.9304" layer="95" font="vector" ratio="10" xref="yes"/>
-<pinref part="P7" gate="G$1" pin="M"/>
-<wire x1="220.98" y1="187.96" x2="243.84" y2="187.96" width="0.1524" layer="91"/>
+<segment>
+<pinref part="P13" gate="G$1" pin="5"/>
+<pinref part="SUPPLY57" gate="G$1" pin="-10V"/>
+<wire x1="111.76" y1="375.92" x2="88.9" y2="375.92" width="0.1524" layer="91"/>
 </segment>
 </net>
@@
 </segment>
 </net>
+<net name="+50V" class="0">
+<segment>
+<pinref part="SUPPLY27" gate="+50V" pin="+50V"/>
+<pinref part="P7" gate="G$1" pin="M"/>
+<wire x1="220.98" y1="187.96" x2="243.84" y2="187.96" width="0.1524" layer="91"/>
+</segment>
+<segment>
+<pinref part="P6" gate="G$1" pin="M"/>
+<pinref part="SUPPLY25" gate="+50V" pin="+50V"/>
+<wire x1="111.76" y1="187.96" x2="88.9" y2="187.96" width="0.1524" layer="91"/>
+</segment>
+<segment>
+<pinref part="P13" gate="G$1" pin="7"/>
+<pinref part="SUPPLY3" gate="+50V" pin="+50V"/>
+<wire x1="111.76" y1="360.68" x2="88.9" y2="360.68" width="0.1524" layer="91"/>
+</segment>
+</net>
